File: examples/test_usb_source_measure/design.kicad_pcb (KiCad board)
At the start: 4 copper layers, 120 parts

Commit message: break up big clump
Parts:
- moved reg_5v.fb.top_res 170.4 mm to (34.0, 29.0)
- moved ref_buf.vdd_cap 167.0 mm to (50.0, 51.0)
- moved led_analog.package 157.7 mm to (66.0, 44.0)
- moved reg_5v.hf_in_cap 155.2 mm to (46.8, 15.0)
- moved reg_5v.fb.bottom_res 151.0 mm to (36.0, 35.0)
- moved outp 144.9 mm to (216.0, 73.0), turned to 180 degrees
- moved control.vmeas.amp.vdd_cap 142.3 mm to (41.0, -21.0)
- moved outn 140.4 mm to (215.0, 51.0), turned to 180 degrees
- moved ref_div.bottom_res 139.4 mm to (59.0, 50.0)
- moved control.err_volt.rbot 137.3 mm to (55.0, -4.00)
- moved control.err_source.amp.vdd_cap 136.7 mm to (76.0, 16.0)
- moved control.err_volt.amp.vdd_cap 134.4 mm to (54.0, -7.00)
- moved reg_5v.out_cap 133.6 mm to (50.0, 31.0)
- moved control.err_volt.rout 132.9 mm to (59.0, -9.00)
- moved control.err_volt.rtop 131.3 mm to (65.0, -7.00)
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