File: examples/test_tofarray/TofArrayTest.kicad_pcb (KiCad board)
At the start: 2 copper layers, 200 x 25 mm, 63 parts, among them sw1 3.9x2.9mm Switch

Commit message: Update TofArrayTest.kicad_pcb
Routing:
- net v3v3: track 126.7 -> 346.5 mm, vias 14 -> 13
- net vusb: track 19.8 -> 53.8 mm, vias 4 -> 5
- net usb.S1: track 0.00 -> 17.0 mm
Changed lines of the file:
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@@
     (thickness 1.6)
     (drawings 11)
-    (tracks 454)
+    (tracks 467)
     (zones 0)
     (modules 63)
@@
   (segment (start 83.05 43.95) (end 82 45) (width 0.5) (layer F.Cu) (net 2))
   (segment (start 102.175 51) (end 102.175 49) (width 0.25) (layer F.Cu) (net 2))
-  (via (at 102 50) (size 0.7) (drill 0.3) (layers F.Cu B.Cu) (net 2))
-  (segment (start 102.175 50.175) (end 102 50) (width 0.25) (layer F.Cu) (net 2))
   (segment (start 102.175 51) (end 102.175 50.175) (width 0.25) (layer F.Cu) (net 2))
   (segment (start 93.65 47.65) (end 94 48) (width 0.5) (layer F.Cu) (net 2))
@@
   (segment (start 93.65 45) (end 95 45) (width 0.5) (layer F.Cu) (net 2))
   (segment (start 98 43.35) (end 96.65 43.35) (width 0.5) (layer F.Cu) (net 2))
+  (segment (start 74.5 39) (end 68.5 45) (width 0.5) (layer B.Cu) (net 2))
+  (segment (start 94 39) (end 74.5 39) (width 0.5) (layer B.Cu) (net 2))
+  (segment (start 94 42) (end 94 39) (width 0.5) (layer B.Cu) (net 2))
+  (segment (start 188.5 45) (end 188.5 39) (width 0.5) (layer B.Cu) (net 2))
+  (segment (start 228.5 39) (end 228.5 45) (width 0.5) (layer B.Cu) (net 2))
+  (segment (start 148.5 39) (end 228.5 39) (width 0.5) (layer B.Cu) (net 2))
+  (segment (start 148.5 45) (end 148.5 39) (width 0.5) (layer B.Cu) (net 2))
+  (segment (start 131 49) (end 131 39) (width 0.5) (layer B.Cu) (net 2))
+  (segment (start 131 39) (end 148.5 39) (width 0.5) (layer B.Cu) (net 2))
+  (segment (start 108.5 45) (end 108.5 39) (width 0.5) (layer B.Cu) (net 2))
+  (segment (start 108.5 39) (end 131 39) (width 0.5) (layer B.Cu) (net 2))
+  (segment (start 94 39) (end 108.5 39) (width 0.5) (layer B.Cu) (net 2))
+  (segment (start 102.175 49) (end 102.175 46.825) (width 0.2) (layer F.Cu) (net 2))
+  (segment (start 104 45) (end 108.5 45) (width 0.2) (layer F.Cu) (net 2))
+  (segment (start 102.175 46.825) (end 104 45) (width 0.2) (layer F.Cu) (net 2))
+  (segment (start 68.5 45) (end 68 45) (width 0.2) (layer F.Cu) (net 2))
+  (segment (start 68 45) (end 66 47) (width 0.2) (layer F.Cu) (net 2))
+  (segment (start 66 51.5) (end 63.5 54) (width 0.2) (layer F.Cu) (net 2))
+  (segment (start 66 47) (end 66 51.5) (width 0.2) (layer F.Cu) (net 2))
   (segment (start 170.775 54) (end 170.775 54.775) (width 0.25) (layer F.Cu) (net 3))
   (segment (start 170.95 54.95) (end 170.95 56) (width 0.25) (layer F.Cu) (net 3))
@@
   (segment (start 61.5 47.5) (end 62 47) (width 0.25) (layer F.Cu) (net 3))
   (segment (start 58.5 47.5) (end 61.5 47.5) (width 0.25) (layer F.Cu) (net 3))
+  (via (at 84 49) (size 1.2) (drill 0.8) (layers F.Cu B.Cu) (net 3))
+  (segment (start 84 47.775) (end 84 49) (width 0.5) (layer F.Cu) (net 3))
+  (segment (start 63.5 47.5) (end 58.5 47.5) (width 0.5) (layer B.Cu) (net 3))
+  (segment (start 67 51) (end 63.5 47.5) (width 0.5) (layer B.Cu) (net 3))
+  (segment (start 82 51) (end 67 51) (width 0.5) (layer B.Cu) (net 3))
+  (segment (start 84 49) (end 82 51) (width 0.5) (layer B.Cu) (net 3))
+  (segment (start 58.5 52.5) (end 58.5 47.5) (width 0.5) (layer B.Cu) (net 3))
   (segment (start 143.85 51.1) (end 143.85 50.85) (width 0.16) (layer F.Cu) (net 9))
   (segment (start 143.85 50.85) (end 143 50) (width 0.16) (layer F.Cu) (net 9))
@@
   (segment (start 146 43) (end 148 41) (width 0.2) (layer F.Cu) (net 11))
   (segment (start 194 43) (end 226 43) (width 0.2) (layer F.Cu) (net 11))
-  (segment (start 106 43) (end 101 43) (width 0.2) (layer F.Cu) (net 11))
-  (segment (start 101 43) (end 100 43) (width 0.2) (layer F.Cu) (net 11))
-  (segment (start 100 43) (end 97 40) (width 0.2) (layer F.Cu) (net 11))
-  (segment (start 97 40) (end 83 40) (width 0.2) (layer F.Cu) (net 11))
-  (segment (start 83 40) (end 81 42) (width 0.2) (layer F.Cu) (net 11))
-  (segment (start 81 42) (end 79 42) (width 0.2) (layer F.Cu) (net 11))
-  (segment (start 79 42) (end 78 42) (width 0.2) (layer F.Cu) (net 11))
-  (segment (start 78 42) (end 77 43) (width 0.2) (layer F.Cu) (net 11))
-  (segment (start 77 43) (end 74 43) (width 0.2) (layer F.Cu) (net 11))
-  (segment (start 74 43) (end 72 41) (width 0.2) (layer F.Cu) (net 11))
-  (segment (start 72 41) (end 69 41) (width 0.2) (layer F.Cu) (net 11))
-  (segment (start 69 41) (end 67 43) (width 0.2) (layer F.Cu) (net 11))
   (segment (start 106 47) (end 106 43) (width 0.2) (layer B.Cu) (net 11))
   (segment (start 108 49) (end 106 47) (width 0.2) (layer B.Cu) (net 11))
@@
   (via (at 68 49) (size 0.7) (drill 0.3) (layers F.Cu B.Cu) (net 11))
   (segment (start 69.2 49.2) (end 68.2 49.2) (width 0.2) (layer F.Cu) (net 11))
-  (via (at 67 43) (size 0.7) (drill 0.3) (layers F.Cu B.Cu) (net 11))
-  (segment (start 67 48) (end 67 43) (width 0.2) (layer B.Cu) (net 11))
-  (segment (start 68 49) (end 67 48) (width 0.2) (layer B.Cu) (net 11))
   (segment (start 143.5 43) (end 146 43) (width 0.2) (layer F.Cu) (net 11))
   (segment (start 142.5 42) (end 143.5 43) (width 0.2) (layer F.Cu) (net 11))
@@
   (segment (start 108 41) (end 112 41) (width 0.2) (layer F.Cu) (net 11))
   (segment (start 106 43) (end 108 41) (width 0.2) (layer F.Cu) (net 11))
+  (via (at 66 43) (size 0.7) (drill 0.3) (layers F.Cu B.Cu) (net 11))
+  (segment (start 69 40) (end 66 43) (width 0.2) (layer F.Cu) (net 11))
+  (segment (start 99 40) (end 69 40) (width 0.2) (layer F.Cu) (net 11))
+  (segment (start 102 43) (end 99 40) (width 0.2) (layer F.Cu) (net 11))
+  (segment (start 106 43) (end 102 43) (width 0.2) (layer F.Cu) (net 11))
+  (segment (start 66 47) (end 66 43) (width 0.2) (layer B.Cu) (net 11))
+  (segment (start 68 49) (end 66 47) (width 0.2) (layer B.Cu) (net 11))
   (via (at 148 50) (size 0.7) (drill 0.3) (layers F.Cu B.Cu) (net 12))
   (segment (start 149.2 50) (end 148 50) (width 0.2) (layer F.Cu) (net 12))
@@
   (segment (start 109.2 50) (end 108 50) (width 0.25) (layer F.Cu) (net 12))
   (segment (start 108 50) (end 106 50) (width 0.25) (layer F.Cu) (net 12))
-  (segment (start 74 42) (end 72 40) (width 0.2) (layer F.Cu) (net 12))
-  (segment (start 77 42) (end 74 42) (width 0.2) (layer F.Cu) (net 12))
-  (segment (start 78 41) (end 77 42) (width 0.2) (layer F.Cu) (net 12))
-  (segment (start 69 40) (end 67 42) (width 0.2) (layer F.Cu) (net 12))
-  (segment (start 97 39) (end 83 39) (width 0.2) (layer F.Cu) (net 12))
-  (segment (start 83 39) (end 81 41) (width 0.2) (layer F.Cu) (net 12))
-  (segment (start 100 42) (end 97 39) (width 0.2) (layer F.Cu) (net 12))
-  (segment (start 72 40) (end 69 40) (width 0.2) (layer F.Cu) (net 12))
-  (segment (start 81 41) (end 78 41) (width 0.2) (layer F.Cu) (net 12))
   (segment (start 105 47) (end 105 42) (width 0.2) (layer B.Cu) (net 12))
   (segment (start 108 50) (end 105 47) (width 0.2) (layer B.Cu) (net 12))
-  (segment (start 105 42) (end 100 42) (width 0.2) (layer F.Cu) (net 12))
   (via (at 105 42) (size 0.7) (drill 0.3) (layers F.Cu B.Cu) (net 12))
   (segment (start 148 50) (end 145 47) (width 0.2) (layer B.Cu) (net 12))
@@
   (via (at 68 50) (size 0.7) (drill 0.3) (layers F.Cu B.Cu) (net 12))
   (segment (start 69.2 50) (end 68 50) (width 0.2) (layer F.Cu) (net 12))
-  (segment (start 68 50) (end 66 48) (width 0.2) (layer B.Cu) (net 12))
-  (via (at 66 42) (size 0.7) (drill 0.3) (layers F.Cu B.Cu) (net 12))
-  (segment (start 66 48) (end 66 42) (width 0.2) (layer B.Cu) (net 12))
-  (segment (start 66 42) (end 67 42) (width 0.2) (layer F.Cu) (net 12))
   (segment (start 106 42) (end 105 42) (width 0.2) (layer F.Cu) (net 12))
   (segment (start 108 40) (end 106 42) (width 0.2) (layer F.Cu) (net 12))
@@
   (segment (start 112 40) (end 108 40) (width 0.2) (layer F.Cu) (net 12))
   (segment (start 114 42) (end 112 40) (width 0.2) (layer F.Cu) (net 12))
+  (via (at 65 42) (size 0.7) (drill 0.3) (layers F.Cu B.Cu) (net 12))
+  (segment (start 65 47) (end 65 42) (width 0.2) (layer B.Cu) (net 12))
+  (segment (start 68 50) (end 65 47) (width 0.2) (layer B.Cu) (net 12))
+  (segment (start 66 42) (end 65 42) (width 0.2) (layer F.Cu) (net 12))
+  (segment (start 69 39) (end 66 42) (width 0.2) (layer F.Cu) (net 12))
+  (segment (start 99 39) (end 69 39) (width 0.2) (layer F.Cu) (net 12))
+  (segment (start 102 42) (end 99 39) (width 0.2) (layer F.Cu) (net 12))
+  (segment (start 105 42) (end 102 42) (width 0.2) (layer F.Cu) (net 12))
   (segment (start 57.863002 50.25) (end 57.17 50.25) (width 0.2) (layer F.Cu) (net 24))
   (segment (start 58.005001 50.108001) (end 57.863002 50.25) (width 0.2) (layer F.Cu) (net 24))
@@
   (segment (start 163.175 49.325) (end 163.5 49) (width 0.2) (layer F.Cu) (net 31))
   (segment (start 163.5 49) (end 164.5 49) (width 0.2) (layer F.Cu) (net 31))
+  (segment (start 52.425 54.32) (end 56.605 54.32) (width 0.25) (layer F.Cu) (net 32))
+  (segment (start 52.425 54.32) (end 52.425 45.68) (width 0.25) (layer F.Cu) (net 32))
+  (segment (start 52.425 45.68) (end 56.605 45.68) (width 0.25) (layer F.Cu) (net 32))
   (segment (start 167.85 51.325) (end 166.325 51.325) (width 0.2) (layer F.Cu) (net 36))
   (segment (start 166.325 51.325) (end 166 51) (width 0.2) (layer F.Cu) (net 36))

Commit message: infra & global routing
Parts:
- moved matrix_res2 41.4 mm to (116.0, 53.0)
- moved rgb.package 37.5 mm to (103.0, 50.0), turned to 90 degrees
- moved matrix_res1 31.4 mm to (116.0, 47.0)
- moved i2c_pull.scl_res 27.0 mm to (76.0, 49.0), turned to 180 degrees
- moved i2c_pull.sda_res 27.0 mm to (76.0, 51.0), turned to 180 degrees
- moved sw1 3.61 mm to (117.0, 24.0)
- moved leds.led[0].package 2.00 mm to (70.0, 55.0)
- moved leds.led[1].package 2.00 mm to (110.0, 55.0)
- moved leds.led[2].package 2.00 mm to (150.0, 55.0)
- moved leds.led[3].package 2.00 mm to (190.0, 55.0)
- moved leds.led[4].package 2.00 mm to (230.0, 55.0)
- moved spk 1.00 mm to (179.0, 49.0)
- moved spk_dac.c 1.00 mm to (160.0, 49.0)
- moved spk_dac.r 1.00 mm to (160.0, 51.0)
- moved spk_drv.bulk_cap 1.00 mm to (170.0, 55.0)
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Routing:
- net vusb: track 53.8 -> 168.8 mm
- net mcu.swd.swd.reset: track 0.00 -> 54.3 mm, vias 0 -> 2
- net usb_chain_0.d_N: track 5.72 -> 54.7 mm
- net usb_chain_0.d_P: track 10.1 -> 58.7 mm
- net v3v3: track 346.5 -> 358.7 mm, vias 13 -> 14
- net mcu.ic.swd.swdio: track 0.00 -> 10.6 mm, vias 0 -> 1
- net mcu.ic.swd.swo: track 0.00 -> 10.0 mm, vias 0 -> 1
- net i2c_chain_0.sda: track 224.8 -> 232.8 mm, vias 10 -> 13
- net mcu.swd.swd.swclk: track 0.00 -> 6.71 mm, vias 0 -> 2
- net i2c_chain_0.scl: track 213.3 -> 219.9 mm, vias 10 -> 11
- net matrix_res2.a.3: track 0.00 -> 1.51 mm, vias 0 -> 1
- net matrix_res2.a.2: track 0.00 -> 1.51 mm, vias 0 -> 1
- net matrix_res2.a.1: track 0.00 -> 1.51 mm, vias 0 -> 1
- net gnd: track 87.0 -> 86.4 mm
