File: examples/test_robotdriver/RobotDriverAutorouted.kicad_pcb (KiCad board)
At the start: 2 copper layers, 138 x 72 mm, 68 parts, among them J1 C64658, J10 C64658, J3 C265088, J4 C265088, J5 C265088, J7 C64658, J8 C64658, J9 C64658, SW1 C318884, U1 C500769, U2 C2934560, U3 C86832, U4 C86832, U5 C967633, U6 C50506, U7 C50506

Commit message: silk labels
Other:
- board text added: "+"
- board text added: "3V3"
- board text added: "BAT"
- board text added: "M1A"
- board text added: "M1B"
- board text added: "M2A"
- board text added: "M2B"
- board text added: "RX >"
- board text added: "SCL"
- board text added: "SDA"
- board text added: "TX <"
- board text added: "ToF 0"
- board text added: "ToF 1"
- board text added: "ToF 2"
- board text added: "V+"
- board text added: "⎍"
- board text added: "⏚"
Changed lines of the file:
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@@
     )
     (pad_to_mask_clearance 0)
-    (solder_mask_min_width 0.12)
     (aux_axis_origin 138 48)
     (pcbplotparams
@@
   (gr_line (start 196 39) (end 196 111) (layer "Edge.Cuts") (width 0.05))
   (gr_line (start 58 39) (end 196 39) (layer "Edge.Cuts") (width 0.05))
+  (gr_text "SDA" (at 111 76) (layer "F.SilkS")
+    (effects (font (size 1.5 1) (thickness 0.15)) (justify left))
+  )
+  (gr_text "⎍" (at 85 85) (layer "F.SilkS")
+    (effects (font (size 1.5 1) (thickness 0.15)))
+  )
+  (gr_text "SCL" (at 111 79) (layer "F.SilkS")
+    (effects (font (size 1.5 1) (thickness 0.15)) (justify left))
+  )
+  (gr_text "M2A" (at 70 73) (layer "F.SilkS")
+    (effects (font (size 1.5 1) (thickness 0.15)) (justify left))
+  )
+  (gr_text "ToF 1" (at 130 53) (layer "F.SilkS")
+    (effects (font (size 1.5 1) (thickness 0.15)) (justify left))
+  )
+  (gr_text "⏚" (at 82 81) (layer "F.SilkS")
+    (effects (font (size 1.5 1) (thickness 0.15)) (justify left))
+  )
+  (gr_text "⏚" (at 91 85) (layer "F.SilkS")
+    (effects (font (size 1.5 1) (thickness 0.15)))
+  )
+  (gr_text "+" (at 88 81) (layer "F.SilkS")
+    (effects (font (size 1.5 1) (thickness 0.15)) (justify left))
+  )
   (gr_text "EDG Robot Driver Board v1\nAutorouted Test" (at 162 107) (layer "F.SilkS")
     (effects (font (size 1.5 1) (thickness 0.15)))
   )
+  (gr_text "+" (at 85 88) (layer "F.SilkS")
+    (effects (font (size 1.5 1) (thickness 0.15)))
+  )
+  (gr_text "TX <" (at 93 45) (layer "F.SilkS")
+    (effects (font (size 1.5 1) (thickness 0.15)) (justify left))
+  )
+  (gr_text "3V3" (at 93 43) (layer "F.SilkS")
+    (effects (font (size 1.5 1) (thickness 0.15)) (justify left))
+  )
+  (gr_text "BAT" (at 81 73) (layer "F.SilkS")
+    (effects (font (size 1.5 1) (thickness 0.15)) (justify left))
+  )
+  (gr_text "M2B" (at 70 91) (layer "F.SilkS")
+    (effects (font (size 1.5 1) (thickness 0.15)) (justify left))
+  )
+  (gr_text "M1B" (at 60 91) (layer "F.SilkS")
+    (effects (font (size 1.5 1) (thickness 0.15)) (justify left))
+  )
+  (gr_text "V+\n" (at 91 89) (layer "F.SilkS")
+    (effects (font (size 1.5 1) (thickness 0.15)))
+  )
+  (gr_text "⏚" (at 93 49) (layer "F.SilkS")
+    (effects (font (size 1.5 1) (thickness 0.15)) (justify left))
+  )
+  (gr_text "3V3" (at 97 82) (layer "F.SilkS")
+    (effects (font (size 1.5 1) (thickness 0.15)))
+  )
+  (gr_text "RX >" (at 93 47) (layer "F.SilkS")
+    (effects (font (size 1.5 1) (thickness 0.15)) (justify left))
+  )
+  (gr_text "ToF 0" (at 130 44) (layer "F.SilkS")
+    (effects (font (size 1.5 1) (thickness 0.15)) (justify left))
+  )
+  (gr_text "M1A" (at 60 73) (layer "F.SilkS")
+    (effects (font (size 1.5 1) (thickness 0.15)) (justify left))
+  )
+  (gr_text "⏚" (at 85 91) (layer "F.SilkS")
+    (effects (font (size 1.5 1) (thickness 0.15)))
+  )
+  (gr_text "ToF 2" (at 130 63) (layer "F.SilkS")
+    (effects (font (size 1.5 1) (thickness 0.15)) (justify left))
+  )
   (segment (start 180.0484 42.8628) (end 181.555 42.8628) (width 0.16) (layer "F.Cu") (net 1))
