File: examples/test_robotdriver2/RobotDriver2_Blimp.kicad_pcb (KiCad board)
At the start: 2 copper layers, 116.5 x 82.3 mm, 89 parts, among them J1 B2B-PH-K (JST), J10 B2B-PH-K (JST), J11 B2B-PH-K (JST), J12 B2B-PH-K (JST), J13 PinHeader2.54 1x3 (Generic), J2 PinHeader2.54 1x4 (Generic), J3 B6B-PH-K (JST), J4 B6B-PH-K (JST), J5 B6B-PH-K (JST), J6 FH12-15S-0.5SH (Hirose), J7 B2B-PH-K (JST), J8 B3B-PH-K (JST), J9 B2B-PH-K (JST), SW1 5.1mm switch, U1 LMV321 (Texas Instruments), U10 Duck, U11 LeadFree, U12 IdDots4, U2 AP3418 (Diodes Incorporated), U3 ESP32-WROOM-32 (Espressif Sys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, U4 LSM6DS3TR-C (STMicroelectroni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, U5 PCF8574AT (NXP), U6 TPA2005D1 (Texas Instruments), U7 DRV8833PWP (Texas Instruments), U8 DRV8833PWP (Texas Instruments), U9 Lemur

Commit message: small changes made to blimp board
Parts:
- moved U9 60.4 mm to (136.5, 115.0)
- moved U10 52.1 mm to (142.0, 115.5)
- moved U11 43.4 mm to (149.0, 114.5)
- moved U12 43.1 mm to (149.0, 117.0)
- moved H1 10.1 mm to (100.5, 48.0)
- moved H2 7.73 mm to (100.5, 113.5)
Other:
- board text added: "EDG Robot Driver Board v2a Ducky Lin Nathan Nguyendinh Kai Jun Tay"
- board text removed: "EDG Robot Driver Board v1b Ducky Lin Nathan Nguyendinh Kai Jun Tay"
Changed lines of the file:
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@@
   )
   (footprint "edg:JlcToolingHole_1.152mm" (layer "F.Cu")
-    (at 97.5 57.65)
+    (at 100.5 48)
     (descr "Tooling holes for JLC assembly, 1.152 mm hole + 1.3mm soldermask opening")
     (property "Sheetfile" "edg.BoardTop.JlcToolingHoles")
@@
   )
   (footprint "edg:Indicator_IdDots_4" (layer "F.Cu")
-    (at 183.006295 90.5)
+    (at 149 117)
     (property "Sheetfile" "")
     (property "Sheetname" "")
@@
   )
   (footprint "edg:Indicator_LeadFree" (layer "F.Cu")
-    (at 183.006295 87.5)
+    (at 149 114.5)
     (property "Sheetfile" "")
     (property "Sheetname" "")
@@
   )
   (footprint "edg:Symbol_LemurSmall" (layer "F.Cu")
-    (at 183 76.5)
+    (at 136.5 115)
     (descr "Converted using: svg2mod -i small.svg -o lemur_small.kicad_mod -c -f 0.2")
     (tags "svg2mod")
@@
   )
   (footprint "edg:JlcToolingHole_1.152mm" (layer "F.Cu")
-    (at 97.5 106.375)
+    (at 100.5 113.5)
     (descr "Tooling holes for JLC assembly, 1.152 mm hole + 1.3mm soldermask opening")
     (property "Sheetfile" "edg.BoardTop.JlcToolingHoles")
@@
   )
   (footprint "edg:Symbol_Duckling" (layer "F.Cu")
-    (at 183.006295 83.280624)
+    (at 142 115.5)
     (descr "Duckling")
     (property "Sheetfile" "")
@@
     (effects (font (size 1.5 1) (thickness 0.15)) (justify left))
   )
-  (gr_text "EDG Robot Driver Board v1b\nDucky Lin\nNathan Nguyendinh\nKai Jun Tay" (at 166 95.5) (layer "F.SilkS")
+  (gr_text "EDG Robot Driver Board v2a\nDucky Lin\nNathan Nguyendinh\nKai Jun Tay" (at 162.5 115) (layer "F.SilkS")
     (effects (font (size 0.9 0.9) (thickness 0.15)))
   )

Commit message: more traces done on the motor
Parts:
- moved D1 29.3 mm to (113.5, 67.3)
- moved C16 0.50 mm to (127.0, 91.5)
- moved D2 0.50 mm to (132.0, 93.5)
- moved D3 0.50 mm to (132.0, 95.5)
- moved D4 0.50 mm to (132.0, 97.5)
- moved D5 0.50 mm to (132.0, 99.5)
- moved R12 0.50 mm to (127.0, 93.5)
- moved R13 0.50 mm to (127.0, 95.5)
- moved R14 0.50 mm to (127.0, 97.5)
- moved R15 0.50 mm to (127.0, 99.5)
- moved U5 0.50 mm to (141.0, 95.5)
Connections:
- net expander.io.tof_xshut_2 renamed tof.xshut.2
- net isense.amp.amp.inn renamed isense.amp.r1.b
- net isense.amp.r2.b renamed isense.amp.(adapter)r2.b.src
- net lcd.device.c1n renamed lcd.c1_cap.neg
- net lcd.vcc_cap2.pwr renamed lcd.vcc_cap1.pwr
- net lcd.vcomh_cap.pos renamed lcd.device.vcomh
- net led[1].package.k renamed led[1].res.a
- net mcu.en_pull.io renamed mcu.ic.chip_pu
- net mcu.gpio.pwm renamed servo.pins.1
- net mcu.ic.io0 renamed mcu.prog.a
- net mcu.ic.uart0.rx renamed mcu.uart0.uart.tx
- net mcu.uart0.uart.rx renamed mcu.ic.uart0.tx
- net motor_driver1.vint_cap.pwr renamed motor_driver1.ic.vint
- net reg_3v3.ic.fb renamed reg_3v3.fb.center
- net spk_drv.(adapter)inn_res.b.dst renamed spk_drv.ic.inn
- net spk_drv.inn_cap.pos renamed spk_drv.inn_res.a
- net spk_drv.inp_cap.pos renamed spk_drv.inp_res.a
- net tof.xshut.0 renamed expander.io.tof_xshut_0
- net ws2812bArray.led[1].dout renamed ws2812bArray.led[2].din
- net ws2812bArray.led[2].dout renamed ws2812bArray.led[3].din
- net ws2812bArray.led[3].dout renamed ws2812bArray.led[4].din
- U7 pad 2: m1_a.pins.1 -> m1_a.pins.2
- U7 pad 4: m1_a.pins.2 -> m1_a.pins.1
- U7 pad 5: m1_b.pins.2 -> m1_b.pins.1
- U7 pad 7: m1_b.pins.1 -> m1_b.pins.2
- U8 pad 2: m2_a.pins.1 -> m2_a.pins.2
- U8 pad 4: m2_a.pins.2 -> m2_a.pins.1
- U8 pad 5: m2_b.pins.2 -> m2_b.pins.1
- U8 pad 7: m2_b.pins.1 -> m2_b.pins.2
Routing:
- net m1_b.pins.1: track 0.00 -> 20.0 mm
- net m2_b.pins.1: track 0.00 -> 18.7 mm
- net m1_b.pins.2: track 0.00 -> 14.1 mm
- net m2_b.pins.2: track 0.00 -> 12.8 mm
- net m1_a.pins.2: track 0.00 -> 11.8 mm
- net m1_a.pins.1: track 0.00 -> 10.8 mm
- net m2_a.pins.2: track 0.00 -> 10.2 mm
- net m2_a.pins.1: track 0.00 -> 9.30 mm
- net gnd: track 63.3 -> 70.4 mm

Commit message: wip layout
Parts:
- removed the R12 at (127.0, 93.5)
- removed the R13 at (127.0, 95.5)
- removed R14, R15: 0603WAF1001T5E (UNI-ROYAL(Uniroyal Elec)) - ±1% 1/10W Thick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, Resistor_SMD:R_0603_1608Metric
- added RN1: , Resistor_SMD:R_Array_Concave_4x0603, F.Cu at (131.0, 97.0)
- C1, C10, C12, C14, C15, C16, C17, C5, C7, C8: value CC0603KRX7R9BB104 (YAGEO) - 50V 100nF X7R ±10% 0603 Multilayer Ceramic Capacitors MLCC - SMD/SMT ROHS -> (none)
- C11, C18, C2, C22, C25, C3, C9: value CL21A475KAQNNNE (Samsung Electro-Mechanics) - 25V 4.7uF X5R ±10% 0805 Multilayer Ceramic Capacitors MLCC - SMD/SMT ROHS -> (none)
- C13, C21, C24: value CL21A106KAYNNNE (Samsung Electro-Mechanics) - X5R 25V ±10% 10uF 0805 Multilayer Ceramic Capacitors MLCC - SMD/SMT ROHS -> (none)
- C19, C20, C6: value CL10A105KB8NNNC (Samsung Electro-Mechanics) - 50V 1uF X5R ±10% 0603 Multilayer Ceramic Capacitors MLCC - SMD/SMT ROHS -> (none)
- C23, C26: value 0603B103K500NT (FH(Guangdong Fenghua Advanced Tech)) - 50V 10nF X7R ±10% 0603 Multilayer Ceramic Capacitors MLCC - SMD/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 -> (none)
- C4: value CL31A226KPHNNNE (Samsung Electro-Mechanics) - 10V 22uF X5R ±10% 1206 Multilayer Ceramic Capacitors MLCC - SMD/SMT ROHS -> (none)
- D1: value BZT52C3V6 (SMC(Sangdest Microelectronicstronic (Nanjing))) - 5μA@1V 90Ω Single 3.6V~3.8V 350mW 3.4V SOD-123 Zener Diode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 -> BZT52C3V6 (SMC(Sangdest Microelectronicstronic (Nanjing))) - 5?A@1V 90? Single 3.6V~3.8V 350mW 3.4V SOD-123 Zener Diode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
- L1: value MPL2012S3R3MHT (Sunlord) - 900mA 3.3uH ±20% 190mΩ 0805 Inductors (SMD) ROHS -> (none)
- R1: value RTT25R050FTE (RALEC) - ±1% 1W Thick Film Resistors 200V ±500ppm/℃ -55℃~+155℃ 0.05Ω 2512 Chip Resistor - Surface Mount R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 -> (none)
- R10, R9: value 0603WAF4701T5E (UNI-ROYAL(Uniroyal Elec)) - ±1% 1/10W Thick Film Resistors 75V ±100ppm/℃ -55℃~+155℃ 4.7kΩ 0603 Chip Res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 -> (none)
- R11: value 0603WAF5603T5E (UNI-ROYAL(Uniroyal Elec)) - ±1% 1/10W Thick Film Resistors 75V ±100ppm/℃ -55℃~+155℃ 560kΩ 0603 Chip Res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 -> (none)
- R12: renamed from R16; value 0603WAF3002T5E (UNI-ROYAL(Uniroyal Elec)) - ±1% 1/10W Thick Film Resistors 75V ±100ppm/℃ -55℃~+155℃ 30kΩ 0603 Chip Resi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 -> (none)
- R13: renamed from R17; value 0603WAF3002T5E (UNI-ROYAL(Uniroyal Elec)) - ±1% 1/10W Thick Film Resistors 75V ±100ppm/℃ -55℃~+155℃ 30kΩ 0603 Chip Resi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 -> (none)
- R2, R3, R8: value 0603WAF1002T5E (UNI-ROYAL(Uniroyal Elec)) - ±1% 1/10W Thick Film Resistors 75V ±100ppm/℃ -55℃~+155℃ 10kΩ 0603 Chip Resi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 -> (none)
- R4, R5: value 0603WAF2003T5E (UNI-ROYAL(Uniroyal Elec)) - ±1% 1/10W Thick Film Resistors 75V ±100ppm/℃ -55℃~+155℃ 200kΩ 0603 Chip Res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 -> (none)
- R6: value 0603WAF6802T5E (UNI-ROYAL(Uniroyal Elec)) - ±1% 1/10W Thick Film Resistors 75V ±100ppm/℃ -55℃~+155℃ 68kΩ 0603 Chip Resi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 -> (none)
- R7: value 0603WAF1502T5E (UNI-ROYAL(Uniroyal Elec)) - ±1% 1/10W Thick Film Resistors 75V ±100ppm/℃ -55℃~+155℃ 15kΩ 0603 Chip Resi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 -> (none)
- TP1: value RCU-0C (TE Connectivity) - anon_link_0 -> RCU-0C (TE Connectivity) - vbatt
- moved D1 16.4 mm to (126.0, 78.0), turned to 180 degrees
- moved C1 9.22 mm to (130.0, 57.0)
- moved R5 6.08 mm to (127.0, 56.0), turned to 0 degrees
- moved D2 6.02 mm to (126.0, 94.0), turned to 180 degrees
- moved D3 6.02 mm to (126.0, 96.0), turned to 180 degrees
- moved D4 6.02 mm to (126.0, 98.0), turned to 180 degrees
- moved D5 6.02 mm to (126.0, 100.0), turned to 180 degrees
- moved R3 5.00 mm to (127.0, 58.0)
- moved R2 4.61 mm to (127.0, 64.0)
- moved TP3 4.13 mm to (140.0, 78.0)
- moved U1 4.12 mm to (129.0, 61.0)
- moved R4 3.91 mm to (127.0, 66.0), turned to 0 degrees
- moved R1 3.61 mm to (123.0, 61.0), turned to -90 degrees
- moved TP1 2.24 mm to (117.0, 64.0)
- moved TP2 2.00 mm to (117.0, 68.0)
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Connections:
- net expander.io.tof_xshut_1 renamed tof.xshut.1
- net isense.amp.(adapter)r2.b.src renamed isense.amp.amp.inp
- net isense.amp.r1.b renamed isense.amp.amp.inn
- net lcd.device.c2p renamed lcd.c2_cap.pos
- net lcd.vcc_cap1.pwr renamed lcd.vcc_cap2.pos
- net mcu.ic.chip_pu renamed mcu.en_pull.output
- net mcu.uart0.uart.tx renamed mcu.ic.uart0.rx
- net motor_driver1.ic.vcp renamed motor_driver1.vcp_cap.pos
- net motor_driver2.vcp_cap.pos renamed motor_driver2.ic.vcp
- net reg_3v3.fb.center renamed reg_3v3.ic.fb
- net spk_drv.inn_res.a renamed spk_drv.inn_cap.pos
- net tof.xshut.2 renamed expander.io.tof_xshut_2
- D2 pad 1: led[0].res.a -> led_res.a.0
- D2 pad 2: expander.io.led0 -> v3v3
- D3 pad 1: led[1].res.a -> led_res.a.1
- D3 pad 2: expander.io.led1 -> v3v3
- D4 pad 1: led[2].res.a -> led_res.a.2
- D4 pad 2: expander.io.led2 -> v3v3
- D5 pad 1: led[3].package.k -> led_res.a.3
- D5 pad 2: expander.io.led3 -> v3v3
- TP1 pad 1: batt.pins.2 -> vbatt
- U5 pad 4: expander.io.led0 -> led_res.b.0
- U5 pad 5: expander.io.led1 -> leds.signals.1
- U5 pad 6: expander.io.led2 -> leds.signals.2
- U5 pad 7: expander.io.led3 -> expander.io.led_3
Routing:
- net gnd: track 70.4 -> 433.2 mm, vias 21 -> 42
- net vbatt: track 0.00 -> 202.3 mm
- net v3v3: track 16.5 -> 178.9 mm, vias 2 -> 0
- net led_res.b.0: track 0.00 -> 4.89 mm
- net expander.io.led_3: track 0.00 -> 4.70 mm
- net leds.signals.1: track 0.00 -> 4.69 mm
- net leds.signals.2: track 0.00 -> 4.50 mm
- net expander.io.led0: track 4.13 -> 0.00 mm
- net led_res.a.3: track 0.00 -> 4.11 mm
- net led_res.a.0: track 0.00 -> 4.11 mm
- net expander.io.led3: track 3.90 -> 0.00 mm
- net expander.io.led1: track 3.83 -> 0.00 mm
- net batt.pins.2: track 14.2 -> 10.5 mm
- net mcu.adc.isense: track 3.25 -> 6.86 mm
- net led_res.a.2: track 0.00 -> 3.61 mm
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
Commit message: coarse layout doneish?
Parts:
- moved TP3 14.1 mm to (126.0, 76.0)
- moved D1 5.00 mm to (126.0, 73.0)
- moved R10 4.00 mm to (141.0, 83.0)
- moved R9 4.00 mm to (141.0, 85.0)
- moved TP4 4.00 mm to (137.0, 85.0)
- moved TP5 4.00 mm to (137.0, 83.0)
- moved C3 3.61 mm to (150.0, 76.0), turned to 0 degrees
- moved L1 2.24 mm to (145.0, 76.0), turned to 0 degrees
- moved R6 0.50 mm to (150.0, 74.0)
- moved R7 0.50 mm to (150.0, 72.0)
- turned R4 to 180 degrees
- turned R5 to 180 degrees
Routing:
- net v3v3: track 178.9 -> 204.4 mm, vias 0 -> 2
- net spk_chain_1.b: track 0.00 -> 11.4 mm, vias 0 -> 1
- net spk_chain_1.a: track 0.00 -> 9.43 mm, vias 0 -> 1
- net isense.amp.amp.inn: track 2.07 -> 5.33 mm
- net i2c_chain_0.scl: track 9.34 -> 7.58 mm
- net mcu.adc.isense: track 6.86 -> 5.40 mm
- net i2c_chain_0.sda: track 8.82 -> 7.37 mm
- net isense.amp.amp.inp: track 4.07 -> 5.33 mm
- net gnd: track 433.2 -> 434.3 mm, vias 42 -> 45
- net reg_3v3.power_path.switch: track 3.04 -> 2.08 mm
- net reg_3v3.ic.fb: track 5.56 -> 5.06 mm

Commit message: cleanup
Routing:
- net i2c_chain_0.scl: track 7.58 -> 112.6 mm, vias 0 -> 2
- net i2c_chain_0.sda: track 7.37 -> 102.1 mm, vias 0 -> 3
- net mcu.gpio.ledArray: track 0.00 -> 80.2 mm, vias 0 -> 2
- net spk_chain_0: track 2.07 -> 81.6 mm, vias 0 -> 4
- net lcd.spi.sck: track 0.00 -> 73.4 mm, vias 0 -> 2
- net mcu.gpio.motor_1b2: track 0.00 -> 69.9 mm, vias 0 -> 2
- net lcd.spi.mosi: track 0.00 -> 68.3 mm, vias 0 -> 4
- net mcu.gpio.lcd_dc: track 0.00 -> 67.8 mm, vias 0 -> 4
- net mcu.gpio.motor_2b1: track 0.00 -> 65.1 mm, vias 0 -> 2
- net mcu.gpio.motor_2b2: track 0.00 -> 64.8 mm, vias 0 -> 2
- net mcu.gpio.lcd_cs: track 0.00 -> 64.1 mm, vias 0 -> 4
- net mcu.gpio.motor_1b1: track 0.00 -> 63.0 mm, vias 0 -> 2
- net mcu.adc.isense: track 5.40 -> 67.8 mm, vias 0 -> 2
- net mcu.gpio.lcd_reset: track 0.00 -> 58.5 mm, vias 0 -> 2
- net mcu.gpio.motor_2a2: track 0.00 -> 53.2 mm, vias 0 -> 2
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
Commit message: Update RobotDriver2_Blimp.kicad_pcb
Other:
- board text added: "<RX"
- board text added: "TX>"
- board text removed: "RX>"
- board text removed: "TX<"
Changed lines of the file:
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@@
     (effects (font (size 1.5 1) (thickness 0.1524)))
   )
-  (gr_text "⏚" (at 106.5 57) (layer "F.SilkS")
+  (gr_text "⏚" (at 106.5 57.5) (layer "F.SilkS")
     (effects (font (size 1.5 1) (thickness 0.1524)))
   )
@@
     (effects (font (size 1.5 1) (thickness 0.15)) (justify left))
   )
-  (gr_text "+" (at 106.5 59.5) (layer "F.SilkS")
+  (gr_text "+" (at 106.5 60) (layer "F.SilkS")
     (effects (font (size 1.5 1) (thickness 0.1524)))
   )
@@
     (effects (font (size 1.5 1) (thickness 0.15)) (justify left))
   )
-  (gr_text "⎍" (at 106.5 62) (layer "F.SilkS")
+  (gr_text "⎍" (at 106.5 62.5) (layer "F.SilkS")
     (effects (font (size 1.5 1) (thickness 0.1524)))
   )
-  (gr_text "RX>" (at 98.842857 59.589999) (layer "F.SilkS")
+  (gr_text "<RX" (at 98.842857 59.589999) (layer "F.SilkS")
     (effects (font (size 1 0.8) (thickness 0.1524)))
   )
@@
     (effects (font (size 1.5 1) (thickness 0.15)) (justify left))
   )
-  (gr_text "TX<" (at 98.937295 62) (layer "F.SilkS")
+  (gr_text "TX>" (at 98.937295 62) (layer "F.SilkS")
     (effects (font (size 1 0.8) (thickness 0.154)))
   )

Commit message: gerbs
Parts:
- C1, C10, C12, C14, C15, C16, C17, C5, C7, C8: value (none) -> C14663
- C11, C18, C2, C22, C25, C3, C9: value (none) -> C1779
- C13, C21, C24: value (none) -> C15850
- C19, C20, C6: value (none) -> C15849
- C23, C26: value (none) -> C57112
- C4: value (none) -> C5672
- D1: value BZT52C3V6 (SMC(Sangdest Microelectronicstronic (Nanjing))) - 5?A@1V 90? Single 3.6V~3.8V 350mW 3.4V SOD-123 Zener Diode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 -> C499796
- D10, D6, D7, D8, D9: value WS2812B (Worldsemi) -> C2920042
- D2, D3, D4, D5: value KT-0603R (Hubei KENTO Elec) - Red 615~630nm 1.9~2.2V 0603 Light Emitting Diodes (LED) RoHS -> C2286
- J1, J10, J11, J12, J7, J9: value B2B-PH-K (JST) -> (none)
- J13: value PinHeader2.54 1x3 (Generic) -> (none)
- J2: value PinHeader2.54 1x4 (Generic) -> (none)
- J3, J4, J5: value B6B-PH-K (JST) -> (none)
- J6: value FH12-15S-0.5SH (Hirose) -> (none)
- J8: value B3B-PH-K (JST) -> (none)
- L1: value (none) -> C98331
- R1: value (none) -> C305115
- R10, R9: value (none) -> C23162
- R11: value (none) -> C23203
- R12, R13: value (none) -> C22984
- R2, R3, R8: value (none) -> C25804
- R4, R5: value (none) -> C25811
- R6: value (none) -> C23231
- R7: value (none) -> C22809
- RN1: value (none) -> C20197
- SW1: value 5.1mm switch -> C318884
- TP1: value RCU-0C (TE Connectivity) - vbatt -> (none)
- TP2: value RCU-0C (TE Connectivity) - gnd -> (none)
- TP3: value RCU-0C (TE Connectivity) - v3v3 -> (none)
- TP4: value RCU-0C (TE Connectivity) - i2c_chain_0.scl -> (none)
- TP5: value RCU-0C (TE Connectivity) - i2c_tp.anon_link_1 -> (none)
- TP6: value RCU-0C (TE Connectivity) - spk_chain_0 -> (none)
- U1: value LMV321 (Texas Instruments) -> C7972
- U10: value Duck -> (none)
- U11: value LeadFree -> (none)
- U12: value IdDots4 -> (none)
- U2: value AP3418 (Diodes Incorporated) -> C500769
- U3: value ESP32-WROOM-32 (Espressif Systems) -> C701342
- U4: value LSM6DS3TR-C (STMicroelectronics) -> C967633
- U5: value PCF8574AT (NXP) -> C86832
- U6: value TPA2005D1 (Texas Instruments) -> C27396
- U7, U8: value DRV8833PWP (Texas Instruments) -> C50506
- U9: value Lemur -> (none)
Connections:
- net expander.io.led_3 renamed leds.signals.3
- net expander.io.tof_xshut_2 renamed tof.xshut.2
- net isense.amp.amp.inn renamed isense.amp.(adapter)rf.b.src
- net isense.amp.amp.inp renamed isense.amp.(adapter)r2.b.src
- net lcd.c1_cap.neg renamed lcd.device.c1n
- net lcd.device.c1p renamed lcd.c1_cap.pos
- net lcd.device.vcomh renamed lcd.vcomh_cap.pos
- net lcd.vcc_cap2.pos renamed lcd.vcc_cap2.pwr
- net leds.signals.1 renamed expander.io.led_1
- net leds.signals.2 renamed expander.io.led_2
- net mcu.en_pull.output renamed mcu.ic.chip_pu
- net mcu.ic.uart0.rx renamed mcu.uart0.uart.tx
- net mcu.prog.a renamed mcu.ic.io0
- net motor_driver1.ic.vint renamed motor_driver1.vint_cap.pwr
- net motor_driver1.vcp_cap.pos renamed motor_driver1.ic.vcp
- net reg_3v3.ic.fb renamed reg_3v3.fb.output
- net reg_3v3.power_path.switch renamed reg_3v3.ic.sw
- net spk_drv.ic.inn renamed spk_drv.(adapter)inn_res.b.src
- net tof.xshut.1 renamed expander.io.tof_xshut_1
- net ws2812bArray.led[2].din renamed ws2812bArray.led[1].dout
- net ws2812bArray.led[4].din renamed ws2812bArray.led[3].dout
