File: examples/test_bldc/BldcDriverBoard.kicad_pcb (KiCad board)
At the start: 2 copper layers, 78 x 57 mm, 81 parts, among them sw1 5.1mm switch, sw2 5.1mm switch, sw3 5.1mm switch

Commit message: doneish layout
Parts:
- moved lemur 86.6 mm to (127.0, 58.0)
- moved duck 81.9 mm to (132.0, 58.0)
- moved leadfree 75.4 mm to (123.0, 106.0)
- moved id 74.0 mm to (116.0, 106.0)
- moved i2c_tp.tp_scl 33.3 mm to (113.0, 79.0), turned to 90 degrees
- moved i2c_pull.scl_res 31.3 mm to (113.0, 83.0), turned to 90 degrees
- moved mcu.crystal.package 30.0 mm to (141.0, 87.0), turned to -90 degrees
- moved i2c_pull.sda_res 29.4 mm to (110.0, 83.0), turned to 90 degrees
- moved mcu.swd 28.0 mm to (141.0, 58.0)
- moved i2c 27.8 mm to (111.5, 67.0), turned to -90 degrees
- moved mcu.pwr_cap[0] 25.6 mm to (133.0, 82.0), turned to -90 degrees
- moved i2c_tp.tp_sda 25.2 mm to (110.0, 79.0), turned to 90 degrees
- moved mcu.vdda_cap_1 24.4 mm to (148.0, 82.0), turned to -90 degrees
- moved mcu.crystal.cap_a 24.0 mm to (141.0, 84.0), turned to 0 degrees
- moved mcu.pwr_cap[3] 23.3 mm to (135.0, 82.0), turned to -90 degrees
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Connections:
- net bldc_drv.(adapter)ic.v3p3.src renamed bldc_drv.nsleep_default.out
- net bldc_drv.cp_cap.pos renamed bldc_drv.ic.cph
- net bldc_drv.outs.1 renamed bldc.pins.1
- net conv.(adapter)in_high_switch.output.dst renamed conv.in_low_diode.cathode
- net conv.(adapter)out_high_diode.anode.dst renamed conv.(adapter)out_high_diode.anode.src
- net conv.in_high_switch.(adapter)pull.b.dst renamed conv.in_high_switch.(adapter)pre.drain.dst
- net curr_amp[2].(adapter)r1.b.src renamed curr_amp[2].(adapter)r1.b.dst
- net curr_amp[3].(adapter)r2.a.dst renamed curr_amp[3].(adapter)r2.a.src
- net mcu.ic.swd.reset renamed mcu.swd.swd.reset
- net mcu.swd.swd.swclk renamed mcu.ic.swd.swclk
- net mcu.swd.swd.swo renamed mcu.ic.swd.swo
- net pd.cc.cc2 renamed usb.cc.cc2
- net usb.cc.cc1 renamed pd.cc.cc1
- net usb.usb.dm renamed usb_esd.usb.dm
- net usb_esd.usb.dp renamed usb.usb.dp
- bldc_drv.ic pad 22: bldc_drv.ens.3 -> mcu.gpio.bldc_en_3
- bldc_drv.ic pad 26: mcu.gpio.bldc_en_1 -> bldc_drv.ens.1
- i2c pad 3: i2c.i2c.sda -> i2c_tp.io.sda
- i2c pad 4: i2c_tp.io.scl -> i2c.i2c.scl
- i2c_pull.scl_res pad 2: i2c_tp.io.scl -> i2c.i2c.scl
- i2c_pull.sda_res pad 2: i2c.i2c.sda -> i2c_tp.io.sda
- i2c_tp.tp_scl pad 1: i2c_tp.io.scl -> i2c.i2c.scl
- i2c_tp.tp_sda pad 1: i2c.i2c.sda -> i2c_tp.io.sda
- mcu.ic pad 11: mcu.adc.curr_1 -> mcu.gpio.buck_pwm
- mcu.ic pad 12: mcu.adc.curr_3 -> mcu.gpio.boost_pwm
- mcu.ic pad 13: mcu.adc.curr_2 -> mcu.adc.conv_sense
- mcu.ic pad 14: mcu.adc.conv_sense -> mcu.adc.curr_2
- mcu.ic pad 15: mcu.gpio.boost_pwm -> mcu.adc.curr_1
- mcu.ic pad 16: mcu.gpio.bldc_reset -> mcu.adc.curr_3
- mcu.ic pad 17: mcu.gpio.buck_pwm -> bldc_drv.ins.1
- mcu.ic pad 18: mcu.gpio.sw3 -> bldc_drv.ens.1
- mcu.ic pad 19: mcu.gpio.bldc_fault -> mcu.gpio.bldc_in_2
- mcu.ic pad 20: mcu.gpio.sw1 -> mcu.gpio.bldc_en_2
- mcu.ic pad 21: i2c_tp.io.scl -> bldc_drv.ins.3
- mcu.ic pad 22: i2c.i2c.sda -> mcu.gpio.bldc_en_3
- mcu.ic pad 25: mcu.gpio.sw2 -> mcu.gpio.bldc_fault
- mcu.ic pad 26: mcu.gpio.pd_int -> mcu.gpio.bldc_reset
- mcu.ic pad 27: mcu.gpio.bldc_en_2 -> mcu.gpio.sw3
- mcu.ic pad 28: mcu.gpio.bldc_en_1 -> mcu.gpio.sw1
- mcu.ic pad 29: bldc_drv.ens.3 -> mcu.gpio.sw2
- mcu.ic pad 30: mcu.gpio.bldc_in_2 -> (no net)
- mcu.ic pad 31: bldc_drv.ins.1 -> (no net)
- mcu.ic pad 38: bldc_drv.ins.3 -> (no net)
- mcu.ic pad 42: (no net) -> i2c.i2c.scl
- mcu.ic pad 43: (no net) -> i2c_tp.io.sda
- mcu.ic pad 45: (no net) -> mcu.gpio.pd_int
- pd.ic pad 6: i2c_tp.io.scl -> i2c.i2c.scl
- pd.ic pad 7: i2c.i2c.sda -> i2c_tp.io.sda
Routing:
- net v3v3: track 81.6 -> 279.3 mm, vias 8 -> 12
- net vusb: track 94.3 -> 230.9 mm, vias 11 -> 13
- net mag.pins.2: track 0.00 -> 57.3 mm, vias 0 -> 3
- net mcu.adc.curr_2: track 3.33 -> 45.5 mm
- net i2c_tp.io.sda: track 0.00 -> 41.6 mm, vias 0 -> 3
- net mcu.adc.curr_3: track 3.33 -> 43.3 mm, vias 0 -> 2
- net i2c.i2c.scl: track 0.00 -> 37.7 mm, vias 0 -> 3
- net mcu.adc.conv_sense: track 2.35 -> 39.4 mm
- net mcu.gpio.boost_pwm: track 0.00 -> 35.6 mm
- net mcu.adc.curr_1: track 3.33 -> 38.3 mm
- net usb_esd.usb.dm: track 9.21 -> 37.0 mm
- net mcu.swd.swd.reset: track 0.00 -> 26.0 mm, vias 0 -> 2
- net usb.usb.dp: track 11.3 -> 36.3 mm
- net mcu.ic.swd.swo: track 0.00 -> 19.6 mm, vias 0 -> 2
- net mcu.gpio.buck_pwm: track 0.00 -> 19.0 mm
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- added copper zone on B.Cu, net gnd
- added copper zone on F.Cu, net gnd
Other:
- outline, holes or cut-outs redrawn
- board text added: "EDG BLDC / Buck-Boost Oct '22"

Commit message: wip neopixel brokenish
Parts:
- removed sw2, sw3: 5.1mm switch, Button_Switch_SMD:SW_SPST_SKQG_WithoutStem
- added reg_5v.ic: LD1117S50TR (STMicroelectronics), Package_TO_SOT_SMD:SOT-223-3_TabPin2, F.Cu at (133.0, 100.0)
- added reg_5v.in_cap: , Capacitor_SMD:C_0603_1608Metric, F.Cu at (133.0, 105.0)
- added reg_5v.out_cap: , Capacitor_SMD:C_1206_3216Metric, F.Cu at (133.0, 95.0)
- added rgb: SK6812MINI-E (Opsco Optoelectronics), edg:LED_SK6812MINI-E, F.Cu at (124.0, 90.0)
- added tp_5v: RCT-0C (TE Connectivity) - v5, edg:TestPoint_TE_RCT_0805, F.Cu at (133.0, 92.0)
- i2c_tp.tp_scl: value RCT-0C (TE Connectivity) - anon_chain_5_0.scl -> RCT-0C (TE Connectivity) - anon_chain_4_0.scl
- sw1: value 5.1mm switch -> PG151101S11 (Kailh); footprint Button_Switch_SMD:SW_SPST_SKQG_WithoutStem -> Switch_Keyboard_Hotswap_Kailh:SW_Hotswap_Kailh_MX
- moved sw1 70.5 mm to (124.0, 84.0)
- moved conv.power_path.in_cap.c[0] 1.00 mm to (140.0, 103.0)
Connections:
- net bldc.phases.3 renamed bldc_drv.outs.3
- net bldc_drv.cp_cap.neg renamed bldc_drv.ic.cpl
- net bldc_drv.ens.1 renamed mcu.gpio.bldc_en_1
- net bldc_drv.ic.cph renamed bldc_drv.cp_cap.pos
- net bldc_drv.ins.1 renamed mcu.gpio.bldc_in_1
- net bldc_drv.ins.3 renamed mcu.gpio.bldc_in_3
- net bldc_drv.nsleep_default.out renamed bldc_drv.v3p3_cap.pwr
- net bldc_drv.outs.2 renamed bldc.pins.2
- net conv.(adapter)out_high_diode.anode.src renamed conv.out_low_switch.drain
- net conv.in_high_switch.(adapter)pre.drain.dst renamed conv.in_high_switch.(adapter)drv.gate.dst
- net curr_amp[1].(adapter)r1.b.dst renamed curr_amp[1].(adapter)r2.a.dst
- net curr_amp[2].(adapter)r1.b.dst renamed curr_amp[2].(adapter)r1.b.src
- net curr_amp[3].(adapter)r2.a.src renamed curr_amp[3].r2.a
- net i2c.i2c.scl renamed i2c_pull.i2c.scl
- net i2c_tp.io.sda renamed pd.i2c.sda
- net mcu.gpio.bldc_en_3 renamed bldc_drv.ens.3
- net mcu.gpio.bldc_in_2 renamed bldc_drv.ins.2
- net mcu.ic.osc.xtal_out renamed mcu.crystal.crystal.b
- net pd.cc.cc1 renamed usb.cc.cc1
- net usb.usb.dp renamed usb_esd.usb.dp
- net usb_esd.usb.dm renamed usb.usb.dm
- mcu.ic pad 27: mcu.gpio.sw3 -> (no net)
- mcu.ic pad 28: mcu.gpio.sw1 -> (no net)
- mcu.ic pad 29: mcu.gpio.sw2 -> (no net)
- mcu.ic pad 40: (no net) -> mcu.gpio.sw1
- mcu.ic pad 41: (no net) -> mcu.gpio.rgb
Routing:
- net v5: track 0.00 -> 32.0 mm, vias 0 -> 1
- net mcu.gpio.rgb: track 0.00 -> 28.6 mm, vias 0 -> 1
- net vusb: track 230.9 -> 244.6 mm
- net mcu.gpio.sw1: track 0.00 -> 11.8 mm, vias 0 -> 1
- net v3v3: track 279.3 -> 271.5 mm, vias 12 -> 11
- net gnd: track 215.9 -> 219.9 mm, vias 42 -> 43
