File: electronics_abstract_parts/resources/opamp_amplifier.kicad_sch (KiCad schematic)
At the start: 3 parts

Commit message: working opamp amplifier I think, maybe
Parts:
- r1: value #Resistor(top_resistance) -> ~
- r2: value #Resistor(bottom_resistance) -> ~
Changed lines of the file:
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@@
       (effects (font (size 1.27 1.27)) (justify left))
     )
-    (property "Value" "#Resistor(bottom_resistance)" (id 1) (at 137.16 109.2199 0)
+    (property "Value" "~" (id 1) (at 137.16 109.2199 0)
       (effects (font (size 1.27 1.27)) (justify left))
     )
@@
       (effects (font (size 1.27 1.27)) (justify left))
     )
-    (property "Value" "#Resistor(top_resistance)" (id 1) (at 137.16 96.5199 0)
+    (property "Value" "~" (id 1) (at 137.16 96.5199 0)
       (effects (font (size 1.27 1.27)) (justify left))
     )
@@
     )
     (path "/8191dcd1-5cad-46b4-ac40-399ad1332adc"
-      (reference "r1") (unit 1) (value "#Resistor(top_resistance)") (footprint "")
+      (reference "r1") (unit 1) (value "~") (footprint "")
     )
     (path "/6b0d5df9-b2da-44e2-8a2b-ae179529fe85"
-      (reference "r2") (unit 1) (value "#Resistor(bottom_resistance)") (footprint "")
+      (reference "r2") (unit 1) (value "~") (footprint "")
     )
   )

Commit message: Update opamp_amplifier.kicad_sch
Parts:
- removed r1: ~, symbol Device:R
- added r2: ~, symbol Device:R
- renumbered r2 to r1
Connections:
- net output: now also r1.1
- net ref: now also r2.2; no longer r1.2
- net at amp.2 (-): now also r1.2, r2.1; no longer r1.1
Other:
- moved on the sheet: r1
Changed lines of the file:
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@@
     )
   )
-  (symbol (lib_id "Device:R") (at 134.62 107.95 0) (unit 1)
+  (symbol (lib_id "Device:R") (at 134.62 95.25 0) (unit 1)
     (in_bom yes) (on_board yes)
-    (property "Reference" "r2" (id 0) (at 137.16 106.6799 0)
-      (effects (font (size 1.27 1.27)) (justify left))
-    )
-    (property "Value" "~" (id 1) (at 137.16 109.2199 0)
-      (effects (font (size 1.27 1.27)) (justify left))
-    )
-    (property "Footprint" "" (id 2) (at 132.842 107.95 90)
-      (effects (font (size 1.27 1.27)) hide)
-    )
-    (property "Datasheet" "~" (id 3) (at 134.62 107.95 0)
-      (effects (font (size 1.27 1.27)) hide)
-    )
-    (pin "1")
-    (pin "2")
-  )
-  (symbol (lib_name "R_1") (lib_id "Device:R") (at 134.62 95.25 0) (unit 1)
-    (in_bom yes) (on_board yes) (fields_autoplaced)
     (property "Reference" "r1" (id 0) (at 137.16 93.9799 0)
       (effects (font (size 1.27 1.27)) (justify left))
@@
     (pin "5")
   )
+  (symbol (lib_id "Device:R") (at 134.62 107.95 0) (unit 1)
+    (in_bom yes) (on_board yes)
+    (property "Reference" "r2" (id 0) (at 137.16 106.6799 0)
+      (effects (font (size 1.27 1.27)) (justify left))
+    )
+    (property "Value" "~" (id 1) (at 137.16 109.2199 0)
+      (effects (font (size 1.27 1.27)) (justify left))
+    )
+    (property "Footprint" "" (id 2) (at 132.842 107.95 90)
+      (effects (font (size 1.27 1.27)) hide)
+    )
+    (property "Datasheet" "~" (id 3) (at 134.62 107.95 0)
+      (effects (font (size 1.27 1.27)) hide)
+    )
+    (pin "1")
+    (pin "2")
+  )
   (sheet_instances
     (path "/" (page "1"))
@@
       (reference "amp") (unit 1) (value "~") (footprint "")
     )
-    (path "/8191dcd1-5cad-46b4-ac40-399ad1332adc"
+    (path "/6b0d5df9-b2da-44e2-8a2b-ae179529fe85"
       (reference "r1") (unit 1) (value "~") (footprint "")
     )
-    (path "/6b0d5df9-b2da-44e2-8a2b-ae179529fe85"
+    (path "/bc85c8b6-5c82-4cf8-ad22-158c3a6558a0"
       (reference "r2") (unit 1) (value "~") (footprint "")
     )
