File: electronics_abstract_parts/resources/OpampFollower.kicad_sch (KiCad schematic)
At the start: 1 part

Commit message: wip
Parts:
- added forced: #ForcedAnalogSignal(output_voltage), symbol edg_importable:Adapter
- amp: value ~ -> (none); Spice_Netlist_Enabled Y -> (none); Spice_Primitive X -> (none)
Connections:
- net output: now also forced.2; no longer amp.3
- new net: amp.3, forced.1
Changed lines of the file:
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@@
-(kicad_sch (version 20211123) (generator eeschema)
+(kicad_sch (version 20230121) (generator eeschema)
   (paper "A4")
   (wire (pts (xy 116.84 91.44) (xy 119.38 91.44))
-    (stroke (width 0) (type default) (color 0 0 0 0))
+    (stroke (width 0) (type default))
   )
   (wire (pts (xy 116.84 91.44) (xy 116.84 100.33))
-    (stroke (width 0) (type default) (color 0 0 0 0))
+    (stroke (width 0) (type default))
   )
-  (wire (pts (xy 134.62 100.33) (xy 134.62 88.9))
-    (stroke (width 0) (type default) (color 0 0 0 0))
+  (wire (pts (xy 139.7 100.33) (xy 139.7 88.9))
+    (stroke (width 0) (type default))
   )
-  (wire (pts (xy 116.84 100.33) (xy 134.62 100.33))
-    (stroke (width 0) (type default) (color 0 0 0 0))
+  (wire (pts (xy 116.84 100.33) (xy 139.7 100.33))
+    (stroke (width 0) (type default))
   )
   (global_label "pwr" (shape input) (at 124.46 81.28 180) (fields_autoplaced)
     (effects (font (size 1.27 1.27)) (justify right))
-    (property "Intersheet References" "${INTERSHEET_REFS}" (id 0) (at 118.7812 81.3594 0)
+    (property "Intersheetrefs" "${INTERSHEET_REFS}" (at 118.7812 81.3594 0)
       (effects (font (size 1.27 1.27)) (justify right) hide)
     )
@@
   (global_label "input" (shape input) (at 119.38 86.36 180) (fields_autoplaced)
     (effects (font (size 1.27 1.27)) (justify right))
-    (property "Intersheet References" "${INTERSHEET_REFS}" (id 0) (at 112.1893 86.2806 0)
+    (property "Intersheetrefs" "${INTERSHEET_REFS}" (at 112.1893 86.2806 0)
       (effects (font (size 1.27 1.27)) (justify right) hide)
     )
   )
-  (global_label "output" (shape output) (at 134.62 88.9 0) (fields_autoplaced)
+  (global_label "output" (shape output) (at 139.7 88.9 0) (fields_autoplaced)
     (effects (font (size 1.27 1.27)) (justify left))
-    (property "Intersheet References" "${INTERSHEET_REFS}" (id 0) (at 143.0807 88.8206 0)
+    (property "Intersheetrefs" "${INTERSHEET_REFS}" (at 148.6532 88.9 0)
       (effects (font (size 1.27 1.27)) (justify left) hide)
     )
@@
   (global_label "gnd" (shape input) (at 124.46 96.52 180) (fields_autoplaced)
     (effects (font (size 1.27 1.27)) (justify right))
-    (property "Intersheet References" "${INTERSHEET_REFS}" (id 0) (at 118.5998 96.5994 0)
+    (property "Intersheetrefs" "${INTERSHEET_REFS}" (at 118.5998 96.5994 0)
       (effects (font (size 1.27 1.27)) (justify right) hide)
     )
   )
-  (symbol (lib_id "Simulation_SPICE:OPAMP") (at 127 88.9 0) (unit 1)
-    (in_bom yes) (on_board yes)
-    (property "Reference" "amp" (id 0) (at 127 83.82 0))
-    (property "Value" "~" (id 1) (at 137.16 86.741 0))
-    (property "Footprint" "" (id 2) (at 127 88.9 0)
+  (symbol (lib_id "edg_importable:Adapter") (at 137.16 88.9 0) (unit 1)
+    (in_bom yes) (on_board yes) (dnp no)
+    (property "Reference" "forced" (at 137.16 83.82 0)
+      (effects (font (size 1.27 1.27)))
+    )
+    (property "Value" "#ForcedAnalogSignal(output_voltage)" (at 151.13 86.36 0)
+      (effects (font (size 1.27 1.27)))
+    )
+    (property "Footprint" "" (at 137.16 88.9 0)
       (effects (font (size 1.27 1.27)) hide)
     )
-    (property "Datasheet" "~" (id 3) (at 127 88.9 0)
+    (property "Datasheet" "~" (at 137.16 88.9 0)
       (effects (font (size 1.27 1.27)) hide)
     )
-    (property "Spice_Netlist_Enabled" "Y" (id 4) (at 127 88.9 0)
-      (effects (font (size 1.27 1.27)) (justify left) hide)
+    (pin "1")
+    (pin "2")
+    (instances
+      (project "OpampFollower"
+        (path "/b55f6c44-5d5d-4524-bb86-893662f64598"
+          (reference "forced") (unit 1)
+        )
+      )
     )
-    (property "Spice_Primitive" "X" (id 5) (at 127 88.9 0)
-      (effects (font (size 1.27 1.27)) (justify left) hide)
+  )
+  (symbol (lib_id "Simulation_SPICE:OPAMP") (at 127 88.9 0) (unit 1)
+    (in_bom yes) (on_board yes) (dnp no)
+    (property "Reference" "amp" (at 127 83.82 0)
+      (effects (font (size 1.27 1.27)))
+    )
+    (property "Value" "" (at 137.16 86.741 0)
+      (effects (font (size 1.27 1.27)))
+    )
+    (property "Footprint" "" (at 127 88.9 0)
+      (effects (font (size 1.27 1.27)) hide)
+    )
+    (property "Datasheet" "~" (at 127 88.9 0)
+      (effects (font (size 1.27 1.27)) hide)
     )
     (pin "1")
@@
     (pin "4")
     (pin "5")
+    (instances
+      (project "OpampFollower"
+        (path "/b55f6c44-5d5d-4524-bb86-893662f64598"
+          (reference "amp") (unit 1)
+        )
+      )
+    )
   )
   (sheet_instances
     (path "/" (page "1"))
   )
-  (symbol_instances
-    (path "/95a16bc8-5b0b-4a19-9511-bfbdba477838"
-      (reference "amp") (unit 1) (value "~") (footprint "")
-    )
-  )
 )

Commit message: tighten isense signal output
Parts:
- amp: value (none) -> ~
- forced: value #ForcedAnalogSignal(output_voltage) -> ~
Changed lines of the file:
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@@
   (symbol (lib_id "edg_importable:Adapter") (at 137.16 88.9 0) (unit 1)
     (in_bom yes) (on_board yes) (dnp no)
-    (property "Reference" "forced" (at 137.16 83.82 0)
+    (property "Reference" "forced" (at 137.16 86.36 0)
       (effects (font (size 1.27 1.27)))
     )
-    (property "Value" "#ForcedAnalogSignal(output_voltage)" (at 151.13 86.36 0)
+    (property "Value" "~" (at 151.13 86.36 0)
       (effects (font (size 1.27 1.27)))
     )
@@
       (effects (font (size 1.27 1.27)))
     )
-    (property "Value" "" (at 137.16 86.741 0)
+    (property "Value" "~" (at 137.16 86.741 0)
       (effects (font (size 1.27 1.27)))
     )
