File: examples/resources/FetPowerGate.kicad_sch (KiCad schematic)
At the start: 7 parts

Commit message: wip
Other:
- note added: "Additional pushbutton latching switches: https://hackaday.com/2019/06/24/ditch-the-switch-a-soft-latching-circuit-roundup/ Most are variations on this same basic idea."
- note added: "control and btn_out can be the same GPIO, if the GPIO supports a pull-up resistor that is much lower resistance (overpowers) amp_res."
Changed lines of the file:
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@@
     (stroke (width 0) (type default) (color 0 0 0 0))
   )
-  (wire (pts (xy 116.84 72.39) (xy 124.46 72.39))
+  (wire (pts (xy 119.38 139.7) (xy 127 139.7))
     (stroke (width 0) (type default) (color 0 0 0 0))
   )
@@
     (stroke (width 0) (type default) (color 0 0 0 0))
   )
-  (text "Resistor keeps it off by default" (at 63.5 93.98 0)
+  (text "Resistor keeps it off by default" (at 63.5 92.71 0)
+    (effects (font (size 1.27 1.27)) (justify left bottom))
+  )
+  (text "Additional pushbutton latching switches:\nhttps://hackaday.com/2019/06/24/ditch-the-switch-a-soft-latching-circuit-roundup/\n\nMost are variations on this same basic idea."
+    (at 50.8 139.7 0)
     (effects (font (size 1.27 1.27)) (justify left bottom))
   )
   (text "amp_fet isolates the control pin from\nbeing pack-powered by pull_res"
-    (at 69.85 123.19 0)
+    (at 63.5 118.11 0)
     (effects (font (size 1.27 1.27)) (justify left bottom))
   )
   (text "These two diodes allow the button to be\nread indepedently of the gate control.\nctl_diode prevents a control low from\n  flowing into the button pin.\nbtn_diode prevents a control high from\n  flowing into the external pin,\n  including back-powering the pin\n  from pull_res"
-    (at 50.8 118.11 0)
+    (at 50.8 110.49 0)
     (effects (font (size 1.27 1.27)) (justify left bottom))
   )
-  (global_label "gnd" (shape input) (at 116.84 72.39 180) (fields_autoplaced)
+  (text "control and btn_out can be the same GPIO,\nif the GPIO supports a pull-up resistor\nthat is much lower resistance (overpowers)\namp_res."
+    (at 63.5 128.27 0)
+    (effects (font (size 1.27 1.27)) (justify left bottom))
+  )
+  (global_label "gnd" (shape input) (at 119.38 139.7 180) (fields_autoplaced)
     (effects (font (size 1.27 1.27)) (justify right))
-    (property "Intersheet References" "${INTERSHEET_REFS}" (id 0) (at 110.9798 72.4694 0)
+    (property "Intersheet References" "${INTERSHEET_REFS}" (id 0) (at 113.5198 139.7794 0)
       (effects (font (size 1.27 1.27)) (justify right) hide)
     )
@@
     (in_bom yes) (on_board yes)
     (property "Reference" "pwr_fet" (id 0) (at 119.38 85.09 90))
-    (property "Value" "~" (id 1) (at 119.38 83.82 90))
+    (property "Value" "~" (id 1) (at 121.92 151.13 90))
     (property "Footprint" "" (id 2) (at 121.92 86.36 0)
       (effects (font (size 1.27 1.27)) hide)
@@
     (pin "1")
   )
-  (symbol (lib_id "power:GND") (at 124.46 72.39 0) (unit 1)
+  (symbol (lib_id "power:GND") (at 127 139.7 0) (unit 1)
     (in_bom yes) (on_board yes)
-    (property "Reference" "#PWR?" (id 0) (at 124.46 78.74 0)
+    (property "Reference" "#PWR?" (id 0) (at 127 146.05 0)
       (effects (font (size 1.27 1.27)) hide)
     )
-    (property "Value" "GND" (id 1) (at 120.65 73.66 0))
-    (property "Footprint" "" (id 2) (at 124.46 72.39 0)
+    (property "Value" "GND" (id 1) (at 123.19 140.97 0))
+    (property "Footprint" "" (id 2) (at 127 139.7 0)
       (effects (font (size 1.27 1.27)) hide)
     )
-    (property "Datasheet" "" (id 3) (at 124.46 72.39 0)
+    (property "Datasheet" "" (id 3) (at 127 139.7 0)
       (effects (font (size 1.27 1.27)) hide)
     )
@@
     (pin "2")
   )
-  (symbol (lib_id "Device:D") (at 105.41 107.95 180) (unit 1)
+  (symbol (lib_name "D_1") (lib_id "Device:D") (at 105.41 107.95 180) (unit 1)
     (in_bom yes) (on_board yes)
     (property "Reference" "btn_diode" (id 0) (at 105.41 105.41 0))

Commit message: a version
Parts:
- amp_fet: value ~ -> #Fet.NFet(**amp_fet)
- amp_res, pull_res: value ~ -> 10k
- btn: value ~ -> #Switch(**btn)
- btn_diode: value ~ -> #Diode(**btn_diode)
- ctl_diode: value ~ -> #Diode(**ctl_diode)
- pwr_fet: value ~ -> #Fet.PFet(**pwr_fet)
Other:
- moved on the sheet: amp_fet, amp_res, btn, btn_diode, ctl_diode

Commit message: wip style
Parts:
- amp_fet: value #Fet.NFet(**amp_fet) -> ~
- amp_res, pull_res: value 10k -> ~
- btn: value #Switch(**btn) -> ~
- btn_diode: value #Diode(**btn_diode) -> ~
- ctl_diode: value #Diode(**ctl_diode) -> ~
- pwr_fet: value #Fet.PFet(**pwr_fet) -> ~
Other:
- moved on the sheet: amp_fet, amp_res, btn, btn_diode, ctl_diode
