File: examples/resources/MultimeterCurrentDriver.kicad_sch (KiCad schematic)
At the start: 5 parts

Commit message: wip broken
Parts:
- amp: value Opamp -> ~
- diode: renamed from D?; value D -> ~
Connections:
- net GND: now also range. (V-), sw. (V-)
- net VDD: now also range. (V-), range.com, sw. (V-); no longer range.1 (common)
- net enable: now also sw. (V-); no longer sw.S
- net select: now also range.control; no longer range.3 (control)
- net at amp.2 (-), fet.3 (S), sw.1: now also range.sw; no longer range.2 (switch)
Other:
- note added: "Opamp feedback holds the fet's source node at the control voltage, providing a constant current through the ranging resistor"

Commit message: rebaseline netlist, working
Connections:
- net enable is gone; now on net VDD: sw. (V-)
Other:
- note added: "sw select connected in HDL, see code comments for details"
Changed lines of the file:
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@@
     (stroke (width 0) (type default) (color 0 0 0 0))
   )
-  (text "Opamp feedback holds the fet's\nsource node at the control voltage,\nproviding a constant current through\nthe ranging resistor"
-    (at 129.54 120.65 0)
+  (text "sw select connected in HDL,\nsee code comments for details"
+    (at 128.27 120.65 0)
     (effects (font (size 1.27 1.27)) (justify left bottom))
   )
-  (global_label "enable" (shape input) (at 118.11 114.3 0) (fields_autoplaced)
-    (effects (font (size 1.27 1.27)) (justify left))
-    (property "Intersheet References" "${INTERSHEET_REFS}" (id 0) (at 126.8126 114.3794 0)
-      (effects (font (size 1.27 1.27)) (justify left) hide)
-    )
+  (text "Opamp feedback holds the fet's\nsource node at the control voltage,\nproviding a constant current through\nthe ranging resistor"
+    (at 134.62 111.76 0)
+    (effects (font (size 1.27 1.27)) (justify left bottom))
   )
   (global_label "gnd" (shape input) (at 93.98 81.28 180) (fields_autoplaced)

Commit message: Update MultimeterCurrentDriver.kicad_sch
Other:
- note added: "FET provides negative voltage standoff Diode provides positive voltage standoff"
- note added: "Opamp feedback holds the fet's source node at the control voltage, providing a constant voltage across (and current through) the ranging resistor"
- note removed: "Opamp feedback holds the fet's source node at the control voltage, providing a constant current through the ranging resistor"
Changed lines of the file:
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@@
   (junction (at 127 100.33) (diameter 0) (color 0 0 0 0)
+  )
+  (wire (pts (xy 132.08 110.49) (xy 132.08 107.95))
+    (stroke (width 0) (type default) (color 0 0 0 0))
   )
   (wire (pts (xy 109.22 100.33) (xy 109.22 111.76))
@@
   )
   (wire (pts (xy 109.22 111.76) (xy 111.76 111.76))
-    (stroke (width 0) (type default) (color 0 0 0 0))
-  )
-  (wire (pts (xy 132.08 110.49) (xy 132.08 107.95))
     (stroke (width 0) (type default) (color 0 0 0 0))
   )
@@
   )
   (text "sw select connected in HDL,\nsee code comments for details"
+    (at 99.06 125.73 0)
+    (effects (font (size 1.27 1.27)) (justify left bottom))
+  )
+  (text "FET provides negative voltage standoff\nDiode provides positive voltage standoff"
+    (at 133.35 110.49 0)
+    (effects (font (size 1.27 1.27)) (justify left bottom))
+  )
+  (text "Opamp feedback holds the fet's source node\nat the control voltage, providing a\nconstant voltage across (and current through)\nthe ranging resistor"
     (at 128.27 120.65 0)
     (effects (font (size 1.27 1.27)) (justify left bottom))
   )
-  (text "Opamp feedback holds the fet's\nsource node at the control voltage,\nproviding a constant current through\nthe ranging resistor"
-    (at 134.62 111.76 0)
-    (effects (font (size 1.27 1.27)) (justify left bottom))
-  )
