File: examples/resources/Hx711.kicad_sch (KiCad schematic)
At the start: 10 parts, among them Q1 Q_PNP_BCE, U1 HX711

Commit message: full example
Parts:
- C1, C2: value 10uF -> 10uF 10V
- C3, C4: value 0.1uF -> 0.1uF 10V
- Q1: value Q_PNP_BCE -> ~
Other:
- moved on the sheet: C2, C4, R3, R4
