File: examples/test_fcml/FcmlBoard.kicad_pcb (KiCad board)
At the start: 2 copper layers, 139 x 123 mm, 160 parts

Commit message: diffpair wip
Routing:
- net mcu.ic.qspi_cs: track 0.00 -> 18.5 mm
- net mcu.ic.qspi.mosi: track 0.00 -> 17.7 mm, vias 0 -> 2
- net mcu.ic.qspi.sck: track 0.00 -> 17.4 mm
- net mcu.ic.qspi.miso: track 0.00 -> 16.8 mm
- net v3v3: track 116.4 -> 130.2 mm, vias 14 -> 15
- net gnd: track 59.9 -> 62.2 mm, vias 51 -> 53
Changed lines of the file:
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@@
   (segment (start -138 138.775) (end -138 139.5) (width 0.15) (layer "F.Cu") (net 1))
   (segment (start 52.225 125.18) (end 52.225 126) (width 0.2) (layer "F.Cu") (net 1))
+  (segment (start -141.475 114.905) (end -142.905 114.905) (width 0.16) (layer "F.Cu") (net 1))
   (segment (start 72.225 125.18) (end 72.225 126) (width 0.2) (layer "F.Cu") (net 1))
   (segment (start 28.5 123) (end 28 123.5) (width 0.5) (layer "F.Cu") (net 1))
@@
   (segment (start -148.775 126) (end -149.5 126) (width 0.15) (layer "F.Cu") (net 1))
   (segment (start 35 127) (end 36.05 127) (width 0.5) (layer "F.Cu") (net 1))
+  (segment (start -139.775 109) (end -140.5 109) (width 0.16) (layer "F.Cu") (net 1))
   (segment (start 28 124) (end 31.75 124) (width 0.5) (layer "F.Cu") (net 1))
   (segment (start -42.825 131) (end -43.5 131) (width 0.15) (layer "F.Cu") (net 1))
@@
   (segment (start -38.775 126) (end -39.5 126) (width 0.15) (layer "F.Cu") (net 1))
   (segment (start 57.775 128.775) (end 58 129) (width 0.2) (layer "F.Cu") (net 1))
+  (segment (start -142.905 114.905) (end -143 115) (width 0.16) (layer "F.Cu") (net 1))
   (via (at 100 105.5) (size 0.9) (drill 0.5) (layers "F.Cu" "B.Cu") (net 1))
   (via (at -138 139.5) (size 0.7) (drill 0.3) (layers "F.Cu" "B.Cu") (net 1))
@@
   (via (at 27.5 108.5) (size 0.9) (drill 0.5) (layers "F.Cu" "B.Cu") (net 1))
   (via (at -39.5 126) (size 0.7) (drill 0.3) (layers "F.Cu" "B.Cu") (net 1))
+  (via (at -140.5 109) (size 0.7) (drill 0.3) (layers "F.Cu" "B.Cu") (net 1))
   (via (at -28 130) (size 0.9) (drill 0.5) (layers "F.Cu" "B.Cu") (net 1))
   (via (at -141 131) (size 0.9) (drill 0.5) (layers "F.Cu" "B.Cu") (net 1))
@@
   (via (at 58 129) (size 0.7) (drill 0.3) (layers "F.Cu" "B.Cu") (net 1))
   (via (at 28 124) (size 0.9) (drill 0.5) (layers "F.Cu" "B.Cu") (net 1))
+  (via (at -143 115) (size 0.7) (drill 0.3) (layers "F.Cu" "B.Cu") (net 1))
   (via (at 41 124) (size 0.7) (drill 0.3) (layers "F.Cu" "B.Cu") (net 1))
   (via (at -149.5 131) (size 0.7) (drill 0.3) (layers "F.Cu" "B.Cu") (net 1))
@@
   (segment (start -37.225 126) (end -36.5 126) (width 0.15) (layer "F.Cu") (net 4))
   (segment (start -28.25 135.75) (end -28 136) (width 0.2) (layer "F.Cu") (net 4))
+  (segment (start -136.525 112.365) (end -138.365 112.365) (width 0.16) (layer "F.Cu") (net 4))
   (segment (start -139.5 127.5) (end -139.8 127.2) (width 0.15) (layer "F.Cu") (net 4))
   (segment (start -139.8 133.4375) (end -139.8 132.7) (width 0.2) (layer "F.Cu") (net 4))
   (segment (start -139.8 124.2) (end -140 124) (width 0.2) (layer "F.Cu") (net 4))
+  (segment (start -135.095 111.095) (end -135 111) (width 0.16) (layer "F.Cu") (net 4))
   (segment (start -139.8 126.5625) (end -139.8 124.2) (width 0.2) (layer "F.Cu") (net 4))
   (segment (start -136 124) (end -136 122.775) (width 0.2) (layer "F.Cu") (net 4))
@@
   (segment (start -137.4 126.5625) (end -137.4 127.4) (width 0.2) (layer "F.Cu") (net 4))
   (segment (start -34.75 127.25) (end -36 126) (width 0.2) (layer "F.Cu") (net 4))
+  (segment (start -139.635 113.635) (end -141.475 113.635) (width 0.16) (layer "F.Cu") (net 4))
   (segment (start -138 136) (end -138 137.225) (width 0.2) (layer "F.Cu") (net 4))
   (segment (start 53.775 126) (end 53.775 120.5) (width 0.2) (layer "F.Cu") (net 4))
   (segment (start 53.37 120.095) (end 52.405 120.095) (width 0.2) (layer "F.Cu") (net 4))
   (segment (start -28.25 133.45) (end -28.25 135.75) (width 0.2) (layer "F.Cu") (net 4))
+  (segment (start -136.525 111.095) (end -135.095 111.095) (width 0.16) (layer "F.Cu") (net 4))
   (segment (start -27.25 133.75) (end -27 134) (width 0.2) (layer "F.Cu") (net 4))
   (segment (start -144.6 127.4) (end -146 126) (width 0.2) (layer "F.Cu") (net 4))
@@
   (segment (start -27.25 133.45) (end -27.25 133.75) (width 0.2) (layer "F.Cu") (net 4))
   (segment (start -136.5625 131) (end -132.775 131) (width 0.2) (layer "F.Cu") (net 4))
+  (segment (start -137 109) (end -135 111) (width 0.16) (layer "F.Cu") (net 4))
   (segment (start -147.225 126) (end -146 126) (width 0.2) (layer "F.Cu") (net 4))
   (segment (start 59 127) (end 69 127) (width 0.5) (layer "F.Cu") (net 4))
   (segment (start -139.4 126.5625) (end -139.4 124.6) (width 0.2) (layer "F.Cu") (net 4))
+  (segment (start -135 112) (end -135 111) (width 0.16) (layer "F.Cu") (net 4))
   (segment (start 51.115 120.095) (end 51.02 120) (width 0.2) (layer "F.Cu") (net 4))
   (segment (start -143.4375 127.4) (end -142.6 127.4) (width 0.2) (layer "F.Cu") (net 4))
   (segment (start 72.405 120.095) (end 71.095 120.095) (width 0.2) (layer "F.Cu") (net 4))
+  (segment (start -135.365 112.365) (end -135 112) (width 0.16) (layer "F.Cu") (net 4))
   (segment (start -36 126) (end -37.225 126) (width 0.2) (layer "F.Cu") (net 4))
   (segment (start -135.4 127.4) (end -134 126) (width 0.2) (layer "F.Cu") (net 4))
@@
   (segment (start -33.45 127.25) (end -34.75 127.25) (width 0.2) (layer "F.Cu") (net 4))
   (segment (start -137 120) (end -137 121.775) (width 0.2) (layer "F.Cu") (net 4))
+  (segment (start -138.225 109) (end -137 109) (width 0.16) (layer "F.Cu") (net 4))
   (segment (start -24 129) (end -22.775 129) (width 0.2) (layer "F.Cu") (net 4))
   (segment (start -24.25 128.75) (end -24 129) (width 0.2) (layer "F.Cu") (net 4))
+  (segment (start -136.525 112.365) (end -135.365 112.365) (width 0.16) (layer "F.Cu") (net 4))
   (segment (start -137.8 127.7) (end -137.75 127.75) (width 0.2) (layer "F.Cu") (net 4))
   (segment (start -139.8 134.2) (end -138 136) (width 0.2) (layer "F.Cu") (net 4))
   (segment (start -28 137.225) (end -28 136.5) (width 0.15) (layer "F.Cu") (net 4))
   (segment (start -137.4 127.4) (end -137.75 127.75) (width 0.2) (layer "F.Cu") (net 4))
+  (segment (start -138.365 112.365) (end -139.635 113.635) (width 0.16) (layer "F.Cu") (net 4))
   (segment (start 73.775 126) (end 73.775 120.5) (width 0.2) (layer "F.Cu") (net 4))
   (segment (start -143.4375 127.4) (end -144.6 127.4) (width 0.2) (layer "F.Cu") (net 4))
@@
   (via (at 69 127) (size 0.9) (drill 0.5) (layers "F.Cu" "B.Cu") (net 4))
   (via (at -140 132.5) (size 0.7) (drill 0.3) (layers "F.Cu" "B.Cu") (net 4))
+  (via (at -135 111) (size 0.7) (drill 0.3) (layers "F.Cu" "B.Cu") (net 4))
   (via (at -142.5 131) (size 0.7) (drill 0.3) (layers "F.Cu" "B.Cu") (net 4))
   (via (at -23.5 129) (size 0.7) (drill 0.3) (layers "F.Cu" "B.Cu") (net 4))
@@
   (segment (start -18.825 131) (end -18.825 129.975) (width 0.15) (layer "F.Cu") (net 69))
   (segment (start -18.85 130) (end -18.825 129.975) (width 0.15) (layer "F.Cu") (net 69))
+  (segment (start -143.095 111.095) (end -141.475 111.095) (width 0.16) (layer "F.Cu") (net 82))
+  (segment (start -142.6 126.5625) (end -142.6 125.4) (width 0.16) (layer "F.Cu") (net 82))
+  (segment (start -144.5 123.5) (end -144.5 112.5) (width 0.16) (layer "F.Cu") (net 82))
+  (segment (start -144.5 112.5) (end -143.095 111.095) (width 0.16) (layer "F.Cu") (net 82))
+  (segment (start -142.6 125.4) (end -144.5 123.5) (width 0.16) (layer "F.Cu") (net 82))
+  (segment (start -144 113.5) (end -142.865 112.365) (width 0.16) (layer "F.Cu") (net 83))
+  (segment (start -142.2 126.5625) (end -142.2 125.3) (width 0.16) (layer "F.Cu") (net 83))
+  (segment (start -144 123.5) (end -144 113.5) (width 0.16) (layer "F.Cu") (net 83))
+  (segment (start -142.2 125.3) (end -144 123.5) (width 0.16) (layer "F.Cu") (net 83))
+  (segment (start -142.865 112.365) (end -141.475 112.365) (width 0.16) (layer "F.Cu") (net 83))
+  (segment (start -143.5 118) (end -141.5 116) (width 0.16) (layer "F.Cu") (net 84))
+  (segment (start -141.4 126.5625) (end -141.4 125.6) (width 0.16) (layer "F.Cu") (net 84))
+  (segment (start -137.905 114.905) (end -138 115) (width 0.16) (layer "F.Cu") (net 84))
+  (segment (start -141.4 125.6) (end -143.5 123.5) (width 0.16) (layer "F.Cu") (net 84))
+  (segment (start -136.525 114.905) (end -137.905 114.905) (width 0.16) (layer "F.Cu") (net 84))
+  (segment (start -143.5 123.5) (end -143.5 119) (width 0.16) (layer "F.Cu") (net 84))
+  (segment (start -143.5 119) (end -143.5 118) (width 0.16) (layer "F.Cu") (net 84))
+  (via (at -138 115) (size 0.7) (drill 0.3) (layers "F.Cu" "B.Cu") (net 84))
+  (via (at -141.5 116) (size 0.7) (drill 0.3) (layers "F.Cu" "B.Cu") (net 84))
+  (segment (start -141.5 116) (end -140.5 115) (width 0.16) (layer "B.Cu") (net 84))
+  (segment (start -140.5 115) (end -138 115) (width 0.16) (layer "B.Cu") (net 84))
+  (segment (start -141 125.5) (end -143 123.5) (width 0.16) (layer "F.Cu") (net 85))
+  (segment (start -141 126.5625) (end -141 125.5) (width 0.16) (layer "F.Cu") (net 85))
+  (segment (start -143 123.5) (end -143 118.5) (width 0.16) (layer "F.Cu") (net 85))
+  (segment (start -143 118.5) (end -138.135 113.635) (width 0.16) (layer "F.Cu") (net 85))
+  (segment (start -138.135 113.635) (end -136.525 113.635) (width 0.16) (layer "F.Cu") (net 85))
   (segment (start -142 122.775) (end -141 121.775) (width 0.2) (layer "F.Cu") (net 94))
   (segment (start -138 124) (end -138 122.775) (width 0.2) (layer "F.Cu") (net 94))

Commit message: wip
Connections:
- net mcu.usb_res.usb_rp.dm renamed mcu.usb_chain_0.d_N
- net mcu.usb_res.usb_rp.dp renamed mcu.usb_chain_0.d_P
- net usb_fpga_bitbang.usb.dm renamed usb_fpga_chain_0.d_N
- net usb_fpga_bitbang.usb.dp renamed usb_fpga_chain_0.d_P
- net usb_mcu.usb.dm renamed usb_mcu_chain_0.d_N
- net usb_mcu.usb.dp renamed usb_mcu_chain_0.d_P
Routing:
- net mcu.usb_chain_0.d_N: track 0.00 -> 10.7 mm
- net mcu.usb_chain_0.d_P: track 0.00 -> 10.7 mm

Commit message: better micro block routing
Parts:
- moved mcu.vreg_in_cap 7.21 mm to (-132.0, 122.0), turned to 0 degrees
- moved mcu.avdd_cap 4.47 mm to (-132.0, 124.0), turned to 0 degrees
- moved mcu.mem.ic 4.12 mm to (-140.0, 117.0)
- moved mcu.mem.vcc_cap 4.12 mm to (-140.0, 113.0)
- moved mcu.dvdd_cap[0] 4.00 mm to (-140.0, 122.0)
- moved mcu.iovdd_cap[5] 2.00 mm to (-138.0, 122.0)
- moved mcu.vreg_out_cap 2.00 mm to (-136.0, 122.0)
Routing:
- net v3v3: track 130.2 -> 135.4 mm
- net mcu.usb_chain_0.d_P: track 10.7 -> 6.47 mm
- net mcu.usb_chain_0.d_N: track 10.7 -> 6.56 mm
- net mcu.ic.qspi_cs: track 18.5 -> 14.6 mm
- net mcu.ic.qspi.sck: track 17.4 -> 13.6 mm
- net mcu.ic.qspi.miso: track 16.8 -> 13.2 mm
- net mcu.ic.qspi.mosi: track 17.7 -> 14.9 mm
- net gnd: track 62.2 -> 63.0 mm, vias 53 -> 54
