File: examples/test_eh_buddy/EhBuddyBoard.kicad_pcb (KiCad board)
At the start: 2 copper layers, 65 x 35 mm, 36 parts, among them sw1 5.1mm switch

Commit message: isense circuit
Parts:
- added isense.amp.amp.ic: LMV321 (Texas Instruments), Package_TO_SOT_SMD:SOT-23-5, F.Cu at (95.0, 109.0)
- added isense.amp.amp.vdd_cap: , Capacitor_SMD:C_0603_1608Metric, F.Cu at (91.0, 108.0)
- added isense.amp.r1: , Resistor_SMD:R_0603_1608Metric, F.Cu at (98.0, 111.0)
- added isense.amp.r2: , Resistor_SMD:R_0603_1608Metric, F.Cu at (92.0, 111.0)
- added isense.amp.rf: , Resistor_SMD:R_0603_1608Metric, F.Cu at (100.0, 111.0)
- added isense.amp.rg: , Resistor_SMD:R_0603_1608Metric, F.Cu at (90.0, 111.0)
- added isense.sense.res: , Resistor_SMD:R_0603_1608Metric, F.Cu at (95.0, 113.0)
- moved duck 24.5 mm to (74.0, 108.0)
- moved id 16.0 mm to (74.0, 112.0)
- moved jlc_th.th3 1.00 mm to (118.0, 83.0)
Connections:
- mcu.ic pad 10: (no net) -> sw.control
- mcu.ic pad 15: sw1.out -> isense.out
- mcu.ic pad 3: ledr.signal -> sw1.out
- mcu.ic pad 4: ledg.signal -> ledr.signal
- mcu.ic pad 5: ledb.signal -> ledg.signal
- mcu.ic pad 6: sw.control -> ledb.signal
- sw.drv pad 2: vusb -> isense.pwr_out
- sw.pull pad 1: vusb -> isense.pwr_out

Commit message: Update EhBuddyBoard.kicad_pcb
Parts:
- moved jlc_th.th1 1.00 mm to (58.0, 83.0)
- moved jlc_th.th2 1.00 mm to (58.0, 114.0)
- moved mcu.prog 1.00 mm to (109.0, 102.0)
- moved tp_3v3 1.00 mm to (59.0, 111.0)
- moved tp_gnd 1.00 mm to (69.0, 99.0)
- moved tp_vusb 1.00 mm to (59.0, 99.0)
Other:
- board size 65 x 35 mm -> 64 x 35 mm
Changed lines of the file:
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@@
   )
   (footprint "TestPoint:TestPoint_Keystone_5015_Micro-Minature" (layer "F.Cu")
-    (at 58 99)
+    (at 59 99)
     (descr "SMT Test Point- Micro Miniature 5015, http://www.keyelco.com/product-pdf.cfm?p=1353")
     (tags "Test Point")
@@
   )
   (footprint "TestPoint:TestPoint_Keystone_5015_Micro-Minature" (layer "F.Cu")
-    (at 70 99)
+    (at 69 99)
     (descr "SMT Test Point- Micro Miniature 5015, http://www.keyelco.com/product-pdf.cfm?p=1353")
     (tags "Test Point")
@@
   )
   (footprint "edg:JlcToolingHole_1.152mm" (layer "F.Cu")
-    (at 57 114)
+    (at 58 114)
     (descr "Tooling holes for JLC assembly, 1.152 mm hole + 1.3mm soldermask opening")
     (property "Sheetfile" "edg.BoardTop.JlcToolingHoles")
@@
   )
   (footprint "Button_Switch_SMD:SW_SPST_SKQG_WithoutStem" (layer "F.Cu")
-    (at 109 101)
+    (at 109 102)
     (descr "ALPS 5.2mm Square Low-profile Type (Surface Mount) SKQG Series, Without stem, http://www.alps.com/prod/info/E/HTML/Tact/SurfaceMount/SKQG/SKQGAEE010.html")
     (tags "SPST Button Switch")
@@
       (polygon
         (pts
-          (xy 110 99.7)
-          (xy 113 99.7)
-          (xy 113 102.3)
-          (xy 110 102.3)
+          (xy 110 100.7)
+          (xy 113 100.7)
+          (xy 113 103.3)
+          (xy 110 103.3)
         )
       )
@@
       (polygon
         (pts
-          (xy 105 99.7)
-          (xy 108 99.7)
-          (xy 108 102.3)
-          (xy 105 102.3)
+          (xy 105 100.7)
+          (xy 108 100.7)
+          (xy 108 103.3)
+          (xy 105 103.3)
         )
       )
@@
   )
   (footprint "edg:JlcToolingHole_1.152mm" (layer "F.Cu")
-    (at 57 83)
+    (at 58 83)
     (descr "Tooling holes for JLC assembly, 1.152 mm hole + 1.3mm soldermask opening")
     (property "Sheetfile" "edg.BoardTop.JlcToolingHoles")
@@
   )
   (footprint "TestPoint:TestPoint_Keystone_5015_Micro-Minature" (layer "F.Cu")
-    (at 58 111)
+    (at 59 111)
     (descr "SMT Test Point- Micro Miniature 5015, http://www.keyelco.com/product-pdf.cfm?p=1353")
     (tags "Test Point")
@@
     )
   )
-  (gr_rect (start 55 81) (end 120 116) (layer "Edge.Cuts") (width 0.0381) (fill none))
+  (gr_rect (start 56 81) (end 120 116) (layer "Edge.Cuts") (width 0.0381) (fill none))
   (dimension (type aligned) (layer "Cmts.User")
     (pts (xy 134 42) (xy 134 54))

Commit message: Update EhBuddyBoard.kicad_pcb
Parts:
- moved sw.drv 1.00 mm to (113.0, 110.0)
Changed lines of the file:
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@@
   )
   (footprint "Package_TO_SOT_SMD:SOT-23" (layer "F.Cu")
-    (at 112 110)
+    (at 113 110)
     (descr "SOT, 3 Pin (https://www.jedec.org/system/files/docs/to-236h.pdf variant AB), generated with kicad-footprint-generator ipc_gullwing_generator.py")
     (tags "SOT TO_SOT_SMD")

Commit message: Update EhBuddyBoard.kicad_pcb
Parts:
- moved conn 63.8 mm to (166.0, 44.2)
- moved duck 63.8 mm to (122.0, 66.0)
- moved id 63.8 mm to (122.0, 70.0)
- moved isense.amp.amp.ic 63.8 mm to (143.0, 67.0)
- moved isense.amp.amp.vdd_cap 63.8 mm to (139.0, 66.0)
- moved isense.amp.r1 63.8 mm to (146.0, 69.0)
- moved isense.amp.r2 63.8 mm to (140.0, 69.0)
- moved isense.amp.rf 63.8 mm to (148.0, 69.0)
- moved isense.amp.rg 63.8 mm to (138.0, 69.0)
- moved isense.sense.res 63.8 mm to (143.0, 71.0)
- moved jlc_th.th1 63.8 mm to (106.0, 41.0)
- moved jlc_th.th2 63.8 mm to (106.0, 72.0)
- moved jlc_th.th3 63.8 mm to (166.0, 41.0)
- moved ledb.package 63.8 mm to (130.0, 58.0)
- moved ledb.res 63.8 mm to (134.0, 58.0)
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