File: examples/test_switch_controller/SwitchControllerBoard.kicad_pcb (KiCad board)
At the start: 2 copper layers, 64 x 35 mm, 55 parts, among them J1 COM-15111 (Sparkfun), J2 PinHeader2.54 1x4 (Generic), J3 AFC01-S015FCA-00 (Jushuo), J4 PinHeader2.54 1x4 (Generic), Q1 ER-OLED-0.91-e (EastRising), Q2 2N7002 (Changjiang Electronic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, Q3 AO3401A (Alpha & Omega Semico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, SW1 5.1mm switch, SW2 5.1mm switch, U1 LD1117S33TR (STMicroelectroni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, U2 ESP32-WROOM-32 (Espressif Sys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, U3 CP2102 (Silicon Labs), U4 PESD5V0X1BT (Nexperia), U5 LMV321 (Texas Instruments), U6 Duck, U7 IdDots4

Commit message: wip
Parts:
- moved C15 90.5 mm to (120.0, 57.0)
- moved C13 85.8 mm to (124.0, 57.0)
- moved C14 85.6 mm to (124.0, 59.0)
- moved U4 80.7 mm to (122.0, 52.0)
- moved U5 77.4 mm to (117.0, 43.0)
- moved U3 31.5 mm to (148.0, 46.1)
- moved C11 29.9 mm to (155.0, 42.0), turned to 180 degrees
- moved J3 29.7 mm to (161.0, 48.0)
- moved R7 29.6 mm to (155.0, 46.0), turned to 180 degrees
- moved C7 28.6 mm to (155.0, 54.0), turned to 180 degrees
- moved C10 26.6 mm to (151.0, 50.0), turned to 180 degrees
- moved C8 26.1 mm to (155.0, 44.0), turned to 180 degrees
- moved C9 25.5 mm to (155.0, 50.0), turned to 180 degrees
- moved C12 25.2 mm to (151.0, 42.0), turned to 180 degrees
- moved C6 22.4 mm to (155.0, 52.0), turned to 180 degrees
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- renumbered Q2 to Q1, Q3 to Q2, Q1 to U3, U3 to U4, U4 to U5, U5 to U6, U6 to U7, U7 to U8
Connections:
- U2 pad 10: lcd.spi.miso -> usb_uart.uart.tx
- U2 pad 12: usb_uart.uart.tx -> ledg.signal
- U2 pad 13: conn.uart.rx -> ledr.signal
- U2 pad 14: conn.uart.tx -> ledb.signal
- U2 pad 23: ledr.signal -> isense.out
- U2 pad 26: ledg.signal -> sw.control
- U2 pad 27: ledb.signal -> conn.uart.tx
- U2 pad 28: lcd.cs -> conn.uart.rx
- U2 pad 29: lcd.reset -> lcd.cs
- U2 pad 30: lcd.dc -> lcd.reset
- U2 pad 31: (no net) -> lcd.dc
- U2 pad 33: (no net) -> lcd.spi.sck
- U2 pad 36: (no net) -> lcd.spi.mosi
- U2 pad 37: sw.control -> (no net)
- U2 pad 4: isense.out -> (no net)
- U2 pad 8: lcd.spi.sck -> (no net)
- U2 pad 9: lcd.spi.mosi -> (no net)
Routing:
- net gnd: track 0.00 -> 294.3 mm, vias 0 -> 20
- net v3v3: track 0.00 -> 158.5 mm, vias 0 -> 3
- net vusb: track 0.00 -> 72.2 mm, vias 0 -> 2
- net conn.uart.tx: track 0.00 -> 26.9 mm
- net conn.uart.rx: track 0.00 -> 25.8 mm
- net isense.out: track 0.00 -> 25.0 mm
- net ledg.signal: track 0.00 -> 24.0 mm
- net sw.control: track 0.00 -> 22.5 mm
- net usb.usb.dm: track 0.00 -> 20.4 mm, vias 0 -> 2
- net mcu.prog.out: track 0.00 -> 20.2 mm
- net lcd.spi.mosi: track 0.00 -> 19.9 mm, vias 0 -> 2
- net isense.pwr_out: track 0.00 -> 19.3 mm
- net sw1.out: track 0.00 -> 18.1 mm
- net ledr.signal: track 0.00 -> 16.8 mm
- net usb.usb.dp: track 0.00 -> 16.8 mm
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Other:
- board size 64 x 35 mm -> 64 x 39 mm
- board text added: "+5v"
- board text added: "3v3"
- board text added: "DUT"
- board text added: "GND"
- board text added: "PROG"
- board text added: "RX"
- board text added: "RX<"
- board text added: "Switch Controller Feb '23"
- board text added: "TX"
- board text added: "TX>"
- board text added: "▲"
