File: electronics_lib/resources/test_kicad_import_jlc.kicad_sch (KiCad schematic)
At the start: 2 parts, among them U1 MCP9700AT-ETT

Commit message: make it all work
Parts:
- U1: edg_blackbox (none) -> KiCadJlcBlackbox
Changed lines of the file:
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@@
       (effects (font (size 1.27 1.27)) hide)
     )
-    (property "edg_blackbox_handler" "" (id 4) (at 137.16 91.44 0)
+    (property "edg_blackbox" "KiCadJlcBlackbox" (id 4) (at 137.16 91.44 0)
       (effects (font (size 1.27 1.27)) hide)
     )
