File: electronics_lib/resources/EinkBoostPowerPath.kicad_sch (KiCad schematic)
At the start: 10 parts

Commit message: wip
Connections:
- net gdr renamed gate
- net rese renamed isense
- net vcc renamed pwr_in
- net vgh renamed pos_out
- net vgl renamed neg_out
