File: electronics_lib/resources/BootstrapVoltageAdder.kicad_sch (KiCad schematic)
At the start: 10 parts

Commit message: zero ercs!
Connections:
- net GND renamed gnd
Changed lines of the file:
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@@
     (effects (font (size 1.27 1.27)) (justify right))
+  )
+  (hierarchical_label "gnd" (shape input) (at 153.67 91.44 0) (fields_autoplaced)
+    (effects (font (size 1.27 1.27)) (justify left))
   )
   (hierarchical_label "pwr" (shape input) (at 153.67 86.36 0) (fields_autoplaced)
@@
         )
       )
-    )
-  )
-  (symbol (lib_id "power:GND") (at 153.67 91.44 0) (unit 1)
-    (in_bom yes) (on_board yes) (dnp no)
-    (property "Reference" "#PWR01" (at 153.67 97.79 0)
-      (effects (font (size 1.27 1.27)) hide)
-    )
-    (property "Value" "GND" (at 157.48 92.71 0)
-      (effects (font (size 1.27 1.27)))
-    )
-    (property "Footprint" "" (at 153.67 91.44 0)
-      (effects (font (size 1.27 1.27)) hide)
-    )
-    (property "Datasheet" "" (at 153.67 91.44 0)
-      (effects (font (size 1.27 1.27)) hide)
-    )
-    (pin "1")
-    (instances
-      (project "BootstrapVoltageAdder"
-        (path "/b55f6c44-5d5d-4524-bb86-893662f64598"
-          (reference "#PWR01") (unit 1)
-        )
-      )
