File: examples/IotKnob/IotKnob.kicad_pcb (KiCad board)
At the start: 2 copper layers, 153 x 113 mm, 91 parts

Commit message: prettier layout
Parts:
- removed the rgb_ring.led[0] at (102.6, 80.2)
- removed the rgb_ring.led[10] at (107.7, 118.5)
- removed the rgb_ring.led[11] at (102.6, 119.8)
- removed the rgb_ring.led[12] at (97.4, 119.8)
- removed the rgb_ring.led[13] at (92.3, 118.5)
- removed the rgb_ring.led[14] at (87.8, 115.9)
- removed the rgb_ring.led[15] at (84.1, 112.2)
- removed the rgb_ring.led[16] at (81.5, 107.7)
- removed the rgb_ring.led[17] at (80.2, 102.6)
- removed the rgb_ring.led[18] at (80.2, 97.4)
- removed the rgb_ring.led[19] at (81.5, 92.3)
- removed the rgb_ring.led[1] at (107.7, 81.5)
- removed the rgb_ring.led[20] at (84.1, 87.8)
- removed the rgb_ring.led[21] at (87.8, 84.1)
- removed the rgb_ring.led[22] at (92.3, 81.5)
- removed the rgb_ring.led[23] at (97.4, 80.2)
- removed the rgb_ring.led[2] at (112.2, 84.1)
- removed the rgb_ring.led[3] at (115.9, 87.8)
- removed the rgb_ring.led[4] at (118.5, 92.3)
- removed the rgb_ring.led[5] at (119.8, 97.4)
- removed the rgb_ring.led[6] at (119.8, 102.6)
- removed the rgb_ring.led[7] at (118.5, 107.7)
- removed the rgb_ring.led[8] at (115.9, 112.2)
- removed the rgb_ring.led[9] at (112.2, 115.9)
- removed rgb_sw.led[23] (x6): , SvgPcb:
- removed the sw[0] at (100.0, 68.0)
- removed the sw[1] at (127.7, 84.0)
- removed the sw[2] at (127.7, 116.0)
- removed the sw[3] at (100.0, 132.0)
- removed the sw[4] at (72.3, 116.0)
- removed the sw[5] at (72.3, 84.0)
- added dist.ic: VL53L0X (STMicroelectronics), OptoDevice:ST_VL53L0X, F.Cu at (168.2, 105.0)
- added dist.vdd_cap[0]: , Capacitor_SMD:C_0603_1608Metric, F.Cu at (171.7, 108.2)
- added dist.vdd_cap[1]: , Capacitor_SMD:C_0805_2012Metric, F.Cu at (167.5, 108.5)
- added env.ic: BME680 (Bosch Sensortec), Package_LGA:Bosch_LGA-8_3x3mm_P0.8mm_ClockwisePinNumbering, F.Cu at (171.6, 98.3)
- added env.vdd_cap: , Capacitor_SMD:C_0603_1608Metric, F.Cu at (167.3, 97.3)
- added env.vddio_cap: , Capacitor_SMD:C_0603_1608Metric, F.Cu at (167.3, 99.8)
- added rgb_knob.led[0]: SK6805-EC15 (Opsco Optoelectronics), LED_SMD:LED_SK6812_EC15_1.5x1.5mm, F.Cu at (93.0, 91.0)
- added rgb_knob.led[1]: SK6805-EC15 (Opsco Optoelectronics), LED_SMD:LED_SK6812_EC15_1.5x1.5mm, F.Cu at (107.0, 91.0)
- added rgb_knob.led[2]: SK6805-EC15 (Opsco Optoelectronics), LED_SMD:LED_SK6812_EC15_1.5x1.5mm, F.Cu at (107.0, 109.0)
- added rgb_knob.led[3]: SK6805-EC15 (Opsco Optoelectronics), LED_SMD:LED_SK6812_EC15_1.5x1.5mm, F.Cu at (94.0, 109.0)
- added rgb_ring.led[0]: SK6805-EC15 (Opsco Optoelectronics), LED_SMD:LED_SK6812_EC15_1.5x1.5mm, F.Cu at (102.6, 80.2)
- added rgb_ring.led[10]: SK6805-EC15 (Opsco Optoelectronics), LED_SMD:LED_SK6812_EC15_1.5x1.5mm, F.Cu at (107.7, 118.5)
- added rgb_ring.led[11]: SK6805-EC15 (Opsco Optoelectronics), LED_SMD:LED_SK6812_EC15_1.5x1.5mm, F.Cu at (102.6, 119.8)
- added rgb_ring.led[12]: SK6805-EC15 (Opsco Optoelectronics), LED_SMD:LED_SK6812_EC15_1.5x1.5mm, F.Cu at (97.4, 119.8)
- added rgb_ring.led[13]: SK6805-EC15 (Opsco Optoelectronics), LED_SMD:LED_SK6812_EC15_1.5x1.5mm, F.Cu at (92.3, 118.5)
- added rgb_ring.led[14]: SK6805-EC15 (Opsco Optoelectronics), LED_SMD:LED_SK6812_EC15_1.5x1.5mm, F.Cu at (87.8, 115.9)
- added rgb_ring.led[15]: SK6805-EC15 (Opsco Optoelectronics), LED_SMD:LED_SK6812_EC15_1.5x1.5mm, F.Cu at (84.1, 112.2)
- added rgb_ring.led[16]: SK6805-EC15 (Opsco Optoelectronics), LED_SMD:LED_SK6812_EC15_1.5x1.5mm, F.Cu at (81.5, 107.7)
- added rgb_ring.led[17]: SK6805-EC15 (Opsco Optoelectronics), LED_SMD:LED_SK6812_EC15_1.5x1.5mm, F.Cu at (80.2, 102.6)
- added rgb_ring.led[18]: SK6805-EC15 (Opsco Optoelectronics), LED_SMD:LED_SK6812_EC15_1.5x1.5mm, F.Cu at (80.2, 97.4)
- added rgb_ring.led[19]: SK6805-EC15 (Opsco Optoelectronics), LED_SMD:LED_SK6812_EC15_1.5x1.5mm, F.Cu at (81.5, 92.3)
- added rgb_ring.led[1]: SK6805-EC15 (Opsco Optoelectronics), LED_SMD:LED_SK6812_EC15_1.5x1.5mm, F.Cu at (107.7, 81.5)
- added rgb_ring.led[20]: SK6805-EC15 (Opsco Optoelectronics), LED_SMD:LED_SK6812_EC15_1.5x1.5mm, F.Cu at (84.1, 87.8)
- added rgb_ring.led[21]: SK6805-EC15 (Opsco Optoelectronics), LED_SMD:LED_SK6812_EC15_1.5x1.5mm, F.Cu at (87.8, 84.1)
- added rgb_ring.led[22]: SK6805-EC15 (Opsco Optoelectronics), LED_SMD:LED_SK6812_EC15_1.5x1.5mm, F.Cu at (92.3, 81.5)
- added rgb_ring.led[23]: SK6805-EC15 (Opsco Optoelectronics), LED_SMD:LED_SK6812_EC15_1.5x1.5mm, F.Cu at (97.4, 80.2)
- added rgb_ring.led[2]: SK6805-EC15 (Opsco Optoelectronics), LED_SMD:LED_SK6812_EC15_1.5x1.5mm, F.Cu at (112.2, 84.1)
- added rgb_ring.led[3]: SK6805-EC15 (Opsco Optoelectronics), LED_SMD:LED_SK6812_EC15_1.5x1.5mm, F.Cu at (115.9, 87.8)
- added rgb_ring.led[4]: SK6805-EC15 (Opsco Optoelectronics), LED_SMD:LED_SK6812_EC15_1.5x1.5mm, F.Cu at (118.5, 92.3)
- added rgb_ring.led[5]: SK6805-EC15 (Opsco Optoelectronics), LED_SMD:LED_SK6812_EC15_1.5x1.5mm, F.Cu at (119.8, 97.4)
- added rgb_ring.led[6]: SK6805-EC15 (Opsco Optoelectronics), LED_SMD:LED_SK6812_EC15_1.5x1.5mm, F.Cu at (119.8, 102.6)
- added rgb_ring.led[7]: SK6805-EC15 (Opsco Optoelectronics), LED_SMD:LED_SK6812_EC15_1.5x1.5mm, F.Cu at (118.5, 107.7)
- added rgb_ring.led[8]: SK6805-EC15 (Opsco Optoelectronics), LED_SMD:LED_SK6812_EC15_1.5x1.5mm, F.Cu at (115.9, 112.2)
- added rgb_ring.led[9]: SK6805-EC15 (Opsco Optoelectronics), LED_SMD:LED_SK6812_EC15_1.5x1.5mm, F.Cu at (112.2, 115.9)
- added rgb_sw.led[5]: SK6805-EC15 (Opsco Optoelectronics), LED_SMD:LED_SK6812_EC15_1.5x1.5mm, F.Cu at (84.0, 72.3)
- added sw[0]: 5.1mm switch, Button_Switch_SMD:SW_SPST_SKQG_WithoutStem, F.Cu at (118.0, 68.8)
- added sw[1]: 5.1mm switch, Button_Switch_SMD:SW_SPST_SKQG_WithoutStem, F.Cu at (136.0, 100.0)
- added sw[2]: 5.1mm switch, Button_Switch_SMD:SW_SPST_SKQG_WithoutStem, F.Cu at (118.0, 131.2)
- added sw[3]: 5.1mm switch, Button_Switch_SMD:SW_SPST_SKQG_WithoutStem, F.Cu at (82.0, 131.2)
- added sw[4]: 5.1mm switch, Button_Switch_SMD:SW_SPST_SKQG_WithoutStem, F.Cu at (64.0, 100.0)
- added sw[5]: 5.1mm switch, Button_Switch_SMD:SW_SPST_SKQG_WithoutStem, F.Cu at (82.0, 68.8)
- moved rgb_sw.led[4] 161.3 mm to (68.0, 100.0), turned to 180 degrees
- moved rgb_sw.led[3] 156.9 mm to (84.0, 127.7), turned to -120 degrees
- moved rgb_sw.led[0] 136.2 mm to (116.0, 72.3), turned to 60 degrees
- moved rgb_sw.led[1] 132.3 mm to (132.0, 100.0)
- moved rgb_sw.led[2] 130.8 mm to (116.0, 127.7), turned to -60 degrees
- moved usb.cc_pull.cc1 3.00 mm to (97.0, 125.0)
- moved usb.cc_pull.cc2 3.00 mm to (103.0, 125.0)
- moved usb_esd 3.00 mm to (100.0, 125.0)
- moved usb.conn 1.75 mm to (100.0, 137.8)
Connections:
- mcu.ic pad 10: oled.reset -> sw[5].out
- mcu.ic pad 11: rgb_shift.input -> oled.reset
- mcu.ic pad 23: (no net) -> rgb_shift.input
- rgb_sw.led[4] pad 3: rgb_sw.dout -> rgb_sw.led[4].dout
Routing:
- net (no net): track 746.9 -> 0.00 mm
- net vusb: track 0.00 -> 295.6 mm
- net gnd: track 236.8 -> 0.00 mm
- net rgb_sw.led[3].dout: track 0.00 -> 33.2 mm
- net rgb_sw.led[0].dout: track 0.00 -> 33.2 mm
- net rgb_sw.led[1].dout: track 0.00 -> 33.2 mm
- net rgb_sw.led[4].dout: track 0.00 -> 33.2 mm
- net rgb_ring.led[21].dout: track 0.00 -> 4.55 mm
- net rgb_ring.led[9].dout: track 0.00 -> 4.55 mm
- net rgb_ring.led[3].dout: track 0.00 -> 4.55 mm
- net rgb_ring.led[15].dout: track 0.00 -> 4.55 mm
- net rgb_ring.led[6].dout: track 0.00 -> 4.55 mm
- net rgb_ring.led[0].dout: track 0.00 -> 4.55 mm
- net rgb_ring.led[12].dout: track 0.00 -> 4.55 mm
- net rgb_ring.led[18].dout: track 0.00 -> 4.55 mm
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Other:
- board size 153 x 113 mm -> 80 x 80 mm

Commit message: wip layout
Parts:
- removed env.vddio_cap: , Capacitor_SMD:C_0603_1608Metric
- added ledw.package: C2290 (Hubei KENTO Elec) - White 0603 Light Emitting Diodes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, LED_SMD:LED_0603_1608Metric, F.Cu at (126.0, 75.5)
- added ledw.res: , Resistor_SMD:R_0603_1608Metric, F.Cu at (127.5, 77.0)
- UU4, UU6: moved to F.Cu
- env.ic: value BME680 (Bosch Sensortec) -> SHTC3 (Sensirion AG); footprint Package_LGA:Bosch_LGA-8_3x3mm_P0.8mm_ClockwisePinNumbering -> Sensor_Humidity:Sensirion_DFN-4-1EP_2x2mm_P1mm_EP0.7x1.6mm
- moved i2c_pull.scl_res 159.3 mm to (90.0, 127.0)
- moved i2c_pull.sda_res 159.0 mm to (90.0, 129.0)
- moved ledb.res 152.0 mm to (123.0, 72.5), turned to -135 degrees
- moved jlc_th.th1 151.2 mm to (125.0, 71.0)
- moved i2c_tp.tp_scl 150.7 mm to (94.0, 127.0)
- moved i2c_tp.tp_sda 150.2 mm to (94.0, 129.0)
- moved ledb.package 149.0 mm to (124.5, 74.0), turned to -135 degrees
- moved reg_3v3.in_cap 141.8 mm to (123.0, 85.0), turned to 0 degrees
- moved UU5 141.4 mm to (130.0, 120.0)
- moved reg_3v3.ic 136.5 mm to (119.0, 81.0), turned to 45 degrees
- moved mcu.vcc_cap0 136.4 mm to (112.0, 77.0), turned to -90 degrees
- moved mcu.vcc_cap1 135.2 mm to (112.0, 72.0), turned to -90 degrees
- moved reg_3v3.out_cap 134.3 mm to (115.0, 77.0), turned to -90 degrees
- moved oled.c2_cap 130.1 mm to (93.0, 68.0), turned to -90 degrees
- moved oled.c1_cap 129.0 mm to (95.0, 68.0), turned to -90 degrees
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Connections:
- env.ic pad 1: gnd -> v3v3
- env.ic pad 2: v3v3 -> i2c_chain_0.scl
- env.ic pad 4: i2c_chain_0.scl -> gnd
- mcu.ic pad 10: sw[5].out -> sw[4].out
- mcu.ic pad 11: oled.reset -> sw[5].out
- mcu.ic pad 17: knob.a -> ledw.signal
- mcu.ic pad 18: knob.b -> knob.a
- mcu.ic pad 19: knob.sw -> knob.b
- mcu.ic pad 20: sw[0].out -> knob.sw
- mcu.ic pad 21: sw[1].out -> sw[0].out
- mcu.ic pad 22: sw[2].out -> sw[1].out
- mcu.ic pad 23: rgb_shift.input -> oled.reset
- mcu.ic pad 25: (no net) -> rgb_shift.input
- mcu.ic pad 8: sw[3].out -> sw[2].out
- mcu.ic pad 9: sw[4].out -> sw[3].out
Routing:
- net gnd: track 0.00 -> 97.8 mm, vias 0 -> 23
- net rgb_knob.led[1].dout: track 0.00 -> 26.8 mm
- net v3v3: track 0.00 -> 24.5 mm, vias 0 -> 4
- net rgb_shift.output: track 0.00 -> 12.0 mm
- net i2c_chain_0.scl: track 0.00 -> 8.71 mm
- net i2c_chain_0.sda: track 0.00 -> 8.71 mm
- net rgb_knob.led[2].dout: track 0.00 -> 8.22 mm, vias 0 -> 1
- net rgb_knob.led[0].dout: track 0.00 -> 8.22 mm
- net oled.c2_cap.pos: track 0.00 -> 5.57 mm
- net oled.c1_cap.pos: track 0.00 -> 4.87 mm
- net oled.iref_res.a: track 0.00 -> 4.14 mm
- net rgb_ring.dout: track 3.28 -> 0.00 mm
- net oled.c2_cap.neg: track 0.00 -> 2.69 mm
- net oled.device.vcc: track 0.00 -> 2.63 mm
- net oled.device.vcomh: track 0.00 -> 2.51 mm
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
Commit message: route beginnings
Parts:
- removed knob: EC11J1525402 (Alps Alpine), edg:RotaryEncoder_Alps_EC11J15-Switch
- added enc: EC11J1525402 (Alps Alpine), edg:RotaryEncoder_Alps_EC11J15-Switch, F.Cu at (100.0, 100.0)
- added v5v_sense.bottom_res: , Resistor_SMD:R_0603_1608Metric, F.Cu at (123.0, 90.0)
- added v5v_sense.top_res: , Resistor_SMD:R_0603_1608Metric, F.Cu at (123.0, 88.0)
- moved tp_3v3 5.00 mm to (110.0, 135.0)
- moved tp_pwr 2.00 mm to (112.0, 135.0)
- moved tp_gnd 1.00 mm to (89.0, 135.0)
Connections:
- mcu.ic pad 10: sw[4].out -> spk_drv.i2s.ws
- mcu.ic pad 11: sw[5].out -> enc.sw
- mcu.ic pad 12: ledb.signal -> rgb_shift.input
- mcu.ic pad 15: spk_drv.i2s.sd -> ledb.signal
- mcu.ic pad 18: knob.a -> oled.reset
- mcu.ic pad 19: knob.b -> (no net)
- mcu.ic pad 20: knob.sw -> (no net)
- mcu.ic pad 21: sw[0].out -> (no net)
- mcu.ic pad 22: sw[1].out -> (no net)
- mcu.ic pad 23: oled.reset -> (no net)
- mcu.ic pad 24: (no net) -> ledg.signal
- mcu.ic pad 25: rgb_shift.input -> ledr.signal
- mcu.ic pad 31: (no net) -> enc.b
- mcu.ic pad 32: (no net) -> enc.a
- mcu.ic pad 33: (no net) -> i2c_chain_0.sda
- mcu.ic pad 34: (no net) -> i2c_chain_0.scl
- mcu.ic pad 35: (no net) -> sw[3].out
- mcu.ic pad 38: spk_drv.i2s.ws -> sw[4].out
- mcu.ic pad 39: spk_drv.i2s.sck -> sw[5].out
- mcu.ic pad 4: i2c_chain_0.scl -> sw[0].out
- mcu.ic pad 5: i2c_chain_0.sda -> sw[1].out
- mcu.ic pad 6: ledr.signal -> sw[2].out
- mcu.ic pad 7: ledg.signal -> v5v_sense.output
- mcu.ic pad 8: sw[2].out -> spk_drv.i2s.sd
- mcu.ic pad 9: sw[3].out -> spk_drv.i2s.sck
Routing:
- net sw[2].out: track 0.00 -> 85.9 mm, vias 0 -> 1
- net vusb: track 297.0 -> 380.9 mm, vias 9 -> 10
- net sw[3].out: track 0.00 -> 83.6 mm, vias 0 -> 3
- net v3v3: track 24.5 -> 95.5 mm, vias 4 -> 6
- net sw[1].out: track 0.00 -> 49.8 mm, vias 0 -> 1
- net sw[4].out: track 0.00 -> 46.8 mm, vias 0 -> 1
- net mcu.program_en_node: track 0.00 -> 42.2 mm, vias 0 -> 3
- net rgb_sw.led[2].dout: track 0.00 -> 39.7 mm, vias 0 -> 2
- net mcu.program_uart_node.b_tx: track 0.00 -> 22.2 mm, vias 0 -> 1
- net sw[5].out: track 0.00 -> 16.7 mm, vias 0 -> 1
- net sw[0].out: track 0.00 -> 16.1 mm, vias 0 -> 1
- net mcu.program_boot_node: track 0.00 -> 14.3 mm, vias 0 -> 1
- net i2c_chain_0.sda: track 8.71 -> 22.4 mm, vias 0 -> 2
- net mcu.program_uart_node.a_tx: track 0.00 -> 13.3 mm, vias 0 -> 1
- net i2c_chain_0.scl: track 8.71 -> 20.0 mm, vias 0 -> 2
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
Commit message: wip pinning
Parts:
- added io8_pur: , Resistor_SMD:R_0603_1608Metric, F.Cu at (137.2, 70.0)
- added spk_dac.c: , Capacitor_SMD:C_0603_1608Metric, F.Cu at (134.2, 63.5)
- added spk_dac.r: , Resistor_SMD:R_0603_1608Metric, F.Cu at (134.2, 66.0)
- added spk_drv.inn_cap: , Capacitor_SMD:C_0603_1608Metric, F.Cu at (140.2, 63.5)
- added spk_drv.inp_cap: , Capacitor_SMD:C_0603_1608Metric, F.Cu at (140.2, 66.0)
- added spk_tp: 5015 (Keystone) - _spk_dac_output_link, edg:TestPoint_TE_RCT_0805, F.Cu at (134.4, 58.8)
- spk_drv.ic: value MAX98357AEWL+T (Maxim Integrated) -> PAM8302AASCR (Diodes Incorporated); footprint Package_BGA:Maxim_WLP-9_1.595x1.415_Layout3x3_P0.4mm_Ball0.27mm_Pad0.25mm_NSMD -> Package_SO:MSOP-8_3x3mm_P0.65mm
Connections:
- mcu.ic pad 10: spk_drv.i2s.ws -> io8_pur.io
- mcu.ic pad 11: enc.sw -> enc.b
- mcu.ic pad 12: rgb_shift.input -> enc.a
- mcu.ic pad 15: ledb.signal -> spk_dac.input
- mcu.ic pad 17: ledw.signal -> (no net)
- mcu.ic pad 31: enc.b -> enc.sw
- mcu.ic pad 32: enc.a -> i2c_chain_0.sda
- mcu.ic pad 33: i2c_chain_0.sda -> i2c_chain_0.scl
- mcu.ic pad 34: i2c_chain_0.scl -> (no net)
- mcu.ic pad 8: spk_drv.i2s.sd -> ledb.signal
- mcu.ic pad 9: spk_drv.i2s.sck -> ledw.signal
- rgb_shift.ic pad 2: rgb_shift.input -> io8_pur.io
- spk pad 1: spk_drv.out.a -> spk_drv.spk.a
- spk pad 2: spk_drv.out.b -> spk_drv.spk.b
