File: examples/JacdacKeyswitch/JacdacKeyswitch.kicad_pcb (KiCad board)
At the start: 2 copper layers, 35 x 25 mm, 37 parts

Commit message: layout!
Parts:
- moved edge.tvs_jd_data 1.00 mm to (138.0, 104.0)
- moved edge.tvs_jd_pwr 1.00 mm to (138.0, 96.0)
- moved edge2.tvs_jd_data 1.00 mm to (162.0, 96.0)
- moved edge2.tvs_jd_pwr 1.00 mm to (162.0, 104.0)
- turned rgb.blue_res to 0 degrees
- turned rgb.green_res to 0 degrees
- turned rgb.red_res to 0 degrees
Connections:
- mcu.ic pad 13: rgb.signals.green -> (no net)
- mcu.ic pad 15: (no net) -> rgb.signals.red
- mcu.ic pad 16: rgb.signals.red -> rgb.signals.green
- mcu.ic pad 17: (no net) -> rgb.signals.blue
- mcu.ic pad 19: (no net) -> sw.out
- mcu.ic pad 2: sw.out -> (no net)
- mcu.ic pad 27: rgb.signals.blue -> (no net)
Routing:
- net jd_pwr: track 0.00 -> 69.9 mm, vias 0 -> 2
- net v3v3: track 0.00 -> 54.5 mm, vias 0 -> 6
- net jd_data.jd_data: track 0.00 -> 46.3 mm, vias 0 -> 3
- net jd_status: track 0.00 -> 39.3 mm, vias 0 -> 2
- net jd_if.signal: track 0.00 -> 30.7 mm
- net rgb.red_res.a: track 0.00 -> 15.7 mm, vias 0 -> 1
- net gnd: track 0.00 -> 14.3 mm, vias 0 -> 13
- net mcu.reset_node: track 0.00 -> 14.2 mm, vias 0 -> 2
- net sw.out: track 0.00 -> 13.8 mm
- net rgb.green_res.a: track 0.00 -> 12.2 mm, vias 0 -> 1
- net rgb.blue_res.a: track 0.00 -> 9.57 mm, vias 0 -> 1
- net jd_if.ferrite.b: track 0.00 -> 9.33 mm
- net mcu.swd_node.swdio: track 0.00 -> 5.92 mm
- net mcu.swd_node.swclk: track 0.00 -> 5.48 mm
- net rgb.signals.blue: track 0.00 -> 4.61 mm
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- added copper zone on B.Cu, net gnd
- added copper zone on F.Cu, net gnd

Commit message: Update JacdacKeyswitch.kicad_pcb
Parts:
- added duck: G***, edg:Symbol_Duckling, F.Cu at (146.5, 109.8)
- added svg2mod: G***, edg:Symbol_LemurSmall, F.Cu at (152.5, 109.5)
Routing:
- net jd_status: track 39.3 -> 42.7 mm
- net jd_pwr: track 69.9 -> 71.7 mm
- net mcu.reset_node: track 14.2 -> 13.2 mm
- net rgb.green_res.a: track 12.2 -> 11.6 mm

Commit message: layout rc1
Parts:
- moved R3 1.41 mm to (143.0, 110.0), turned to -90 degrees
- moved R4 1.41 mm to (145.0, 110.0), turned to -90 degrees
- moved R5 1.41 mm to (143.0, 106.0), turned to -90 degrees
- moved C3 1.00 mm to (157.0, 110.0)
- moved C4 1.00 mm to (155.0, 110.0)
- renumbered reg_3v3.in_cap to C1, reg_3v3.out_cap to C2, mcu.pwr_cap0 to C3, mcu.pwr_cap1 to C4, jd_if.rc.c to C5, edge.status_led.package to D1, edge.tvs_jd_pwr to D2, edge.tvs_jd_data to D3, edge2.status_led.package to D4, edge2.tvs_jd_pwr to D5, edge2.tvs_jd_data to D6, rgb.package to D7, jd_if.clamp_hi to D8, jd_if.clamp_lo to D9, edge.conn to EC1, edge2.conn to EC2, jd_if.ferrite to FB1, jlc_th.th1 to H1, jlc_th.th2 to H2, jlc_th.th3 to H3, mcu.swd to J1, jd_mh1 to MH1, jd_mh2 to MH2, jd_mh3 to MH3, jd_mh4 to MH4, edge.status_led.res to R1, edge2.status_led.res to R2, rgb.red_res to R3, rgb.green_res to R4, rgb.blue_res to R5, jd_if.rc.r to R6, sw to SW1, tp_jd_pwr to TP1, tp_gnd to TP2, tp_3v3 to TP3, reg_3v3.ic to U1, mcu.ic to U2
Connections:
- U2 pad 15: rgb.signals.red -> rgb.signals.blue
- U2 pad 16: rgb.signals.green -> rgb.signals.red
- U2 pad 17: rgb.signals.blue -> rgb.signals.green
- U2 pad 23: jd_if.signal -> (no net)
- U2 pad 26: (no net) -> jd_if.signal
Routing:
- net rgb.signals.blue: track 4.61 -> 12.4 mm
- net rgb.red_res.a: track 15.7 -> 12.5 mm
- net rgb.signals.red: track 3.38 -> 6.21 mm
- net v3v3: track 54.5 -> 56.8 mm
- net rgb.green_res.a: track 11.6 -> 9.34 mm
- net jd_if.signal: track 30.7 -> 28.8 mm
- net rgb.blue_res.a: track 9.10 -> 8.04 mm
- net jd_pwr: track 71.7 -> 72.7 mm
- net mcu.reset_node: track 13.2 -> 13.9 mm
Other:
- board text added: "Keyswitch Socket with RGB rv1"
