File: examples/IotIron/IotIron.kicad_pcb (KiCad board)
At the start: 2 copper layers, 100 x 36 mm, 93 parts

Commit message: layout wip
Parts:
- moved spk_drv.pwr_cap0 101.1 mm to (146.0, 55.0)
- moved spk_drv.pwr_cap1 101.1 mm to (146.0, 57.0)
- moved spk_drv.ic 95.1 mm to (151.0, 56.0), turned to -90 degrees
- moved spk 94.1 mm to (159.0, 56.0), turned to 180 degrees
- moved reg_gate.out_cap 43.6 mm to (195.0, 78.0), turned to 0 degrees
- moved reg_gate.ic 38.7 mm to (190.1, 77.0), turned to 180 degrees
- moved reg_gate.in_cap 38.1 mm to (195.0, 76.0), turned to 0 degrees
- moved i2c_pull.scl_res 30.9 mm to (146.0, 68.0), turned to 90 degrees
- moved i2c_pull.sda_res 28.2 mm to (148.0, 68.0), turned to 90 degrees
- moved tp_gate 21.4 mm to (185.0, 75.0)
- moved ledr.package 16.1 mm to (194.0, 42.0)
- moved ledr.res 13.6 mm to (194.0, 44.0)
- moved tp_pwm_h 13.6 mm to (185.0, 77.0)
- moved tp_pwm_l 13.6 mm to (185.0, 79.0)
- moved tp_v 9.16 mm to (182.0, 44.0)
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Routing:
- net Itamp.input_positive: track 0.00 -> 19.2 mm, vias 0 -> 2
- net Ivgate: track 4.12 -> 21.9 mm, vias 0 -> 3
- net Iv3v3: track 64.9 -> 82.2 mm, vias 8 -> 10
- net Iconv.sw.out: track 25.3 -> 8.26 mm
- net Ispk_drv.out.a: track 0.00 -> 11.6 mm
- net Ivusb: track 40.7 -> 29.6 mm, vias 6 -> 11
- net Ii2c_pull.i2c.sda: track 0.00 -> 10.3 mm, vias 0 -> 1
- net Imcu.program_en_node: track 0.00 -> 9.97 mm
- net Ispk_drv.out.b: track 0.00 -> 8.64 mm
- net Iconv.pwm_low: track 0.00 -> 8.21 mm
- net Ii2c_pull.i2c.scl: track 0.00 -> 8.05 mm, vias 0 -> 1
- net Iconv.pwm_high: track 0.00 -> 7.41 mm
- net Ignd: track 11.8 -> 6.45 mm, vias 18 -> 22
- net Itp_i.output: track 2.02 -> 7.26 mm
- net Ipd.int: track 0.00 -> 1.84 mm, vias 0 -> 1
- added copper zone on F.Cu, net Iconv.sw.out
- added copper zone on F.Cu, net Ivusb
Other:
- board text removed: "Crawler Controller rv2 Aug '23"

Commit message: wip
Parts:
- moved spk_drv.pwr_cap0 5.10 mm to (147.0, 60.0)
- moved spk_drv.pwr_cap1 5.10 mm to (147.0, 62.0)
- moved spk 4.00 mm to (155.0, 56.0)
- moved spk_drv.ic 4.00 mm to (147.0, 56.0), turned to 0 degrees
Routing:
- net Ireg_3v3.en_res.b: track 26.4 -> 11.6 mm
- net Ispk_drv.out.b: track 8.64 -> 4.67 mm
- net Iv3v3: track 82.2 -> 85.9 mm
- net Ispk_drv.out.a: track 11.6 -> 8.08 mm
- net Ispk_drv.i2s.ws: track 0.00 -> 1.17 mm, vias 0 -> 1
- net Ispk_drv.i2s.sd: track 0.00 -> 1.17 mm, vias 0 -> 1
- net Ispk_drv.i2s.sck: track 0.00 -> 1.17 mm, vias 0 -> 1

Commit message: Update IotIron.kicad_pcb
Routing:
- net Ivusb: track 29.6 -> 28.9 mm
Changed lines of the file:
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@@
   (segment (start 193.5 76) (end 194.05 76) (width 0.5) (layer "F.Cu") (net 3))
   (segment (start 133.67 72.55) (end 134.95 72.55) (width 0.2) (layer "F.Cu") (net 3))
+  (segment (start 140 70.5) (end 140 69.2625) (width 0.2) (layer "F.Cu") (net 3))
   (segment (start 135.775 58.225) (end 135.775 59) (width 0.5) (layer "F.Cu") (net 3))
   (segment (start 133.67 67.45) (end 134.95 67.45) (width 0.2) (layer "F.Cu") (net 3))
@@
   (segment (start 134.95 72.55) (end 135 72.5) (width 0.2) (layer "F.Cu") (net 3))
   (segment (start 136.475 57.525) (end 135.775 58.225) (width 0.5) (layer "F.Cu") (net 3))
-  (segment (start 140 71) (end 140 69.2625) (width 0.2) (layer "F.Cu") (net 3))
   (segment (start 132.895 67.75) (end 133.67 67.75) (width 0.2) (layer "F.Cu") (net 3))
   (segment (start 135.775 59) (end 137 59) (width 0.5) (layer "F.Cu") (net 3))
@@
   (via (at 135 67.5) (size 0.9) (drill 0.5) (layers "F.Cu" "B.Cu") (net 3))
   (via (at 193 75.5) (size 0.7) (drill 0.3) (layers "F.Cu" "B.Cu") (net 3))
-  (via (at 140 71) (size 0.7) (drill 0.3) (layers "F.Cu" "B.Cu") (net 3))
+  (via (at 140 70.5) (size 0.7) (drill 0.3) (layers "F.Cu" "B.Cu") (net 3))
   (via (at 137.5 55.5) (size 0.9) (drill 0.5) (layers "F.Cu" "B.Cu") (net 3))
   (via (at 203 74.5) (size 0.9) (drill 0.5) (layers "F.Cu" "B.Cu") (net 3))
@@
   (via (at 132 57) (size 0.9) (drill 0.5) (layers "F.Cu" "B.Cu") (net 3))
   (via (at 135 72.5) (size 0.9) (drill 0.5) (layers "F.Cu" "B.Cu") (net 3))
-  (segment (start 136.5 67.5) (end 140 71) (width 0.2) (layer "B.Cu") (net 3))
-  (segment (start 135 67.5) (end 136.5 67.5) (width 0.2) (layer "B.Cu") (net 3))
+  (segment (start 138 70.5) (end 135 67.5) (width 0.2) (layer "B.Cu") (net 3))
+  (segment (start 140 70.5) (end 138 70.5) (width 0.2) (layer "B.Cu") (net 3))
   (segment (start 145.5625 56.25) (end 146.5 56.25) (width 0.2) (layer "F.Cu") (net 4))
   (segment (start 133.67 73.755) (end 133.67 73.35) (width 0.2) (layer "F.Cu") (net 4))
@@
       0d21ae96-2daa-474f-a3a7-d79d4792b5b2
       0ded325b-6ac3-49f7-8175-7a20026109cf
+      0f1ec1c9-dbf0-4d51-9b56-e5f23e76bb40
       11aa9a10-edfd-42d9-8035-eec5f5ac0ec1
       12299290-c0e5-4407-9de9-b31833e28f51
@@
       61eef90d-cc08-445c-b41c-5bb22086a5f0
       629b89a6-7f3b-43c3-a5cc-dad2f612e232
+      680c9fb0-26ab-4640-8bd3-d7b203450555
       6ab5854d-f830-4714-b2fa-0742e3bfd0fc
+      6be1ea21-7127-4e72-95b1-20e3b9ba4b75
       754fab17-a229-44a8-a0b7-2e60cb356246
       76b3256e-79bd-4915-92e3-67d793cf8f84
@@
       7a471fa2-cc53-41a3-abef-a48c5e686c82
       8422cfc1-f5bc-42f1-85ff-49716f3c9d26
-      86b3cff4-767e-4708-9fd5-11427b076157
       89668dc8-29ef-40c8-b578-6a3a4cd0354d
       89f0feab-c873-41a9-8a25-39d51095b8bf

Commit message: routing
Parts:
- moved ledr.package 74.9 mm to (130.0, 81.0), turned to 180 degrees
- moved ledr.res 70.5 mm to (134.0, 81.0), turned to 0 degrees
- moved prot_3v3 30.1 mm to (177.0, 77.0)
- moved tp_v 29.8 mm to (189.0, 73.0)
- moved vfilt.c 29.4 mm to (185.0, 71.0)
- moved vsense.bottom_res 27.2 mm to (189.0, 71.0)
- moved vsense.top_res 27.2 mm to (189.0, 69.0), turned to 180 degrees
- moved vfilt.r 25.5 mm to (185.0, 69.0), turned to 180 degrees
- moved mcu.en_pull.r 2.00 mm to (177.0, 75.0)
- moved tp_pwr 2.00 mm to (139.0, 76.0)
- moved vusb_sense.top_res 2.00 mm to (139.0, 79.0)
- moved mcu.prog 0.14 mm to (130.0, 77.5)
- turned spk_drv.pwr_cap0 to 0 degrees
- turned spk_drv.pwr_cap1 to 0 degrees
Connections:
- net Iusb.A6 renamed Iusb_chain_0.d_P
- net Iusb.A7 renamed Iusb_chain_0.d_N
- ledr.package pad 2: Iv3v3 -> Iledr.signal
- ledr.res pad 2: Iledr.signal -> Ignd
- mcu.ic pad 10: Ispk_drv.i2s.sd -> (no net)
- mcu.ic pad 12: Ienc.a -> Ienc.sw
- mcu.ic pad 15: Itp_i.output -> Ivfilt.output
- mcu.ic pad 17: Ienc.b -> Ioled.reset
- mcu.ic pad 18: Ienc.sw -> Iconv.pwm_low
- mcu.ic pad 19: Ioled.reset -> Iconv.pwm_high
- mcu.ic pad 20: Iledr.signal -> Ispk_drv.i2s.sck
- mcu.ic pad 21: Iconv.pwm_low -> Ispk_drv.i2s.ws
- mcu.ic pad 22: Iconv.pwm_high -> Ispk_drv.i2s.sd
- mcu.ic pad 33: (no net) -> Ii2c_pull.i2c.sda
- mcu.ic pad 34: (no net) -> Ii2c_pull.i2c.scl
- mcu.ic pad 35: (no net) -> Ipd.int
- mcu.ic pad 38: Ivfilt.output -> Ivusb_sense.output
- mcu.ic pad 39: Ivusb_sense.output -> Iledr.signal
- mcu.ic pad 4: Itamp.output -> Itp_i.output
- mcu.ic pad 5: Ii2c_pull.i2c.scl -> Itamp.output
- mcu.ic pad 6: Ii2c_pull.i2c.sda -> Ienc.a
- mcu.ic pad 7: Ipd.int -> Ienc.b
- mcu.ic pad 8: Ispk_drv.i2s.sck -> (no net)
- mcu.ic pad 9: Ispk_drv.i2s.ws -> (no net)
Routing:
- net Iv3v3: track 85.9 -> 141.2 mm
- net Imcu.program_en_node: track 9.97 -> 55.0 mm, vias 0 -> 2
- net Imcu.program_boot_node: track 0.00 -> 42.4 mm, vias 0 -> 3
- net Ivusb: track 28.9 -> 63.2 mm, vias 11 -> 13
- net Imcu.program_uart_node.a_tx: track 0.00 -> 26.4 mm, vias 0 -> 2
- net Imcu.program_uart_node.b_tx: track 0.00 -> 24.7 mm
- net Iledr.signal: track 0.00 -> 24.1 mm
- net Ivusb_sense.output: track 0.00 -> 13.4 mm
- net Ipd.int: track 1.84 -> 13.7 mm, vias 1 -> 2
- net Ii2c_pull.i2c.scl: track 8.05 -> 17.8 mm, vias 1 -> 2
- net Ii2c_pull.i2c.sda: track 10.3 -> 17.5 mm
- net Ivsense.output: track 0.00 -> 4.35 mm
- net Iusb_chain_0.d_N: track 10.3 -> 13.5 mm, vias 2 -> 3
- net Iledr.res.a: track 0.00 -> 2.39 mm
- net Ivfilt.output: track 0.00 -> 2.02 mm
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
Commit message: continued routing
Connections:
- ledr.package pad 2: Iledr.signal -> Iv3v3
- ledr.res pad 2: Ignd -> Imcu.program_boot_node
- mcu.ic pad 10: (no net) -> Ienc.sw
- mcu.ic pad 11: (no net) -> Ioled.reset
- mcu.ic pad 12: Ienc.sw -> Itamp.output
- mcu.ic pad 15: Ivfilt.output -> (no net)
- mcu.ic pad 17: Ioled.reset -> (no net)
- mcu.ic pad 18: Iconv.pwm_low -> (no net)
- mcu.ic pad 19: Iconv.pwm_high -> (no net)
- mcu.ic pad 20: Ispk_drv.i2s.sck -> (no net)
- mcu.ic pad 21: Ispk_drv.i2s.ws -> (no net)
- mcu.ic pad 22: Ispk_drv.i2s.sd -> (no net)
- mcu.ic pad 31: (no net) -> Ispk_drv.i2s.ws
- mcu.ic pad 32: (no net) -> Ispk_drv.i2s.sck
- mcu.ic pad 33: Ii2c_pull.i2c.sda -> Ispk_drv.i2s.sd
- mcu.ic pad 34: Ii2c_pull.i2c.scl -> Ii2c_pull.i2c.sda
- mcu.ic pad 35: Ipd.int -> Ii2c_pull.i2c.scl
- mcu.ic pad 38: Ivusb_sense.output -> Ipd.int
- mcu.ic pad 39: Iledr.signal -> Ivusb_sense.output
- mcu.ic pad 4: Itp_i.output -> Iconv.pwm_low
- mcu.ic pad 5: Itamp.output -> Iconv.pwm_high
- mcu.ic pad 6: Ienc.a -> Ivfilt.output
- mcu.ic pad 7: Ienc.b -> Itp_i.output
- mcu.ic pad 8: (no net) -> Ienc.a
- mcu.ic pad 9: (no net) -> Ienc.b
Routing:
- net Iledr.signal: track 24.1 -> 0.00 mm
- net Ispk_drv.i2s.sd: track 1.17 -> 22.6 mm, vias 1 -> 2
- net Ispk_drv.i2s.sck: track 1.17 -> 21.4 mm, vias 1 -> 2
- net Ispk_drv.i2s.ws: track 1.17 -> 19.4 mm, vias 1 -> 2
- net Iv3v3: track 141.2 -> 150.9 mm, vias 10 -> 11
- net Ipd.int: track 13.7 -> 18.5 mm
- net Ii2c_pull.i2c.sda: track 17.5 -> 20.1 mm, vias 1 -> 2
- net Ii2c_pull.i2c.scl: track 17.8 -> 20.2 mm
- net Ipd.ic.vconn: track 0.00 -> 1.68 mm
- net Ivusb: track 63.2 -> 62.4 mm, vias 13 -> 10
- net Imcu.program_uart_node.a_tx: track 26.4 -> 25.7 mm
- net Imcu.program_boot_node: track 42.4 -> 43.1 mm
- net Ignd: vias 26 -> 27

Commit message: routed
Parts:
- moved prot_3v3 28.0 mm to (161.0, 54.0)
- moved tp_t 16.5 mm to (197.0, 69.0)
- moved iamp 8.25 mm to (189.0, 61.0)
- moved tp_v 5.66 mm to (193.0, 69.0)
- moved temp.vdd_cap 4.00 mm to (223.0, 59.0), turned to 0 degrees
- moved mcu.en_pull.r 2.00 mm to (177.0, 77.0)
- moved temp.ic 2.00 mm to (223.0, 62.0), turned to 180 degrees
- turned tp_i.c to 0 degrees
Connections:
- mcu.ic pad 10: Ienc.sw -> Ienc.a
- mcu.ic pad 8: Ienc.a -> Ienc.sw
Routing:
- net Iv3v3: track 150.9 -> 284.5 mm, vias 11 -> 14
- net Ii2c_pull.i2c.sda: track 20.1 -> 104.2 mm, vias 2 -> 4
- net Ii2c_pull.i2c.scl: track 20.2 -> 102.7 mm, vias 2 -> 4
- net Ienc.sw: track 0.00 -> 53.2 mm, vias 0 -> 2
- net Iisense.pwr_out: track 0.00 -> 44.3 mm, vias 0 -> 2
- net Ienc.a: track 0.00 -> 39.5 mm, vias 0 -> 2
- net Ienc.b: track 0.00 -> 38.5 mm, vias 0 -> 2
- net Iusb_chain_0.d_P: track 11.3 -> 43.4 mm, vias 3 -> 4
- net Iusb_chain_0.d_N: track 13.5 -> 44.8 mm, vias 3 -> 4
- net Iconv_out: track 1.18 -> 30.9 mm, vias 1 -> 2
- net Itamp.output: track 5.46 -> 33.6 mm, vias 0 -> 2
- net Itp_i.output: track 7.26 -> 30.3 mm
- net Ioled.reset: track 0.00 -> 21.3 mm, vias 0 -> 2
- net Iconv.pwm_low: track 8.21 -> 28.1 mm
- net Iconv.pwm_high: track 7.41 -> 25.8 mm
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- added copper zone on F.Cu, net Iconv_out
- added copper zone on F.Cu, net Iisense.pwr_out
- added copper zone on B.Cu, net Ivusb

Commit message: Update IotIron.kicad_pcb
Parts:
- renumbered reg_3v3.hf_in_cap to IC1, mcu.en_pull.c to IC10, pd.vdd_cap[0] to IC11, pd.vdd_cap[1] to IC12, temp.vdd_cap to IC13, oled.c1_cap to IC14, oled.c2_cap to IC15, oled.vcomh_cap to IC16, oled.vdd_cap1 to IC17, oled.vbat_cap to IC18, oled.vcc_cap to IC19, reg_3v3.boot_cap to IC2, spk_drv.pwr_cap0 to IC20, spk_drv.pwr_cap1 to IC21, conv.power_path.in_cap.c[0] to IC22, conv.power_path.in_cap.c[1] to IC23, conv.power_path.out_cap to IC24, conv.sw.driver.cap to IC25, conv.sw.driver.boot_cap to IC26, vfilt.c to IC27, tp_i.c to IC28, packed_opamp.vdd_cap to IC29, reg_3v3.power_path.in_cap.c[0] to IC3, reg_3v3.power_path.in_cap.c[1] to IC4, reg_3v3.power_path.out_cap to IC5, reg_gate.in_cap to IC6, reg_gate.out_cap to IC7, mcu.vcc_cap0 to IC8, mcu.vcc_cap1 to IC9, prot_3v3 to ID1, ledr.package to ID2, jlc_th.th1 to IH1, jlc_th.th2 to IH2, jlc_th.th3 to IH3, usb to IJ1, mcu.prog to IJ2, oled.device to IJ3, spk to IJ4, iron to IJ5, reg_3v3.power_path.inductor to IL1, conv.power_path.inductor to IL2, conv.sw.low_fet to IQ1, conv.sw.high_fet to IQ2, reg_3v3.fb.top_res to IR1, ledr.res to IR10, conv.sw.low_gate_res to IR11, conv.sw.high_gate_res to IR12, isense to IR13, vsense.top_res to IR14, vsense.bottom_res to IR15, vfilt.r to IR16, ifilt.r1 to IR17, ifilt.r2 to IR18, tp_i.r to IR19, reg_3v3.fb.bottom_res to IR2, tamp.r1 to IR20, tamp.r2 to IR21, tamp.rf to IR22, tamp.rg to IR23, reg_3v3.en_res to IR3, mcu.en_pull.r to IR4, i2c_pull.scl_res to IR5, i2c_pull.sda_res to IR6, vusb_sense.top_res to IR7, vusb_sense.bottom_res to IR8, oled.iref_res to IR9, enc to ISW1, tp_pwr to ITP1, tp_t to ITP10, tp_gnd to ITP2, tp_3v3 to ITP3, tp_gate to ITP4, tp_conv to ITP5, tp_pwm_l to ITP6, tp_pwm_h to ITP7, tp_v to ITP8, iamp to ITP9, reg_3v3.ic to IU1, packed_opamp.ic to IU10, reg_gate.ic to IU2, mcu.ic to IU3, pd.ic to IU4, usb_esd to IU5, temp.ic to IU6, oled.lcd to IU7, spk_drv.ic to IU8, conv.sw.driver.ic to IU9
Routing:
- net Ignd: track 23.2 -> 25.0 mm, vias 37 -> 36

Commit message: wip
Parts:
- removed H12: MountingHole_2.7mm_M2.5, MountingHole:MountingHole_2.7mm_M2.5
- UU4, UU5: moved to F.Cu
- moved UU5 121.5 mm to (160.0, 57.0), turned to 0 degrees
- moved UU4 110.5 mm to (166.0, 57.0), turned to 0 degrees
Routing:
- net Iv3v3: track 284.5 -> 285.2 mm, vias 14 -> 15
Other:
- board text added: "IoT Iron Controller"
- board text added: "rv1 Oct'23"
