File: examples/RobotCrawler/CrawlerTimer.kicad_pcb (KiCad board)
At the start: 2 copper layers, 50 x 62 mm, 38 parts

Commit message: preautoroutin g
Connections:
- mcu.ic pad 10: servo_fs90fbs[6].pwm -> servo_fs90fbs[2].pwm
- mcu.ic pad 11: servo_fs90fbs[7].pwm -> servo_fs90fbs[3].pwm
- mcu.ic pad 12: servo_fs90fbs[7].fb -> i2c_pull.i2c.scl
- mcu.ic pad 15: servo_fs90fbs[2].fb -> servo_fs90fbs[4].fb
- mcu.ic pad 17: i2c_pull.i2c.scl -> servo_fs90fbs[5].fb
- mcu.ic pad 19: servo_fs90fbs[0].pwm -> ledy.signal
- mcu.ic pad 20: servo_fs90fbs[1].pwm -> ledw.signal
- mcu.ic pad 21: servo_fs90fbs[2].pwm -> sw.out
- mcu.ic pad 22: servo_fs90fbs[3].pwm -> (no net)
- mcu.ic pad 23: servo_fs90rs[2].pwm -> (no net)
- mcu.ic pad 24: ledy.signal -> (no net)
- mcu.ic pad 25: servo_fs90rs[3].pwm -> servo_fs90fbs[4].pwm
- mcu.ic pad 31: ledw.signal -> servo_fs90fbs[5].pwm
- mcu.ic pad 32: sw.out -> servo_fs90fbs[6].pwm
- mcu.ic pad 33: (no net) -> servo_fs90fbs[7].pwm
- mcu.ic pad 34: (no net) -> servo_fs90rs[2].pwm
- mcu.ic pad 35: (no net) -> servo_fs90rs[3].pwm
- mcu.ic pad 38: servo_fs90fbs[1].fb -> servo_fs90fbs[6].fb
- mcu.ic pad 39: servo_fs90fbs[0].fb -> servo_fs90fbs[7].fb
- mcu.ic pad 4: servo_fs90fbs[3].fb -> servo_fs90fbs[0].fb
- mcu.ic pad 5: servo_fs90fbs[4].fb -> servo_fs90fbs[1].fb
- mcu.ic pad 6: servo_fs90fbs[5].fb -> servo_fs90fbs[2].fb
- mcu.ic pad 7: servo_fs90fbs[6].fb -> servo_fs90fbs[3].fb
- mcu.ic pad 8: servo_fs90fbs[4].pwm -> servo_fs90fbs[0].pwm
- mcu.ic pad 9: servo_fs90fbs[5].pwm -> servo_fs90fbs[1].pwm
Routing:
- net batt.pwr: track 0.00 -> 117.9 mm
- net imu.pwr: track 0.00 -> 79.1 mm
Changed lines of the file:
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@@
       (net 1 "mcu.program_en_node"))
     (pad "4" smd rect (at -8.75 -1.45) (size 1.5 0.9) (layers "F.Cu" "F.Paste" "F.Mask")
+      (net 35 "servo_fs90fbs[0].fb"))
+    (pad "5" smd rect (at -8.75 -0.18) (size 1.5 0.9) (layers "F.Cu" "F.Paste" "F.Mask")
+      (net 34 "servo_fs90fbs[1].fb"))
+    (pad "6" smd rect (at -8.75 1.09) (size 1.5 0.9) (layers "F.Cu" "F.Paste" "F.Mask")
+      (net 24 "servo_fs90fbs[2].fb"))
+    (pad "7" smd rect (at -8.75 2.36) (size 1.5 0.9) (layers "F.Cu" "F.Paste" "F.Mask")
       (net 9 "servo_fs90fbs[3].fb"))
-    (pad "5" smd rect (at -8.75 -0.18) (size 1.5 0.9) (layers "F.Cu" "F.Paste" "F.Mask")
-      (net 10 "servo_fs90fbs[4].fb"))
-    (pad "6" smd rect (at -8.75 1.09) (size 1.5 0.9) (layers "F.Cu" "F.Paste" "F.Mask")
-      (net 11 "servo_fs90fbs[5].fb"))
-    (pad "7" smd rect (at -8.75 2.36) (size 1.5 0.9) (layers "F.Cu" "F.Paste" "F.Mask")
-      (net 12 "servo_fs90fbs[6].fb"))
     (pad "8" smd rect (at -8.75 3.63) (size 1.5 0.9) (layers "F.Cu" "F.Paste" "F.Mask")
-      (net 14 "servo_fs90fbs[4].pwm"))
+      (net 25 "servo_fs90fbs[0].pwm"))
     (pad "9" smd rect (at -8.75 4.9) (size 1.5 0.9) (layers "F.Cu" "F.Paste" "F.Mask")
-      (net 16 "servo_fs90fbs[5].pwm"))
+      (net 26 "servo_fs90fbs[1].pwm"))
     (pad "10" smd rect (at -8.75 6.17) (size 1.5 0.9) (layers "F.Cu" "F.Paste" "F.Mask")
-      (net 17 "servo_fs90fbs[6].pwm"))
+      (net 27 "servo_fs90fbs[2].pwm"))
     (pad "11" smd rect (at -8.75 7.44) (size 1.5 0.9) (layers "F.Cu" "F.Paste" "F.Mask")
-      (net 18 "servo_fs90fbs[7].pwm"))
+      (net 28 "servo_fs90fbs[3].pwm"))
     (pad "12" smd rect (at -8.75 8.71) (size 1.5 0.9) (layers "F.Cu" "F.Paste" "F.Mask")
-      (net 21 "servo_fs90fbs[7].fb"))
+      (net 3 "i2c_pull.i2c.scl"))
     (pad "13" smd rect (at -8.75 9.98) (size 1.5 0.9) (layers "F.Cu" "F.Paste" "F.Mask")
       (net 22 "servo_fs90rs[0].pwm"))
@@
       (net 23 "servo_fs90rs[1].pwm"))
     (pad "15" smd rect (at -6.985 12.5 270) (size 1.5 0.9) (layers "F.Cu" "F.Paste" "F.Mask")
-      (net 24 "servo_fs90fbs[2].fb"))
+      (net 10 "servo_fs90fbs[4].fb"))
     (pad "16" smd rect (at -5.715 12.5 270) (size 1.5 0.9) (layers "F.Cu" "F.Paste" "F.Mask"))
     (pad "17" smd rect (at -4.445 12.5 270) (size 1.5 0.9) (layers "F.Cu" "F.Paste" "F.Mask")
-      (net 3 "i2c_pull.i2c.scl"))
+      (net 11 "servo_fs90fbs[5].fb"))
     (pad "18" smd rect (at -3.175 12.5 270) (size 1.5 0.9) (layers "F.Cu" "F.Paste" "F.Mask")
       (net 6 "i2c_pull.i2c.sda"))
     (pad "19" smd rect (at -1.905 12.5 270) (size 1.5 0.9) (layers "F.Cu" "F.Paste" "F.Mask")
-      (net 25 "servo_fs90fbs[0].pwm"))
+      (net 30 "ledy.signal"))
     (pad "20" smd rect (at -0.635 12.5 270) (size 1.5 0.9) (layers "F.Cu" "F.Paste" "F.Mask")
-      (net 26 "servo_fs90fbs[1].pwm"))
+      (net 33 "ledw.signal"))
     (pad "21" smd rect (at 0.635 12.5 270) (size 1.5 0.9) (layers "F.Cu" "F.Paste" "F.Mask")
-      (net 27 "servo_fs90fbs[2].pwm"))
-    (pad "22" smd rect (at 1.905 12.5 270) (size 1.5 0.9) (layers "F.Cu" "F.Paste" "F.Mask")
-      (net 28 "servo_fs90fbs[3].pwm"))
-    (pad "23" smd rect (at 3.175 12.5 270) (size 1.5 0.9) (layers "F.Cu" "F.Paste" "F.Mask")
-      (net 29 "servo_fs90rs[2].pwm"))
-    (pad "24" smd rect (at 4.445 12.5 270) (size 1.5 0.9) (layers "F.Cu" "F.Paste" "F.Mask")
-      (net 30 "ledy.signal"))
+      (net 13 "sw.out"))
+    (pad "22" smd rect (at 1.905 12.5 270) (size 1.5 0.9) (layers "F.Cu" "F.Paste" "F.Mask"))
+    (pad "23" smd rect (at 3.175 12.5 270) (size 1.5 0.9) (layers "F.Cu" "F.Paste" "F.Mask"))
+    (pad "24" smd rect (at 4.445 12.5 270) (size 1.5 0.9) (layers "F.Cu" "F.Paste" "F.Mask"))
     (pad "25" smd rect (at 5.715 12.5 270) (size 1.5 0.9) (layers "F.Cu" "F.Paste" "F.Mask")
-      (net 32 "servo_fs90rs[3].pwm"))
+      (net 14 "servo_fs90fbs[4].pwm"))
     (pad "26" smd rect (at 6.985 12.5 270) (size 1.5 0.9) (layers "F.Cu" "F.Paste" "F.Mask"))
     (pad "27" smd rect (at 8.75 11.25) (size 1.5 0.9) (layers "F.Cu" "F.Paste" "F.Mask")
@@
     (pad "30" smd rect (at 8.75 7.44) (size 1.5 0.9) (layers "F.Cu" "F.Paste" "F.Mask"))
     (pad "31" smd rect (at 8.75 6.17) (size 1.5 0.9) (layers "F.Cu" "F.Paste" "F.Mask")
-      (net 33 "ledw.signal"))
+      (net 16 "servo_fs90fbs[5].pwm"))
     (pad "32" smd rect (at 8.75 4.9) (size 1.5 0.9) (layers "F.Cu" "F.Paste" "F.Mask")
-      (net 13 "sw.out"))
-    (pad "33" smd rect (at 8.75 3.63) (size 1.5 0.9) (layers "F.Cu" "F.Paste" "F.Mask"))
-    (pad "34" smd rect (at 8.75 2.36) (size 1.5 0.9) (layers "F.Cu" "F.Paste" "F.Mask"))
-    (pad "35" smd rect (at 8.75 1.09) (size 1.5 0.9) (layers "F.Cu" "F.Paste" "F.Mask"))
+      (net 17 "servo_fs90fbs[6].pwm"))
+    (pad "33" smd rect (at 8.75 3.63) (size 1.5 0.9) (layers "F.Cu" "F.Paste" "F.Mask")
+      (net 18 "servo_fs90fbs[7].pwm"))
+    (pad "34" smd rect (at 8.75 2.36) (size 1.5 0.9) (layers "F.Cu" "F.Paste" "F.Mask")
+      (net 29 "servo_fs90rs[2].pwm"))
+    (pad "35" smd rect (at 8.75 1.09) (size 1.5 0.9) (layers "F.Cu" "F.Paste" "F.Mask")
+      (net 32 "servo_fs90rs[3].pwm"))
     (pad "36" smd rect (at 8.75 -0.18) (size 1.5 0.9) (layers "F.Cu" "F.Paste" "F.Mask")
       (net 19 "mcu.program_uart_node.b_tx"))
@@
       (net 20 "mcu.program_uart_node.a_tx"))
     (pad "38" smd rect (at 8.75 -2.72) (size 1.5 0.9) (layers "F.Cu" "F.Paste" "F.Mask")
-      (net 34 "servo_fs90fbs[1].fb"))
+      (net 12 "servo_fs90fbs[6].fb"))
     (pad "39" smd rect (at 8.75 -3.99) (size 1.5 0.9) (layers "F.Cu" "F.Paste" "F.Mask")
-      (net 35 "servo_fs90fbs[0].fb"))
+      (net 21 "servo_fs90fbs[7].fb"))
     (pad "40" smd rect (at 8.75 -5.26) (size 1.5 0.9) (layers "F.Cu" "F.Paste" "F.Mask")
       (net 5 "batt.gnd"))
@@
   (gr_line (start 75 98) (end 75 150)
     (stroke (width 0.0381) (type default)) (layer "Edge.Cuts"))
+  (segment (start 85 97) (end 78 97) (width 0.5) (layer "F.Cu") (net 2))
+  (segment (start 80.525 95) (end 79 95) (width 0.5) (layer "F.Cu") (net 2))
+  (segment (start 89 95) (end 87.775 95) (width 0.5) (layer "F.Cu") (net 2))
+  (segment (start 90.01 96.01) (end 89 95) (width 0.5) (layer "F.Cu") (net 2))
+  (segment (start 78 97) (end 78 112) (width 0.5) (layer "F.Cu") (net 2))
+  (segment (start 97 128) (end 99 130) (width 0.5) (layer "F.Cu") (net 2))
+  (segment (start 85 96) (end 90 96) (width 0.5) (layer "F.Cu") (net 2))
+  (segment (start 85 97) (end 85 96) (width 0.5) (layer "F.Cu") (net 2))
+  (segment (start 91.25 96.01) (end 90.01 96.01) (width 0.5) (layer "F.Cu") (net 2))
+  (segment (start 86.175 97) (end 85 97) (width 0.5) (layer "F.Cu") (net 2))
+  (segment (start 84 118) (end 84 121) (width 0.5) (layer "F.Cu") (net 2))
+  (segment (start 78 112) (end 84 118) (width 0.5) (layer "F.Cu") (net 2))
+  (segment (start 93 130) (end 99.85 130) (width 0.5) (layer "F.Cu") (net 2))
+  (segment (start 99 130) (end 99.85 130) (width 0.5) (layer "F.Cu") (net 2))
+  (segment (start 90 96) (end 90.01 96.01) (width 0.5) (layer "F.Cu") (net 2))
+  (segment (start 99.85 130) (end 106.15 130) (width 0.5) (layer "F.Cu") (net 2))
+  (segment (start 84 121) (end 93 130) (width 0.5) (layer "F.Cu") (net 2))
+  (segment (start 95.95 128) (end 97 128) (width 0.5) (layer "F.Cu") (net 2))
+  (segment (start 79 95) (end 78 96) (width 0.5) (layer "F.Cu") (net 2))
+  (segment (start 78 96) (end 78 97) (width 0.5) (layer "F.Cu") (net 2))
+  (segment (start 82 121) (end 91 130) (width 0.5) (layer "F.Cu") (net 38))
+  (segment (start 96 134) (end 97.3 132.7) (width 0.5) (layer "F.Cu") (net 38))
+  (segment (start 97.3 132.3) (end 97 132) (width 0.5) (layer "F.Cu") (net 38))
+  (segment (start 91 132) (end 93 134) (width 0.5) (layer "F.Cu") (net 38))
+  (segment (start 93 134) (end 96 134) (width 0.5) (layer "F.Cu") (net 38))
+  (segment (start 99.85 132.3) (end 97.3 132.3) (width 0.5) (layer "F.Cu") (net 38))
+  (segment (start 91 130) (end 91 132) (width 0.5) (layer "F.Cu") (net 38))
+  (segment (start 97.3 132.7) (end 97.3 132.3) (width 0.5) (layer "F.Cu") (net 38))
+  (segment (start 97 132) (end 95.775 132) (width 0.5) (layer "F.Cu") (net 38))
+  (segment (start 82 121) (end 79.54 123.46) (width 0.5) (layer "B.Cu") (net 38))
+  (segment (start 120.46 150) (end 120.46 148) (width 0.5) (layer "B.Cu") (net 38))
+  (segment (start 79.54 123.46) (end 79.54 130) (width 0.5) (layer "B.Cu") (net 38))
+  (segment (start 79.54 148) (end 79.54 150) (width 0.5) (layer "B.Cu") (net 38))
+  (segment (start 120.46 148) (end 120.46 130) (width 0.5) (layer "B.Cu") (net 38))
+  (segment (start 79.54 130) (end 79.54 148) (width 0.5) (layer "B.Cu") (net 38))
+  (segment (start 79.54 148) (end 120.46 148) (width 0.5) (layer "B.Cu") (net 38))
   (zone (net 5) (net_name "batt.gnd") (layers "F&B.Cu") (hatch edge 0.508)
     (connect_pads (clearance 0.254))

Commit message: cleaning pinning
Parts:
- moved ledr.package 20.6 mm to (118.0, 115.0)
- moved ledr.res 20.6 mm to (122.0, 115.0)
- moved ledw.package 2.00 mm to (113.0, 97.0)
- moved ledw.res 2.00 mm to (117.0, 97.0)
- moved ledy.package 2.00 mm to (113.0, 95.0)
- moved ledy.res 2.00 mm to (117.0, 95.0)
Changed lines of the file:
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@@
   )
   (footprint "LED_SMD:LED_0603_1608Metric" (layer "F.Cu")
-    (at 113 97 180)
+    (at 113 95 180)
     (descr "LED SMD 0603 (1608 Metric), square (rectangular) end terminal, IPC_7351 nominal, (Body size source: http://www.tortai-tech.com/upload/download/2011102023233369053.pdf), generated with kicad-footprint-generator")
     (tags "LED")
@@
   )
   (footprint "LED_SMD:LED_0603_1608Metric" (layer "F.Cu")
-    (at 113 95 180)
+    (at 118 115 180)
     (descr "LED SMD 0603 (1608 Metric), square (rectangular) end terminal, IPC_7351 nominal, (Body size source: http://www.tortai-tech.com/upload/download/2011102023233369053.pdf), generated with kicad-footprint-generator")
     (tags "LED")
@@
   )
   (footprint "Resistor_SMD:R_0603_1608Metric" (layer "F.Cu")
-    (at 117 97)
+    (at 117 95)
     (descr "Resistor SMD 0603 (1608 Metric), square (rectangular) end terminal, IPC_7351 nominal, (Body size source: IPC-SM-782 page 72, https://www.pcb-3d.com/wordpress/wp-content/uploads/ipc-sm-782a_amendment_1_and_2.pdf), generated with kicad-footprint-generator")
     (tags "resistor")
@@
   )
   (footprint "Resistor_SMD:R_0603_1608Metric" (layer "F.Cu")
-    (at 117 95)
+    (at 122 115)
     (descr "Resistor SMD 0603 (1608 Metric), square (rectangular) end terminal, IPC_7351 nominal, (Body size source: IPC-SM-782 page 72, https://www.pcb-3d.com/wordpress/wp-content/uploads/ipc-sm-782a_amendment_1_and_2.pdf), generated with kicad-footprint-generator")
     (tags "resistor")
@@
   )
   (footprint "LED_SMD:LED_0603_1608Metric" (layer "F.Cu")
-    (at 113 99 180)
+    (at 113 97 180)
     (descr "LED SMD 0603 (1608 Metric), square (rectangular) end terminal, IPC_7351 nominal, (Body size source: http://www.tortai-tech.com/upload/download/2011102023233369053.pdf), generated with kicad-footprint-generator")
     (tags "LED")
@@
   )
   (footprint "Resistor_SMD:R_0603_1608Metric" (layer "F.Cu")
-    (at 117 99)
+    (at 117 97)
     (descr "Resistor SMD 0603 (1608 Metric), square (rectangular) end terminal, IPC_7351 nominal, (Body size source: IPC-SM-782 page 72, https://www.pcb-3d.com/wordpress/wp-content/uploads/ipc-sm-782a_amendment_1_and_2.pdf), generated with kicad-footprint-generator")
     (tags "resistor")

Commit message: preroute
Routing:
- net mcu.program_uart_node.b_tx: track 0.00 -> 3.78 mm
- net mcu.program_en_node: track 0.00 -> 3.08 mm
- net batt.gnd: track 0.00 -> 3.08 mm
- net mcu.program_boot_node: track 0.00 -> 2.88 mm
- net imu.pwr: track 79.1 -> 82.0 mm
- net mcu.program_uart_node.a_tx: track 0.00 -> 2.78 mm
Changed lines of the file:
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@@
   (gr_line (start 75 98) (end 75 150)
     (stroke (width 0.0381) (type default)) (layer "Edge.Cuts"))
+  (segment (start 119.365 107.73) (end 118.970998 107.73) (width 0.16) (layer "F.Cu") (net 1))
+  (segment (start 117.240998 106) (end 117 106) (width 0.16) (layer "F.Cu") (net 1))
+  (segment (start 118.970998 107.73) (end 117.240998 106) (width 0.16) (layer "F.Cu") (net 1))
   (segment (start 85 97) (end 78 97) (width 0.5) (layer "F.Cu") (net 2))
   (segment (start 80.525 95) (end 79 95) (width 0.5) (layer "F.Cu") (net 2))
@@
   (segment (start 86.175 97) (end 85 97) (width 0.5) (layer "F.Cu") (net 2))
   (segment (start 84 118) (end 84 121) (width 0.5) (layer "F.Cu") (net 2))
+  (segment (start 120.635 110.27) (end 121 110.635) (width 0.16) (layer "F.Cu") (net 2))
   (segment (start 78 112) (end 84 118) (width 0.5) (layer "F.Cu") (net 2))
   (segment (start 93 130) (end 99.85 130) (width 0.5) (layer "F.Cu") (net 2))
   (segment (start 99 130) (end 99.85 130) (width 0.5) (layer "F.Cu") (net 2))
   (segment (start 90 96) (end 90.01 96.01) (width 0.5) (layer "F.Cu") (net 2))
+  (segment (start 121 110.635) (end 121 113) (width 0.16) (layer "F.Cu") (net 2))
   (segment (start 99.85 130) (end 106.15 130) (width 0.5) (layer "F.Cu") (net 2))
   (segment (start 84 121) (end 93 130) (width 0.5) (layer "F.Cu") (net 2))
@@
   (segment (start 79 95) (end 78 96) (width 0.5) (layer "F.Cu") (net 2))
   (segment (start 78 96) (end 78 97) (width 0.5) (layer "F.Cu") (net 2))
+  (segment (start 122.759002 106) (end 123 106) (width 0.16) (layer "F.Cu") (net 5))
+  (segment (start 120.635 107.73) (end 121.029002 107.73) (width 0.16) (layer "F.Cu") (net 5))
+  (segment (start 121.029002 107.73) (end 122.759002 106) (width 0.16) (layer "F.Cu") (net 5))
+  (segment (start 119.365 110.27) (end 119 110.635) (width 0.16) (layer "F.Cu") (net 15))
+  (segment (start 119 110.635) (end 119 113) (width 0.16) (layer "F.Cu") (net 15))
+  (segment (start 119.365 109) (end 118.365 110) (width 0.16) (layer "F.Cu") (net 19))
+  (segment (start 118 110) (end 116 110) (width 0.16) (layer "F.Cu") (net 19))
+  (segment (start 118.365 110) (end 118 110) (width 0.16) (layer "F.Cu") (net 19))
+  (segment (start 120.635 109) (end 121.635 110) (width 0.16) (layer "F.Cu") (net 20))
+  (segment (start 121.635 110) (end 123 110) (width 0.16) (layer "F.Cu") (net 20))
   (segment (start 82 121) (end 91 130) (width 0.5) (layer "F.Cu") (net 38))
   (segment (start 96 134) (end 97.3 132.7) (width 0.5) (layer "F.Cu") (net 38))

Commit message: prerouting
Parts:
- turned sw to 0 degrees
Routing:
- net batt.gnd: track 3.08 -> 169.9 mm, vias 0 -> 7
- net batt.pwr: track 117.9 -> 120.2 mm
- net imu.pwr: vias 0 -> 1
Changed lines of the file:
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@@
   )
   (footprint "Button_Switch_SMD:SW_SPST_SKQG_WithoutStem" (layer "F.Cu")
-    (at 120 120 180)
+    (at 120 120)
     (descr "ALPS 5.2mm Square Low-profile Type (Surface Mount) SKQG Series, Without stem, http://www.alps.com/prod/info/E/HTML/Tact/SurfaceMount/SKQG/SKQGAEE010.html")
     (tags "SPST Button Switch")
@@
     (fp_circle (center 0 0) (end 1.5 0)
       (stroke (width 0.1) (type solid)) (fill none) (layer "F.Fab"))
-    (pad "1" smd rect (at -3.1 -1.85 180) (size 1.8 1.1) (layers "F.Cu" "F.Paste" "F.Mask")
+    (pad "1" smd rect (at -3.1 -1.85) (size 1.8 1.1) (layers "F.Cu" "F.Paste" "F.Mask")
       (net 13 "sw.out"))
-    (pad "1" smd rect (at 3.1 -1.85 180) (size 1.8 1.1) (layers "F.Cu" "F.Paste" "F.Mask")
+    (pad "1" smd rect (at 3.1 -1.85) (size 1.8 1.1) (layers "F.Cu" "F.Paste" "F.Mask")
       (net 13 "sw.out"))
-    (pad "2" smd rect (at -3.1 1.85 180) (size 1.8 1.1) (layers "F.Cu" "F.Paste" "F.Mask")
+    (pad "2" smd rect (at -3.1 1.85) (size 1.8 1.1) (layers "F.Cu" "F.Paste" "F.Mask")
       (net 5 "batt.gnd"))
-    (pad "2" smd rect (at 3.1 1.85 180) (size 1.8 1.1) (layers "F.Cu" "F.Paste" "F.Mask")
+    (pad "2" smd rect (at 3.1 1.85) (size 1.8 1.1) (layers "F.Cu" "F.Paste" "F.Mask")
       (net 5 "batt.gnd"))
     (zone (net 0) (net_name "") (layer "F.Cu") (hatch full 0.508)
@@
       (polygon
         (pts
+          (xy 116 118.7)
+          (xy 119 118.7)
           (xy 119 121.3)
           (xy 116 121.3)
-          (xy 116 118.7)
-          (xy 119 118.7)
         )
       )
@@
       (polygon
         (pts
+          (xy 121 118.7)
+          (xy 124 118.7)
           (xy 124 121.3)
           (xy 121 121.3)
-          (xy 121 118.7)
-          (xy 124 118.7)
         )
       )
@@
   (segment (start 79 95) (end 78 96) (width 0.5) (layer "F.Cu") (net 2))
   (segment (start 78 96) (end 78 97) (width 0.5) (layer "F.Cu") (net 2))
+  (via (at 121 113) (size 0.6) (drill 0.3) (layers "F.Cu" "B.Cu") (net 2))
+  (segment (start 82 119) (end 77 114) (width 0.5) (layer "F.Cu") (net 5))
+  (segment (start 94.05 128) (end 93 128) (width 0.5) (layer "F.Cu") (net 5))
+  (segment (start 94.225 132) (end 93 132) (width 0.5) (layer "F.Cu") (net 5))
   (segment (start 122.759002 106) (end 123 106) (width 0.16) (layer "F.Cu") (net 5))
+  (segment (start 86.225 99) (end 85 99) (width 0.5) (layer "F.Cu") (net 5))
+  (segment (start 83.475 95) (end 86.225 95) (width 0.5) (layer "F.Cu") (net 5))
+  (segment (start 99.85 127.7) (end 98.7 127.7) (width 0.5) (layer "F.Cu") (net 5))
+  (segment (start 91.25 94.74) (end 92.74 94.74) (width 0.5) (layer "F.Cu") (net 5))
   (segment (start 120.635 107.73) (end 121.029002 107.73) (width 0.16) (layer "F.Cu") (net 5))
+  (segment (start 77 114) (end 77 96) (width 0.5) (layer "F.Cu") (net 5))
+  (segment (start 98.7 127.7) (end 98 127) (width 0.5) (layer "F.Cu") (net 5))
   (segment (start 121.029002 107.73) (end 122.759002 106) (width 0.16) (layer "F.Cu") (net 5))
+  (segment (start 92.74 94.74) (end 93 95) (width 0.5) (layer "F.Cu") (net 5))
+  (via (at 93 128) (size 0.6) (drill 0.3) (layers "F.Cu" "B.Cu") (net 5))
+  (via (at 93 95) (size 0.6) (drill 0.3) (layers "F.Cu" "B.Cu") (net 5))
+  (via (at 98 127) (size 0.6) (drill 0.3) (layers "F.Cu" "B.Cu") (net 5))
+  (via (at 93 132) (size 0.6) (drill 0.3) (layers "F.Cu" "B.Cu") (net 5))
+  (via (at 85 99) (size 0.6) (drill 0.3) (layers "F.Cu" "B.Cu") (net 5))
+  (via (at 85 95) (size 0.6) (drill 0.3) (layers "F.Cu" "B.Cu") (net 5))
+  (via (at 77 96) (size 0.6) (drill 0.3) (layers "F.Cu" "B.Cu") (net 5))
+  (segment (start 85 95) (end 78 95) (width 0.5) (layer "B.Cu") (net 5))
+  (segment (start 93 128) (end 97 128) (width 0.5) (layer "B.Cu") (net 5))
+  (segment (start 82 124) (end 82 145) (width 0.5) (layer "B.Cu") (net 5))
+  (segment (start 97 128) (end 98 127) (width 0.5) (layer "B.Cu") (net 5))
+  (segment (start 93 128) (end 93 132) (width 0.5) (layer "B.Cu") (net 5))
+  (segment (start 82 145) (end 82 145.92) (width 0.5) (layer "B.Cu") (net 5))
+  (segment (start 82 119) (end 83 119) (width 0.5) (layer "B.Cu") (net 5))
+  (segment (start 82 145.92) (end 82.08 146) (width 0.5) (layer "B.Cu") (net 5))
+  (segment (start 83 119) (end 84 120) (width 0.5) (layer "B.Cu") (net 5))
+  (segment (start 82 149.92) (end 82.08 150) (width 0.5) (layer "B.Cu") (net 5))
+  (segment (start 84 120) (end 84 122) (width 0.5) (layer "B.Cu") (net 5))
+  (segment (start 82 145) (end 82 149.92) (width 0.5) (layer "B.Cu") (net 5))
+  (segment (start 84 122) (end 90 128) (width 0.5) (layer "B.Cu") (net 5))
+  (segment (start 84 122) (end 82 124) (width 0.5) (layer "B.Cu") (net 5))
+  (segment (start 117.92 150) (end 117.92 130) (width 0.5) (layer "B.Cu") (net 5))
+  (segment (start 93 95) (end 85 95) (width 0.5) (layer "B.Cu") (net 5))
+  (segment (start 85 95) (end 85 99) (width 0.5) (layer "B.Cu") (net 5))
+  (segment (start 78 95) (end 77 96) (width 0.5) (layer "B.Cu") (net 5))
+  (segment (start 90 128) (end 93 128) (width 0.5) (layer "B.Cu") (net 5))
+  (segment (start 82.08 150) (end 117.92 150) (width 0.5) (layer "B.Cu") (net 5))
   (segment (start 119.365 110.27) (end 119 110.635) (width 0.16) (layer "F.Cu") (net 15))
   (segment (start 119 110.635) (end 119 113) (width 0.16) (layer "F.Cu") (net 15))
@@
   (segment (start 97.3 132.7) (end 97.3 132.3) (width 0.5) (layer "F.Cu") (net 38))
   (segment (start 97 132) (end 95.775 132) (width 0.5) (layer "F.Cu") (net 38))
+  (segment (start 81 152) (end 119 152) (width 0.5) (layer "B.Cu") (net 38))
   (segment (start 82 121) (end 79.54 123.46) (width 0.5) (layer "B.Cu") (net 38))
   (segment (start 120.46 150) (end 120.46 148) (width 0.5) (layer "B.Cu") (net 38))
   (segment (start 79.54 123.46) (end 79.54 130) (width 0.5) (layer "B.Cu") (net 38))
+  (segment (start 120.46 150.54) (end 120.46 150) (width 0.5) (layer "B.Cu") (net 38))
   (segment (start 79.54 148) (end 79.54 150) (width 0.5) (layer "B.Cu") (net 38))
   (segment (start 120.46 148) (end 120.46 130) (width 0.5) (layer "B.Cu") (net 38))
+  (segment (start 119 152) (end 120.46 150.54) (width 0.5) (layer "B.Cu") (net 38))
+  (segment (start 79.54 150) (end 79.54 150.54) (width 0.5) (layer "B.Cu") (net 38))
+  (segment (start 79.54 150.54) (end 81 152) (width 0.5) (layer "B.Cu") (net 38))
   (segment (start 79.54 130) (end 79.54 148) (width 0.5) (layer "B.Cu") (net 38))
-  (segment (start 79.54 148) (end 120.46 148) (width 0.5) (layer "B.Cu") (net 38))
   (zone (net 5) (net_name "batt.gnd") (layers "F&B.Cu") (hatch edge 0.508)
     (connect_pads (clearance 0.254))
@@
     (polygon
       (pts
-        (xy 126 156)
         (xy 74 156)
+        (xy 22 156)
+        (xy 22 92)
         (xy 74 92)
-        (xy 126 92)
       )
     )
