File: examples/RobotCrawler/CrawlerTimer.kicad_pcb (KiCad board)
At the start: 2 copper layers, 50 x 62 mm, 38 parts

Commit message: Update CrawlerTimer.kicad_pcb
Parts:
- moved jlc_th.th3 1.00 mm to (119.0, 153.0)
- moved servo_fs90fbs[0] 1.00 mm to (78.0, 130.0)
- moved servo_fs90fbs[1] 1.00 mm to (78.0, 134.0)
- moved servo_fs90fbs[2] 1.00 mm to (78.0, 138.0)
- moved servo_fs90fbs[3] 1.00 mm to (78.0, 142.0)
- moved servo_fs90fbs[4] 1.00 mm to (122.0, 130.0)
- moved servo_fs90fbs[5] 1.00 mm to (122.0, 134.0)
- moved servo_fs90fbs[6] 1.00 mm to (122.0, 138.0)
- moved servo_fs90fbs[7] 1.00 mm to (122.0, 142.0)
- moved servo_fs90rs[0] 1.00 mm to (78.0, 146.0)
- moved servo_fs90rs[1] 1.00 mm to (78.0, 150.0)
- moved servo_fs90rs[2] 1.00 mm to (122.0, 146.0)
- moved servo_fs90rs[3] 1.00 mm to (122.0, 150.0)
Routing:
- net batt.gnd: track 169.9 -> 167.4 mm
- net batt.pwr: track 120.2 -> 118.2 mm
- removed copper zone on B.Cu, net batt.gnd
- removed copper zone on F.Cu, net batt.gnd
Other:
- outline, holes or cut-outs redrawn
Changed lines of the file:
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@@
   (net 38 "batt.pwr")
   (footprint "Connector_PinHeader_2.54mm:PinHeader_1x04_P2.54mm_Vertical" (layer "F.Cu")
-    (at 123 134 -90)
+    (at 122 134 -90)
     (descr "Through hole straight pin header, 1x04, 2.54mm pitch, single row")
     (tags "Through hole pin header THT 1x04 2.54mm single row")
@@
   )
   (footprint "Connector_PinHeader_2.54mm:PinHeader_1x03_P2.54mm_Vertical" (layer "F.Cu")
-    (at 123 146 -90)
+    (at 122 146 -90)
     (descr "Through hole straight pin header, 1x03, 2.54mm pitch, single row")
     (tags "Through hole pin header THT 1x03 2.54mm single row")
@@
   )
   (footprint "Connector_PinHeader_2.54mm:PinHeader_1x03_P2.54mm_Vertical" (layer "F.Cu")
-    (at 77 150 90)
+    (at 78 150 90)
     (descr "Through hole straight pin header, 1x03, 2.54mm pitch, single row")
     (tags "Through hole pin header THT 1x03 2.54mm single row")
@@
   )
   (footprint "Connector_PinHeader_2.54mm:PinHeader_1x04_P2.54mm_Vertical" (layer "F.Cu")
-    (at 123 130 -90)
+    (at 122 130 -90)
     (descr "Through hole straight pin header, 1x04, 2.54mm pitch, single row")
     (tags "Through hole pin header THT 1x04 2.54mm single row")
@@
   )
   (footprint "Connector_PinHeader_2.54mm:PinHeader_1x04_P2.54mm_Vertical" (layer "F.Cu")
-    (at 77 134 90)
+    (at 78 134 90)
     (descr "Through hole straight pin header, 1x04, 2.54mm pitch, single row")
     (tags "Through hole pin header THT 1x04 2.54mm single row")
@@
   )
   (footprint "Connector_PinHeader_2.54mm:PinHeader_1x04_P2.54mm_Vertical" (layer "F.Cu")
-    (at 77 142 90)
+    (at 78 142 90)
     (descr "Through hole straight pin header, 1x04, 2.54mm pitch, single row")
     (tags "Through hole pin header THT 1x04 2.54mm single row")
@@
   )
   (footprint "Connector_PinHeader_2.54mm:PinHeader_1x04_P2.54mm_Vertical" (layer "F.Cu")
-    (at 123 138 -90)
+    (at 122 138 -90)
     (descr "Through hole straight pin header, 1x04, 2.54mm pitch, single row")
     (tags "Through hole pin header THT 1x04 2.54mm single row")
@@
   )
   (footprint "Connector_PinHeader_2.54mm:PinHeader_1x03_P2.54mm_Vertical" (layer "F.Cu")
-    (at 123 150 -90)
+    (at 122 150 -90)
     (descr "Through hole straight pin header, 1x03, 2.54mm pitch, single row")
     (tags "Through hole pin header THT 1x03 2.54mm single row")
@@
   )
   (footprint "Connector_PinHeader_2.54mm:PinHeader_1x04_P2.54mm_Vertical" (layer "F.Cu")
-    (at 77 130 90)
+    (at 78 130 90)
     (descr "Through hole straight pin header, 1x04, 2.54mm pitch, single row")
     (tags "Through hole pin header THT 1x04 2.54mm single row")
@@
   )
   (footprint "Connector_PinHeader_2.54mm:PinHeader_1x04_P2.54mm_Vertical" (layer "F.Cu")
-    (at 123 142 -90)
+    (at 122 142 -90)
     (descr "Through hole straight pin header, 1x04, 2.54mm pitch, single row")
     (tags "Through hole pin header THT 1x04 2.54mm single row")
@@
   )
   (footprint "Connector_PinHeader_2.54mm:PinHeader_1x03_P2.54mm_Vertical" (layer "F.Cu")
-    (at 77 146 90)
+    (at 78 146 90)
     (descr "Through hole straight pin header, 1x03, 2.54mm pitch, single row")
     (tags "Through hole pin header THT 1x03 2.54mm single row")
@@
   )
   (footprint "Connector_PinHeader_2.54mm:PinHeader_1x04_P2.54mm_Vertical" (layer "F.Cu")
-    (at 77 138 90)
+    (at 78 138 90)
     (descr "Through hole straight pin header, 1x04, 2.54mm pitch, single row")
     (tags "Through hole pin header THT 1x04 2.54mm single row")
@@
   )
   (footprint "edg:JlcToolingHole_1.152mm" (layer "F.Cu")
-    (at 120 153)
+    (at 119 153)
     (descr "Tooling holes for JLC assembly, 1.152 mm hole + 1.3mm soldermask opening")
     (property "Sheetfile" "edg.BoardTop.JlcToolingHoles")
@@
     )
   )
-  (gr_line (start 125 150) (end 125 98)
+  (gr_line (start 124 150) (end 124 98)
     (stroke (width 0.0381) (type default)) (layer "Edge.Cuts"))
   (gr_line (start 80 155) (end 120 155)
@@
   (gr_arc (start 120 93) (mid 123.535534 94.464466) (end 125 98)
     (stroke (width 0.0381) (type default)) (layer "Edge.Cuts"))
-  (gr_arc (start 125 150) (mid 123.535534 153.535534) (end 120 155)
+  (gr_arc (start 124 150) (mid 122.535534 153.535534) (end 119 155)
     (stroke (width 0.0381) (type default)) (layer "Edge.Cuts"))
   (gr_arc (start 75 98) (mid 76.464466 94.464466) (end 80 93)
@@
   (via (at 77 96) (size 0.6) (drill 0.3) (layers "F.Cu" "B.Cu") (net 5))
   (segment (start 85 95) (end 78 95) (width 0.5) (layer "B.Cu") (net 5))
+  (segment (start 84 122) (end 83 123) (width 0.5) (layer "B.Cu") (net 5))
   (segment (start 93 128) (end 97 128) (width 0.5) (layer "B.Cu") (net 5))
-  (segment (start 82 124) (end 82 145) (width 0.5) (layer "B.Cu") (net 5))
+  (segment (start 83 124) (end 83 145) (width 0.5) (layer "B.Cu") (net 5))
   (segment (start 97 128) (end 98 127) (width 0.5) (layer "B.Cu") (net 5))
   (segment (start 93 128) (end 93 132) (width 0.5) (layer "B.Cu") (net 5))
-  (segment (start 82 145) (end 82 145.92) (width 0.5) (layer "B.Cu") (net 5))
+  (segment (start 83 145) (end 83 145.92) (width 0.5) (layer "B.Cu") (net 5))
   (segment (start 82 119) (end 83 119) (width 0.5) (layer "B.Cu") (net 5))
-  (segment (start 82 145.92) (end 82.08 146) (width 0.5) (layer "B.Cu") (net 5))
+  (segment (start 83 145.92) (end 83.08 146) (width 0.5) (layer "B.Cu") (net 5))
   (segment (start 83 119) (end 84 120) (width 0.5) (layer "B.Cu") (net 5))
-  (segment (start 82 149.92) (end 82.08 150) (width 0.5) (layer "B.Cu") (net 5))
+  (segment (start 83 149.92) (end 83.08 150) (width 0.5) (layer "B.Cu") (net 5))
   (segment (start 84 120) (end 84 122) (width 0.5) (layer "B.Cu") (net 5))
-  (segment (start 82 145) (end 82 149.92) (width 0.5) (layer "B.Cu") (net 5))
+  (segment (start 83 145) (end 83 149.92) (width 0.5) (layer "B.Cu") (net 5))
   (segment (start 84 122) (end 90 128) (width 0.5) (layer "B.Cu") (net 5))
-  (segment (start 84 122) (end 82 124) (width 0.5) (layer "B.Cu") (net 5))
-  (segment (start 117.92 150) (end 117.92 130) (width 0.5) (layer "B.Cu") (net 5))
+  (segment (start 83.08 150) (end 116.92 150) (width 0.5) (layer "B.Cu") (net 5))
+  (segment (start 116.92 150) (end 116.92 130) (width 0.5) (layer "B.Cu") (net 5))
+  (segment (start 83 123) (end 83 124) (width 0.5) (layer "B.Cu") (net 5))
   (segment (start 93 95) (end 85 95) (width 0.5) (layer "B.Cu") (net 5))
   (segment (start 85 95) (end 85 99) (width 0.5) (layer "B.Cu") (net 5))
   (segment (start 78 95) (end 77 96) (width 0.5) (layer "B.Cu") (net 5))
   (segment (start 90 128) (end 93 128) (width 0.5) (layer "B.Cu") (net 5))
-  (segment (start 82.08 150) (end 117.92 150) (width 0.5) (layer "B.Cu") (net 5))
   (segment (start 119.365 110.27) (end 119 110.635) (width 0.16) (layer "F.Cu") (net 15))
   (segment (start 119 110.635) (end 119 113) (width 0.16) (layer "F.Cu") (net 15))
@@
   (segment (start 97.3 132.7) (end 97.3 132.3) (width 0.5) (layer "F.Cu") (net 38))
   (segment (start 97 132) (end 95.775 132) (width 0.5) (layer "F.Cu") (net 38))
-  (segment (start 81 152) (end 119 152) (width 0.5) (layer "B.Cu") (net 38))
   (segment (start 82 121) (end 79.54 123.46) (width 0.5) (layer "B.Cu") (net 38))
-  (segment (start 120.46 150) (end 120.46 148) (width 0.5) (layer "B.Cu") (net 38))
+  (segment (start 82 152) (end 118 152) (width 0.5) (layer "B.Cu") (net 38))
+  (segment (start 118 152) (end 119.46 150.54) (width 0.5) (layer "B.Cu") (net 38))
+  (segment (start 119.46 150) (end 119.46 148) (width 0.5) (layer "B.Cu") (net 38))
   (segment (start 79.54 123.46) (end 79.54 130) (width 0.5) (layer "B.Cu") (net 38))
-  (segment (start 120.46 150.54) (end 120.46 150) (width 0.5) (layer "B.Cu") (net 38))
-  (segment (start 79.54 148) (end 79.54 150) (width 0.5) (layer "B.Cu") (net 38))
-  (segment (start 120.46 148) (end 120.46 130) (width 0.5) (layer "B.Cu") (net 38))
-  (segment (start 119 152) (end 120.46 150.54) (width 0.5) (layer "B.Cu") (net 38))
-  (segment (start 79.54 150) (end 79.54 150.54) (width 0.5) (layer "B.Cu") (net 38))
-  (segment (start 79.54 150.54) (end 81 152) (width 0.5) (layer "B.Cu") (net 38))
-  (segment (start 79.54 130) (end 79.54 148) (width 0.5) (layer "B.Cu") (net 38))
-  (zone (net 5) (net_name "batt.gnd") (layers "F&B.Cu") (hatch edge 0.508)
-    (connect_pads (clearance 0.254))
-    (min_thickness 0.2) (filled_areas_thickness no)
-    (fill (thermal_gap 0.2) (thermal_bridge_width 0.2))
-    (polygon
-      (pts
-        (xy 74 156)
-        (xy 22 156)
-        (xy 22 92)
-        (xy 74 92)
-      )
-    )
-  )
+  (segment (start 80.54 148) (end 80.54 150) (width 0.5) (layer "B.Cu") (net 38))
+  (segment (start 119.46 148) (end 119.46 130) (width 0.5) (layer "B.Cu") (net 38))
+  (segment (start 80.54 150) (end 80.54 150.54) (width 0.5) (layer "B.Cu") (net 38))
+  (segment (start 80.54 150.54) (end 82 152) (width 0.5) (layer "B.Cu") (net 38))
+  (segment (start 80.54 130) (end 80.54 148) (width 0.5) (layer "B.Cu") (net 38))
+  (segment (start 119.46 150.54) (end 119.46 150) (width 0.5) (layer "B.Cu") (net 38))
 )

Commit message: Update CrawlerTimer.kicad_pcb
Parts:
- moved ledw.package 1.00 mm to (113.0, 98.0)
- moved ledw.res 1.00 mm to (117.0, 98.0)
- moved ledy.package 1.00 mm to (113.0, 96.0)
- moved ledy.res 1.00 mm to (117.0, 96.0)
Other:
- outline, holes or cut-outs redrawn
Changed lines of the file:
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@@
   )
   (footprint "LED_SMD:LED_0603_1608Metric" (layer "F.Cu")
-    (at 113 95 180)
+    (at 113 96 180)
     (descr "LED SMD 0603 (1608 Metric), square (rectangular) end terminal, IPC_7351 nominal, (Body size source: http://www.tortai-tech.com/upload/download/2011102023233369053.pdf), generated with kicad-footprint-generator")
     (tags "LED")
@@
   )
   (footprint "Resistor_SMD:R_0603_1608Metric" (layer "F.Cu")
-    (at 117 95)
+    (at 117 96)
     (descr "Resistor SMD 0603 (1608 Metric), square (rectangular) end terminal, IPC_7351 nominal, (Body size source: IPC-SM-782 page 72, https://www.pcb-3d.com/wordpress/wp-content/uploads/ipc-sm-782a_amendment_1_and_2.pdf), generated with kicad-footprint-generator")
     (tags "resistor")
@@
   )
   (footprint "LED_SMD:LED_0603_1608Metric" (layer "F.Cu")
-    (at 113 97 180)
+    (at 113 98 180)
     (descr "LED SMD 0603 (1608 Metric), square (rectangular) end terminal, IPC_7351 nominal, (Body size source: http://www.tortai-tech.com/upload/download/2011102023233369053.pdf), generated with kicad-footprint-generator")
     (tags "LED")
@@
   )
   (footprint "Resistor_SMD:R_0603_1608Metric" (layer "F.Cu")
-    (at 117 97)
+    (at 117 98)
     (descr "Resistor SMD 0603 (1608 Metric), square (rectangular) end terminal, IPC_7351 nominal, (Body size source: IPC-SM-782 page 72, https://www.pcb-3d.com/wordpress/wp-content/uploads/ipc-sm-782a_amendment_1_and_2.pdf), generated with kicad-footprint-generator")
     (tags "resistor")
@@
     )
   )
-  (gr_line (start 124 150) (end 124 98)
+  (gr_line (start 125 150) (end 125 98)
     (stroke (width 0.0381) (type default)) (layer "Edge.Cuts"))
   (gr_line (start 80 155) (end 120 155)
@@
   (gr_arc (start 120 93) (mid 123.535534 94.464466) (end 125 98)
     (stroke (width 0.0381) (type default)) (layer "Edge.Cuts"))
-  (gr_arc (start 124 150) (mid 122.535534 153.535534) (end 119 155)
+  (gr_arc (start 125 150) (mid 123.535534 153.535534) (end 120 155)
     (stroke (width 0.0381) (type default)) (layer "Edge.Cuts"))
   (gr_arc (start 75 98) (mid 76.464466 94.464466) (end 80 93)

Commit message: just one copper duck given
Routing:
- net batt.gnd: track 167.4 -> 277.2 mm
- net servo_fs90fbs[7].pwm: track 0.00 -> 68.0 mm
- net servo_fs90rs[2].pwm: track 0.00 -> 62.7 mm
- net imu.pwr: track 82.0 -> 138.0 mm, vias 1 -> 2
- net servo_fs90rs[3].pwm: track 0.00 -> 55.0 mm
- net servo_fs90fbs[1].fb: track 0.00 -> 51.9 mm, vias 0 -> 1
- net servo_fs90fbs[2].fb: track 0.00 -> 51.7 mm, vias 0 -> 1
- net servo_fs90fbs[7].fb: track 0.00 -> 50.8 mm, vias 0 -> 2
- net servo_fs90fbs[3].fb: track 0.00 -> 50.1 mm, vias 0 -> 1
- net servo_fs90fbs[0].fb: track 0.00 -> 48.7 mm, vias 0 -> 1
- net servo_fs90rs[1].pwm: track 0.00 -> 48.0 mm, vias 0 -> 2
- net servo_fs90fbs[6].pwm: track 0.00 -> 46.7 mm, vias 0 -> 1
- net servo_fs90rs[0].pwm: track 0.00 -> 46.0 mm, vias 0 -> 1
- net servo_fs90fbs[3].pwm: track 0.00 -> 45.5 mm, vias 0 -> 2
- net servo_fs90fbs[6].fb: track 0.00 -> 44.9 mm, vias 0 -> 2
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- added copper zone on B.Cu, net batt.gnd
- added copper zone on F.Cu, net batt.gnd
