File: examples/EspLora/EspLora.kicad_pcb (KiCad board)
At the start: 2 copper layers, 63 x 39 mm, 75 parts

Commit message: Update EspLora.kicad_pcb
Routing:
- net Lgnd: vias 70 -> 73
Changed lines of the file:
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@@
+	)
+	(via
+		(at 165 123.5875)
+		(size 0.7)
+		(drill 0.3)
+		(layers "F.Cu" "B.Cu")
+		(net 2)
 	)
 	(via
@@
 	)
 	(via
+		(at 167 123.575)
+		(size 0.7)
+		(drill 0.3)
+		(layers "F.Cu" "B.Cu")
+		(net 2)
+	)
+	(via
 		(at 188.5 122.5)
 		(size 0.7)
@@
 	)
 	(via
+		(at 163 123.575)
+		(size 0.7)
+		(drill 0.3)
+		(layers "F.Cu" "B.Cu")
+		(net 2)
+	)
+	(via
 		(at 185.5 122.5)
 		(size 0.7)
@@
 	)
 	(via
+		(at 169 123.575)
+		(size 0.7)
+		(drill 0.3)
+		(layers "F.Cu" "B.Cu")
+		(net 2)
+	)
+	(via
 		(at 170 118)
 		(size 0.7)
@@
 		(size 0.7)
 		(drill 0.3)
-		(layers "F.Cu" "B.Cu")
-		(net 2)
-	)
-	(via
-		(at 169 123)
-		(size 0.7)
-		(drill 0.3)

Commit message: wip
Parts:
- moved tp_lora_cs 39.2 mm to (162.0, 126.0), turned to 90 degrees
- moved tp_lora_spi.tp_sck 30.8 mm to (160.0, 126.0), turned to 90 degrees
- moved tp_lora_rst 30.5 mm to (154.0, 126.0), turned to 90 degrees
- moved tp_lora_dio 28.8 mm to (152.0, 126.0), turned to 90 degrees
- moved tp_lora_spi.tp_mosi 28.3 mm to (158.0, 126.0), turned to 90 degrees
- moved tp_lora_spi.tp_miso 26.0 mm to (156.0, 126.0), turned to 90 degrees
- moved tp_gnd 22.2 mm to (170.0, 114.0)
- turned ledb.res to 180 degrees
- turned ledg.res to 180 degrees
- turned ledr.res to 180 degrees
Connections:
- choke pad 1: Lpwr -> Lusb.pwr
- choke pad 2: Lchoke.pwr_out -> Lpwr
- reg_3v3.ic pad 3: Lchoke.pwr_out -> Lpwr
- reg_3v3.in_cap pad 1: Lchoke.pwr_out -> Lpwr
- usb.conn pad A4: Lpwr -> Lusb.pwr
- usb.conn pad A9: Lpwr -> Lusb.pwr
- usb.conn pad B4: Lpwr -> Lusb.pwr
- usb.conn pad B9: Lpwr -> Lusb.pwr
Routing:
- net Lv3v3: track 52.8 -> 68.3 mm, vias 4 -> 6
- net Lmcu.program_boot_node: track 0.00 -> 14.9 mm, vias 0 -> 1
- net Ltp_lora_dio.io: track 0.00 -> 10.0 mm, vias 0 -> 1
- net Ltp_lora_rst.io: track 0.00 -> 8.99 mm, vias 0 -> 1
- net Ltp_lora_spi.io.miso: track 0.00 -> 7.21 mm
- net Lpwr: track 0.00 -> 6.93 mm
- net Ltp_lora_cs.io: track 0.00 -> 5.37 mm
- net Ltp_lora_spi.io.mosi: track 0.00 -> 5.20 mm
- net Ltp_lora_spi.io.sck: track 0.00 -> 4.58 mm
- net Lmcu.program_uart_node.b_tx: track 0.00 -> 3.45 mm, vias 0 -> 2
- net Lmcu.program_uart_node.a_tx: track 0.00 -> 3.34 mm, vias 0 -> 2
- net Lledr.res.a: track 0.00 -> 2.75 mm
- net Lledg.res.a: track 0.00 -> 2.75 mm
- net Lledb.res.a: track 0.00 -> 2.75 mm
- net Lmcu.program_en_node: track 8.25 -> 9.25 mm, vias 0 -> 1
- added copper zone on F.Cu, net Lusb.pwr
- removed copper zone on F.Cu, net Lpwr

Commit message: Update EspLora.kicad_pcb
Routing:
- net Lusb_chain_0.d_N: track 6.83 -> 35.8 mm, vias 1 -> 2
- net Lusb_chain_0.d_P: track 6.81 -> 33.9 mm, vias 1 -> 2
- net Lv3v3: track 68.3 -> 95.1 mm, vias 6 -> 7
- net Ltp_lora_spi.io.sck: track 4.58 -> 29.3 mm, vias 0 -> 2
- net Llora.rf_sw.ctrl: track 1.67 -> 24.9 mm, vias 1 -> 2
- net Ltp_lora_spi.io.mosi: track 5.20 -> 26.8 mm, vias 0 -> 2
- net Ltp_lora_rst.io: track 8.99 -> 29.0 mm, vias 1 -> 2
- net Ltp_lora_spi.io.miso: track 7.21 -> 25.7 mm, vias 0 -> 2
- net Ltp_lora_cs.io: track 5.37 -> 23.0 mm, vias 0 -> 2
- net Lmcu.program_uart_node.a_tx: track 3.34 -> 17.7 mm
- net Lmcu.program_uart_node.b_tx: track 3.45 -> 14.4 mm
- net Lgnd: track 13.3 -> 16.0 mm, vias 73 -> 75

Commit message: Update EspLora.kicad_pcb
Routing:
- net Lmcu.program_en_node: track 9.25 -> 39.4 mm, vias 1 -> 2
- net Lv3v3: track 95.1 -> 98.4 mm
- net Lgnd: track 16.0 -> 18.4 mm, vias 75 -> 76
- net Ltp_lora_spi.io.miso: track 25.7 -> 27.0 mm
- net Ltp_lora_spi.io.sck: track 29.3 -> 28.2 mm
- net Ltp_lora_spi.io.mosi: track 26.8 -> 26.2 mm

Commit message: Update EspLora.kicad_pcb
Routing:
- net Ltp_lora_dio.io: track 10.0 -> 22.1 mm, vias 1 -> 0
- net Ltp_lora_spi.io.sck: track 28.2 -> 25.0 mm
- net Ltp_lora_rst.io: track 29.0 -> 31.0 mm
- net Ltp_lora_cs.io: track 23.0 -> 22.5 mm

Commit message: wip
Parts:
- moved jlc_th.th3 75.9 mm to (198.0, 134.0)
- moved jlc_th.th1 71.4 mm to (198.5, 111.5)
- moved jlc_th.th2 30.3 mm to (139.0, 130.5)
- moved i2c_pull.sda_res 8.94 mm to (174.0, 135.0), turned to -90 degrees
- moved i2c_pull.scl_res 5.66 mm to (176.0, 135.0), turned to -90 degrees
- moved lora.ant 0.50 mm to (195.5, 120.0)
Connections:
- mcu.ic pad 17: Lledb.signal -> (no net)
- mcu.ic pad 34: (no net) -> Lledr.signal
- mcu.ic pad 35: (no net) -> Lledg.signal
- mcu.ic pad 39: Lledr.signal -> Lledb.signal
- mcu.ic pad 4: Lledg.signal -> (no net)
Routing:
- net Lv3v3: track 98.4 -> 232.5 mm, vias 7 -> 10
- net Lsd.cs: track 0.00 -> 45.5 mm, vias 0 -> 2
- net Lsd.spi.mosi: track 0.00 -> 44.3 mm, vias 0 -> 2
- net Lsd.spi.sck: track 0.00 -> 44.1 mm, vias 0 -> 2
- net Lsd.spi.miso: track 0.00 -> 42.8 mm, vias 0 -> 2
- net Li2c_pull.i2c.scl: track 0.00 -> 24.5 mm, vias 0 -> 2
- net Li2c_pull.i2c.sda: track 0.00 -> 23.2 mm
- net Loled_rst.nreset: track 0.00 -> 14.3 mm, vias 0 -> 2
- net Lmcu.program_boot_node: track 14.9 -> 27.5 mm, vias 1 -> 0
- net Lledg.signal: track 0.00 -> 4.91 mm
- net Lledr.signal: track 0.00 -> 3.32 mm
- net Lledb.signal: track 0.00 -> 2.88 mm
- net Lgnd: track 18.4 -> 20.1 mm, vias 76 -> 101
- net Lusb_chain_0.d_N: track 35.8 -> 35.0 mm
- net Ltp_lora_dio.io: track 22.1 -> 22.4 mm, vias 0 -> 2
Other:
- outline, holes or cut-outs redrawn

Commit message: Update EspLora.kicad_pcb
Parts:
- renumbered reg_3v3.in_cap to LC1, lora.vrpa_cap1 to LC10, lora.tx_dcblock to LC11, lora.rfc_dcblock to LC12, lora.tx_l.c_lc to LC13, lora.tx_pi.c2 to LC14, lora.balun.c to LC15, lora.balun.c_p to LC16, lora.ant_pi.c1 to LC17, lora.ant_pi.c2 to LC18, oled.c1_cap to LC19, reg_3v3.out_cap to LC2, oled.c2_cap to LC20, oled.vcomh_cap to LC21, oled.vdd_cap1 to LC22, oled.vbat_cap to LC23, oled.vcc_cap to LC24, tx_cpack to LC25, mcu.vcc_cap0 to LC3, mcu.vcc_cap1 to LC4, mcu.en_pull.c to LC5, lora.vreg_cap to LC6, lora.vbat_cap to LC7, lora.vdd_cap to LC8, lora.vrpa_cap0 to LC9, prot_3v3 to LD1, ledr.package to LD2, ledg.package to LD3, ledb.package to LD4, choke to LFB1, jlc_th.th1 to LH1, jlc_th.th2 to LH2, jlc_th.th3 to LH3, usb.conn to LJ1, mcu.prog to LJ2, lora.ant to LJ3, oled.device to LJ4, sd to LJ5, lora.dcc_l to LL1, lora.vrpa_choke to LL2, lora.tx_l.l to LL3, lora.tx_pi.l to LL4, lora.balun.l to LL5, lora.ant_pi.l to LL6, usb.cc_pull.cc1 to LR1, i2c_pull.scl_res to LR10, i2c_pull.sda_res to LR11, oled_pull to LR12, usb.cc_pull.cc2 to LR2, mcu.en_pull.r to LR3, ledr.res to LR4, ledg.res to LR5, ledb.res to LR6, lora.rf_sw.vdd_res to LR7, lora.rf_sw.ctrl_res to LR8, oled.iref_res to LR9, mcu.boot to LSW1, tp_gnd to LTP1, tp_pwr to LTP2, tp_3v3 to LTP3, tp_lora_spi.tp_sck to LTP4, tp_lora_spi.tp_mosi to LTP5, tp_lora_spi.tp_miso to LTP6, tp_lora_cs to LTP7, tp_lora_rst to LTP8, tp_lora_dio to LTP9, reg_3v3.ic to LU1, mcu.ic to LU2, usb_esd to LU3, lora.ic to LU4, lora.rf_sw.ic to LU5, oled.lcd to LU6, oled_rst to LU7, lora.xtal to LX1
Routing:
- net Ltp_lora_rst.io: track 31.0 -> 31.9 mm
