File: examples/CanAdapter/CanAdapter.kicad_pcb (KiCad board)
At the start: 2 copper layers, 46 x 22 mm, 27 parts

Commit message: final fabrication data
Parts:
- added OFB1: 200mA 1 450m? 600?@100MHz ±25% 0603 Ferrite Beads ROHS, Inductor_SMD:L_0603_1608Metric, F.Cu at (117.0, 99.0)
- added OH1: , edg:JlcToolingHole_1.152mm, F.Cu at (118.0, 104.0)
- added OH2: , edg:JlcToolingHole_1.152mm, F.Cu at (101.0, 92.0)
- added OH3: , edg:JlcToolingHole_1.152mm, F.Cu at (119.5, 96.0)
- OC1, OC2, OC6, OC8: value 100nF -> 50V 100nF X7R ±10% 0603 Multilayer Ceramic Capacitors MLCC - SMD/SMT ROHS
- OC3: value 10uF -> 25V 22uF X5R ±10% 1206 Multilayer Ceramic Capacitors MLCC - SMD/SMT ROHS; footprint Capacitor_SMD:C_1210_3225Metric -> Capacitor_SMD:C_1206_3216Metric
- OC4, OC5: value 10uF -> X5R 25V ±10% 10uF 0805 Multilayer Ceramic Capacitors MLCC - SMD/SMT ROHS
- OC7: value 1uF -> 50V 1uF X5R ±10% 0603 Multilayer Ceramic Capacitors MLCC - SMD/SMT ROHS
- OD2: value LED -> Red 615~630nm 1.9~2.2V 0603 Light Emitting Diodes (LED) RoHS
- OD3: value LED -> 20mA 285mcd 3.3V 518nm Colorless transparence -40?~+85? 520nm~535nm Emerald 120° 110mW 0603 Light Emitting Diodes (LED)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
- OD4: value LED -> White 0603 Light Emitting Diodes (LED) RoHS
- OR1: value 6.8k, 1%, 0.1 W -> ±1% 1/10W Thick Film Resistors 75V ±100ppm/? -55?~+155? 6.8k? 0603 Chip Resistor - Surface Mount ROHS
- OR2: value 1.5k, 1%, 0.1 W -> ±1% 1/10W Thick Film Resistors 75V ±100ppm/? -55?~+155? 1.5k? 0603 Chip Resistor - Surface Mount ROHS
- OR3: value 510k, 1%, 0.1 W -> ±1% 1/10W Thick Film Resistors 75V ±100ppm/? -55?~+155? 510k? 0603 Chip Resistor - Surface Mount ROHS
- OR4, OR9: value 10k, 1%, 0.1 W -> ±1% 1/10W Thick Film Resistors 75V ±100ppm/? -55?~+155? 10k? 0603 Chip Resistor - Surface Mount ROHS
- OR5, OR6, OR7: value 1k, 1%, 0.1 W -> ±1% 1/10W Thick Film Resistors 75V ±100ppm/? -55?~+155? 1k? 0603 Chip Resistor - Surface Mount ROHS
- OR8: value 100k, 1%, 0.1 W -> ±1% 1/10W Thick Film Resistors 75V ±100ppm/? -55?~+155? 91k? 0603 Chip Resistor - Surface Mount ROHS
- moved OC3 1.00 mm to (115.0, 103.0)
Connections:
- OU1 pad 16: Ovobd -> Oobd.pwr
Routing:
- net Ovobd: track 17.6 -> 25.2 mm, vias 2 -> 0
- net Oobd.pwr: track 0.00 -> 6.83 mm, vias 0 -> 1
- net Ov3v3: track 145.0 -> 145.7 mm

Commit message: update boards
Parts:
- OC1: value 50V 100nF X7R ±10% 0603 Multilayer Ceramic Capacitors MLCC - SMD/SMT ROHS -> reg_3v3.hf_in_cap
- OC2: value 50V 100nF X7R ±10% 0603 Multilayer Ceramic Capacitors MLCC - SMD/SMT ROHS -> reg_3v3.boot_cap
- OC3: value 25V 22uF X5R ±10% 1206 Multilayer Ceramic Capacitors MLCC - SMD/SMT ROHS -> reg_3v3.power_path.in_cap
- OC4: value X5R 25V ±10% 10uF 0805 Multilayer Ceramic Capacitors MLCC - SMD/SMT ROHS -> reg_3v3.power_path.out_cap
- OC5: value X5R 25V ±10% 10uF 0805 Multilayer Ceramic Capacitors MLCC - SMD/SMT ROHS -> mcu.vcc_cap0
- OC6: value 50V 100nF X7R ±10% 0603 Multilayer Ceramic Capacitors MLCC - SMD/SMT ROHS -> mcu.vcc_cap1
- OC7: value 50V 1uF X5R ±10% 0603 Multilayer Ceramic Capacitors MLCC - SMD/SMT ROHS -> mcu.en_pull.c
- OC8: value 50V 100nF X7R ±10% 0603 Multilayer Ceramic Capacitors MLCC - SMD/SMT ROHS -> can.vdd_cap
- OD1: value 5?A@1V 90? Single 3.53V~3.67V 200mW 3.6V SOD-323 Zener Diodes ROHS -> prot_3v3
- OD2: value Red 615~630nm 1.9~2.2V 0603 Light Emitting Diodes (LED) RoHS -> ledr.package
- OD3: value 20mA 285mcd 3.3V 518nm Colorless transparence -40?~+85? 520nm~535nm Emerald 120° 110mW 0603 Light Emitting Diodes (LED)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 -> ledg.package
- OD4: value White 0603 Light Emitting Diodes (LED) RoHS -> ledw.package
- OFB1: value 200mA 1 450m? 600?@100MHz ±25% 0603 Ferrite Beads ROHS -> ferrite
- OH1: value (none) -> jlc_th.th1
- OH2: value (none) -> jlc_th.th2
- OH3: value (none) -> jlc_th.th3
- OJ1: value (none) -> mcu.prog
- OL1: value 620mA 22uH ±10% 270m? 1210 Inductors (SMD) ROHS -> reg_3v3.power_path.inductor
- OR1: value ±1% 1/10W Thick Film Resistors 75V ±100ppm/? -55?~+155? 6.8k? 0603 Chip Resistor - Surface Mount ROHS -> reg_3v3.fb.top_res
- OR2: value ±1% 1/10W Thick Film Resistors 75V ±100ppm/? -55?~+155? 1.5k? 0603 Chip Resistor - Surface Mount ROHS -> reg_3v3.fb.bottom_res
- OR3: value ±1% 1/10W Thick Film Resistors 75V ±100ppm/? -55?~+155? 510k? 0603 Chip Resistor - Surface Mount ROHS -> reg_3v3.en_res
- OR4: value ±1% 1/10W Thick Film Resistors 75V ±100ppm/? -55?~+155? 10k? 0603 Chip Resistor - Surface Mount ROHS -> mcu.en_pull.r
- OR5: value ±1% 1/10W Thick Film Resistors 75V ±100ppm/? -55?~+155? 1k? 0603 Chip Resistor - Surface Mount ROHS -> ledr.res
- OR6: value ±1% 1/10W Thick Film Resistors 75V ±100ppm/? -55?~+155? 1k? 0603 Chip Resistor - Surface Mount ROHS -> ledg.res
- OR7: value ±1% 1/10W Thick Film Resistors 75V ±100ppm/? -55?~+155? 1k? 0603 Chip Resistor - Surface Mount ROHS -> ledw.res
- OR8: value ±1% 1/10W Thick Film Resistors 75V ±100ppm/? -55?~+155? 91k? 0603 Chip Resistor - Surface Mount ROHS -> vobd_sense.top_res
- OR9: value ±1% 1/10W Thick Film Resistors 75V ±100ppm/? -55?~+155? 10k? 0603 Chip Resistor - Surface Mount ROHS -> vobd_sense.bottom_res
- OU1: value (none) -> obd
- OU2: value TPS54202H -> reg_3v3.ic
- OU3: value ESP32-C3-WROOM-02 -> mcu.ic
- OU4: value SN65HVD230DR -> can.ic
Changed lines of the file:
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@@
 		(tags "SOD-323")
 		(property "Reference" "OD1"
-			(at -2 0 360)
+			(at -2 0 0)
 			(layer "F.SilkS")
 			(effects
@@
 			)
 		)
-		(property "Value" "5?A@1V 90? Single 3.53V~3.67V 200mW 3.6V SOD-323 Zener Diodes ROHS"
+		(property "Value" "prot_3v3"
 			(at 0.1 1.9 90)
 			(layer "F.Fab")
@@
 			)
 		)
-		(property "Value" "50V 100nF X7R ±10% 0603 Multilayer Ceramic Capacitors MLCC - SMD/SMT ROHS"
+		(property "Value" "reg_3v3.boot_cap"
 			(at 0 1.43 90)
 			(layer "F.Fab")
@@
 			)
 		)
-		(property "Value" "200mA 1 450m? 600?@100MHz ±25% 0603 Ferrite Beads ROHS"
+		(property "Value" "ferrite"
 			(at 0 1.43 90)
 			(layer "F.Fab")
@@
 		(tags "resistor")
 		(property "Reference" "OR4"
-			(at -3 0 360)
+			(at -3 0 0)
 			(layer "F.SilkS")
 			(effects
@@
 			)
 		)
-		(property "Value" "±1% 1/10W Thick Film Resistors 75V ±100ppm/? -55?~+155? 10k? 0603 Chip Resistor - Surface Mount ROHS"
+		(property "Value" "mcu.en_pull.r"
 			(at 0 1.43 90)
 			(layer "F.Fab")
@@
 			)
 		)
-		(property "Value" "ESP32-C3-WROOM-02"
+		(property "Value" "mcu.ic"
 			(at 0 8.33 90)
 			(layer "F.Fab")
@@
 			)
 		)
-		(property "Value" "White 0603 Light Emitting Diodes (LED) RoHS"
+		(property "Value" "ledw.package"
 			(at 0 1.43 90)
 			(layer "F.Fab")
@@
 			)
 		)
-		(property "Value" "20mA 285mcd 3.3V 518nm Colorless transparence -40?~+85? 520nm~535nm Emerald 120° 110mW 0603 Light Emitting Diodes (LED) ROHS"
+		(property "Value" "ledg.package"
 			(at 0 1.43 90)
 			(layer "F.Fab")
@@
 		(tags "capacitor")
 		(property "Reference" "OC4"
-			(at 0 -1.5 360)
+			(at 0 -1.5 0)
 			(layer "F.SilkS")
 			(effects
@@
 			)
 		)
-		(property "Value" "X5R 25V ±10% 10uF 0805 Multilayer Ceramic Capacitors MLCC - SMD/SMT ROHS"
-			(at 0 1.68 360)
+		(property "Value" "reg_3v3.power_path.out_cap"
+			(at 0 1.68 0)
 			(layer "F.Fab")
 			(effects
@@
 		)
 		(fp_text user "${REFERENCE}"
-			(at 0 0 360)
+			(at 0 0 0)
 			(layer "F.Fab")
 			(effects
@@
 			)
 		)
-		(property "Value" "50V 100nF X7R ±10% 0603 Multilayer Ceramic Capacitors MLCC - SMD/SMT ROHS"
+		(property "Value" "reg_3v3.hf_in_cap"
 			(at 0 1.43 90)
 			(layer "F.Fab")
@@
 			)
 		)
-		(property "Value" "±1% 1/10W Thick Film Resistors 75V ±100ppm/? -55?~+155? 91k? 0603 Chip Resistor - Surface Mount ROHS"
+		(property "Value" "vobd_sense.top_res"
 			(at 0 1.43 90)
 			(layer "F.Fab")
@@
 			)
 		)
-		(property "Value" "25V 22uF X5R ±10% 1206 Multilayer Ceramic Capacitors MLCC - SMD/SMT ROHS"
+		(property "Value" "reg_3v3.power_path.in_cap"
 			(at 0 1.85 90)
 			(layer "F.Fab")
@@
 			)
 		)
-		(property "Value" "±1% 1/10W Thick Film Resistors 75V ±100ppm/? -55?~+155? 1k? 0603 Chip Resistor - Surface Mount ROHS"
+		(property "Value" "ledr.res"
 			(at 0 1.43 90)
 			(layer "F.Fab")
@@
 			)
 		)
-		(property "Value" "±1% 1/10W Thick Film Resistors 75V ±100ppm/? -55?~+155? 10k? 0603 Chip Resistor - Surface Mount ROHS"
+		(property "Value" "vobd_sense.bottom_res"
 			(at 0 1.43 90)
 			(layer "F.Fab")
@@
 			)
 		)
-		(property "Value" ""
+		(property "Value" "jlc_th.th3"
 			(at 0 -2 0)
 			(layer "F.Fab")
@@
 		(tags "capacitor")
 		(property "Reference" "OC6"
-			(at -2 0 360)
+			(at -2 0 0)
 			(layer "F.SilkS")
 			(effects
@@
 			)
 		)
-		(property "Value" "50V 100nF X7R ±10% 0603 Multilayer Ceramic Capacitors MLCC - SMD/SMT ROHS"
+		(property "Value" "mcu.vcc_cap1"
 			(at 0 1.43 90)
 			(layer "F.Fab")
@@
 			)
 		)
-		(property "Value" "50V 100nF X7R ±10% 0603 Multilayer Ceramic Capacitors MLCC - SMD/SMT ROHS"
+		(property "Value" "can.vdd_cap"
 			(at 0 1.43 90)
 			(layer "F.Fab")
@@
 			)
 		)
-		(property "Value" "SN65HVD230DR"
+		(property "Value" "can.ic"
 			(at 0 3.4 90)
 			(layer "F.Fab")
@@
 			)
 		)
-		(property "Value" "±1% 1/10W Thick Film Resistors 75V ±100ppm/? -55?~+155? 1.5k? 0603 Chip Resistor - Surface Mount ROHS"
+		(property "Value" "reg_3v3.fb.bottom_res"
 			(at 0 1.43 90)
 			(layer "F.Fab")
@@
 			)
 		)
-		(property "Value" "TPS54202H"
+		(property "Value" "reg_3v3.ic"
 			(at 0 2.4 90)
 			(layer "F.Fab")
@@
 			)
 		)
-		(property "Value" "620mA 22uH ±10% 270m? 1210 Inductors (SMD) ROHS"
+		(property "Value" "reg_3v3.power_path.inductor"
 			(at 0 2.28 0)
 			(layer "F.Fab")
@@
 			)
 		)
-		(property "Value" "X5R 25V ±10% 10uF 0805 Multilayer Ceramic Capacitors MLCC - SMD/SMT ROHS"
+		(property "Value" "mcu.vcc_cap0"
 			(at 0 1.68 90)
 			(layer "F.Fab")
@@
 			)
 		)
-		(property "Value" "50V 1uF X5R ±10% 0603 Multilayer Ceramic Capacitors MLCC - SMD/SMT ROHS"
+		(property "Value" "mcu.en_pull.c"
 			(at 0 1.43 90)
 			(layer "F.Fab")
@@
 			)
 		)
-		(property "Value" "±1% 1/10W Thick Film Resistors 75V ±100ppm/? -55?~+155? 510k? 0603 Chip Resistor - Surface Mount ROHS"
+		(property "Value" "reg_3v3.en_res"
 			(at 0 1.43 90)
 			(layer "F.Fab")
@@
 			)
 		)
-		(property "Value" "±1% 1/10W Thick Film Resistors 75V ±100ppm/? -55?~+155? 1k? 0603 Chip Resistor - Surface Mount ROHS"
+		(property "Value" "ledw.res"
 			(at 0 1.43 90)
 			(layer "F.Fab")
@@
 			)
 		)
-		(property "Value" ""
+		(property "Value" "jlc_th.th1"
 			(at 0 -2 0)
 			(layer "F.Fab")
@@
 			)
 		)
-		(property "Value" "Red 615~630nm 1.9~2.2V 0603 Light Emitting Diodes (LED) RoHS"
+		(property "Value" "ledr.package"
 			(at 0 1.43 90)
 			(layer "F.Fab")
@@
 			)
 		)
-		(property "Value" ""
+		(property "Value" "mcu.prog"
 			(at 0 -2.3 90)
 			(layer "F.Fab")
@@
 			)
 		)
-		(property "Value" ""
+		(property "Value" "jlc_th.th2"
 			(at 0 -2 0)
 			(layer "F.Fab")
@@
 			)
 		)
-		(property "Value" "±1% 1/10W Thick Film Resistors 75V ±100ppm/? -55?~+155? 6.8k? 0603 Chip Resistor - Surface Mount ROHS"
+		(property "Value" "reg_3v3.fb.top_res"
 			(at 0 1.43 90)
 			(layer "F.Fab")
@@
 			)
 		)
-		(property "Value" "±1% 1/10W Thick Film Resistors 75V ±100ppm/? -55?~+155? 1k? 0603 Chip Resistor - Surface Mount ROHS"
+		(property "Value" "ledg.res"
 			(at 0 1.43 90)
 			(layer "F.Fab")
@@
 			)
 		)
-		(property "Value" ""
+		(property "Value" "obd"
 			(at 0 -2 0)
 			(unlocked yes)
