File: examples/UsbSourceMeasure/JfetCurrentClamp.kicad_sch (KiCad schematic)
At the start: 3 parts, among them Q1 MMBFJ112, Q2 MMBFJ112

Commit message: rc2
Parts:
- Q1, Q2: Refdes Prefix (none) -> Q
Changed lines of the file:
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@@
+			)
+		)
+		(property "Refdes Prefix" "Q"
+			(at 115.57 124.46 90)
+			(effects
+				(font
+					(size 1.27 1.27)
+				)
+				(hide yes)
 			)
 		)
@@
 			(at 138.43 129.54 90)
 			(effects
+				(font
+					(size 1.27 1.27)
+				)
+				(hide yes)
+			)
+		)
+		(property "Refdes Prefix" "Q"
+			(at 138.43 129.54 90)
+			(effects
