File: examples/UsbSourceMeasure/SourceMeasureControl.kicad_sch (KiCad schematic)
At the start: 27 parts

Commit message: SMU3.1 fixes (#443)
https://github.com/ducky64/usb-source-measure/issues/7 - slow down
control loop (reduce opamp integrator gain), in particular to get it
slower than the current sense RC filter. Also renames 'factor' to 'gain'
and adds an intuitive meaning of the term in the docs.

https://github.com/ducky64/usb-source-measure/issues/8 - reduce current
sense gain to 5x to allow 3A at full scale

https://github.com/ducky64/usb-source-measure/issues/1 - fix ramp at low
voltages, previously it was calculating the divider for gate voltage
relative to ground, whereas for PMOS it needs to be gate voltage
relative to source = Vin.

These have been tested with board component replacements and work.
Parts:
- imeas: Value2 ratio=10*Ratio(tol=0.05)) -> ratio=5*Ratio(tol=0.05))
- int: Value2 factor=1/4.7e-6*Ratio(tol=0.15), -> gain=100/4.7*kHertz(tol=0.15),; Value3 capacitance=1*nFarad(tol=0.1)) -> capacitance=10*nFarad(tol=0.1))
Changed lines of the file:
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@@
 			)
 		)
-		(property "Value2" "factor=1/4.7e-6*Ratio(tol=0.15),"
+		(property "Value2" "gain=100/4.7*kHertz(tol=0.15),"
 			(at 113.03 101.346 0)
 			(effects
@@
 			)
 		)
-		(property "Value3" "capacitance=1*nFarad(tol=0.1))"
+		(property "Value3" "capacitance=10*nFarad(tol=0.1))"
 			(at 113.03 103.632 0)
 			(effects
@@
 			)
 		)
-		(property "Value2" "ratio=10*Ratio(tol=0.05))"
+		(property "Value2" "ratio=5*Ratio(tol=0.05))"
 			(at 237.49 128.016 0)
 			(effects

Commit message: wip
Parts:
- ifilt: Value3 cutoff_freq=(47, 470)*kHertz) -> cutoff_freq=(1, 10)*MHertz)
Other:
- note added: "only for a bit of CMRR"
Changed lines of the file:
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@@
+		)
+	)
+	(text "only for a bit of CMRR"
+		(exclude_from_sim no)
+		(at 197.358 116.078 0)
+		(effects
+			(font
+				(size 1.27 1.27)
+			)
 		)
 	)
@@
 			)
 		)
-		(property "Value3" "cutoff_freq=(47, 470)*kHertz)"
+		(property "Value3" "cutoff_freq=(1, 10)*MHertz)"
 			(at 214.884 124.206 0)
 			(effects

Commit message: wip new params
Parts:
- int: value #IntegratorInverting( -> #CompensatorType2(; Field7 (none) -> k=2.4, crossover_gain=100); Value2 gain=100/4.7*kHertz(tol=0.15), -> rin=4.7*kOhm(tol=0.02),; Value3 capacitance=10*nFarad(tol=0.1)) -> crossover_freq=500*KHertz(tol=0.25),
Other:
- note added: "plant parameters (crossover_gain) determined using SPICE, see analysis folder"
Changed lines of the file:
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@@
+		)
+	)
+	(text "plant parameters (crossover_gain)\ndetermined using SPICE, see analysis folder"
+		(exclude_from_sim no)
+		(at 100.076 112.014 0)
+		(effects
+			(font
+				(size 1.27 1.27)
+			)
+			(justify left bottom)
 		)
 	)
@@
 			)
 		)
-		(property "Value" "#IntegratorInverting("
+		(property "Value" "#CompensatorType2("
 			(at 113.03 99.06 0)
 			(effects
@@
 			)
 		)
-		(property "Value2" "gain=100/4.7*kHertz(tol=0.15),"
+		(property "Value2" "rin=4.7*kOhm(tol=0.02),"
 			(at 113.03 101.346 0)
 			(effects
@@
 			)
 		)
-		(property "Value3" "capacitance=10*nFarad(tol=0.1))"
+		(property "Value3" "crossover_freq=500*KHertz(tol=0.25),"
 			(at 113.03 103.632 0)
 			(effects
 				(font
+					(size 1.27 1.27)
+				)
+			)
+		)
+		(property "Field7" "k=2.4, crossover_gain=100)"
+			(at 113.03 105.918 0)
+			(effects
+				(font

Commit message: stabilized @ fc=80kHz
Parts:
- int: Field7 k=2.4, crossover_gain=100) -> (none); Value3 crossover_freq=500*KHertz(tol=0.25), -> crossover_freq=100*kHertz(tol=0.10),; Value4 (none) -> k=2.4, crossover_gain=0.075)
Changed lines of the file:
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@@
 			)
 		)
-		(property "Value3" "crossover_freq=500*KHertz(tol=0.25),"
+		(property "Value3" "crossover_freq=100*kHertz(tol=0.10),"
 			(at 113.03 103.632 0)
 			(effects
@@
 			)
 		)
-		(property "Field7" "k=2.4, crossover_gain=100)"
+		(property "Value4" "k=2.4, crossover_gain=0.075)"
 			(at 113.03 105.918 0)
 			(effects

Commit message: tuned control loop
Parts:
- int: Value4 k=2.4, crossover_gain=0.075) -> k=2.4*Ratio(tol=0.20), crossover_gain=0.1)
Changed lines of the file:
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@@
 			)
 		)
-		(property "Value4" "k=2.4, crossover_gain=0.075)"
+		(property "Value4" "k=2.4*Ratio(tol=0.20), crossover_gain=0.1)"
 			(at 113.03 105.918 0)
 			(effects
