File: edg/abstract_parts/resources/CompensatorType2.kicad_sch (KiCad schematic)
At the start: 5 parts

Commit message: stabilized @ fc=80kHz
Parts:
- amp: value ${SIM.PARAMS} -> (none)
Changed lines of the file:
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@@
 			)
 		)
-		(property "Value" "${SIM.PARAMS}"
+		(property "Value" ""
 			(at 137.16 86.741 0)
 			(effects
