File: examples/Keyboard/Keyboard.kicad_pcb (KiCad board)
At the start: 2 copper layers, 26 parts, among them J1 COM-15111, J2 PinHeader1.27 Shrouded 2x5, SW1 PG151101S11, SW2 PG151101S11, SW3 PG151101S11, SW4 PG151101S11, SW5 PG151101S11, SW6 PG151101S11, U1 LDL1117S33R, U2 STM32F103xxT6

Commit message: wip
Parts:
- added C10: , Capacitor_SMD:C_0603_1608Metric, F.Cu at (150.0, 53.0)
- added C9: , Capacitor_SMD:C_0603_1608Metric, F.Cu at (150.0, 47.0)
- added R3: , Resistor_SMD:R_0603_1608Metric, F.Cu at (140.0, 57.0)
- added X1: , Crystal:Crystal_SMD_3225-4Pin_3.2x2.5mm, F.Cu at (150.0, 50.0)
- moved C1 5.00 mm to (138.0, 45.0)
- moved C2 5.00 mm to (142.0, 45.0)
- moved J1 5.00 mm to (125.0, 48.0)
- moved R1 5.00 mm to (127.5, 54.3)
- moved R2 5.00 mm to (122.5, 54.3)
- moved U1 5.00 mm to (140.0, 51.0)
Connections:
- U2 pad 32: (no net) -> usb.usb.dm
- U2 pad 33: (no net) -> usb.usb.dp
- U2 pad 5: mcu.ic.osc.xtal_in -> mcu.xtal_node.driver.xtal_in
- U2 pad 6: mcu.ic.osc.xtal_out -> mcu.xtal_node.driver.xtal_out

Commit message: wip keyboard layout
wow that was fast
Parts:
- removed the C3 at (165.0, 57.0)
- removed the C4 at (165.0, 55.0)
- added C10: sw.sw[0,1].npx.cap, Capacitor_SMD:C_0603_1608Metric, B.Cu at (159.1, 88.0)
- added C11: sw.sw[0,2].npx.cap, Capacitor_SMD:C_0603_1608Metric, B.Cu at (178.1, 88.0)
- added C12: sw.sw[1,0].npx.cap, Capacitor_SMD:C_0603_1608Metric, B.Cu at (140.0, 107.0)
- added C13: sw.sw[1,1].npx.cap, Capacitor_SMD:C_0603_1608Metric, B.Cu at (159.1, 107.0)
- added C14: sw.sw[1,2].npx.cap, Capacitor_SMD:C_0603_1608Metric, B.Cu at (178.1, 107.0)
- added C15: sw.sw[2,0].npx.cap, Capacitor_SMD:C_0603_1608Metric, B.Cu at (140.0, 126.1)
- added C16: sw.sw[2,1].npx.cap, Capacitor_SMD:C_0603_1608Metric, B.Cu at (159.1, 126.1)
- added C17: sw.sw[2,2].npx.cap, Capacitor_SMD:C_0603_1608Metric, B.Cu at (178.1, 126.1)
- added C18: sw.sw[3,0].npx.cap, Capacitor_SMD:C_0603_1608Metric, B.Cu at (140.0, 145.2)
- added C19: sw.sw[3,1].npx.cap, Capacitor_SMD:C_0603_1608Metric, B.Cu at (159.1, 145.2)
- added C20: sw.sw[3,2].npx.cap, Capacitor_SMD:C_0603_1608Metric, B.Cu at (178.1, 145.2)
- added C21: oled.c1_cap, Capacitor_SMD:C_0603_1608Metric, F.Cu at (103.4, 20.4)
- added C22: oled.c2_cap, Capacitor_SMD:C_0603_1608Metric, F.Cu at (103.4, 22.9)
- added C23: oled.vcomh_cap, Capacitor_SMD:C_0805_2012Metric, F.Cu at (98.0, 41.0)
- added C24: oled.vdd_cap1, Capacitor_SMD:C_0603_1608Metric, F.Cu at (103.4, 25.4)
- added C25: oled.vbat_cap, Capacitor_SMD:C_0603_1608Metric, F.Cu at (103.4, 27.9)
- added C26: oled.vcc_cap, Capacitor_SMD:C_0805_2012Metric, F.Cu at (98.0, 44.0)
- added C27: npx_shift.vdd_cap, Capacitor_SMD:C_0603_1608Metric, F.Cu at (93.2, 59.3)
- added C9: sw.sw[0,0].npx.cap, Capacitor_SMD:C_0603_1608Metric, B.Cu at (140.0, 88.0)
- added D10: sw.sw[1,1].d, Diode_SMD:D_SOD-323, B.Cu at (165.1, 104.0)
- added D11: sw.sw[1,1].npx.device, edg:LED_SK6812MINI-E, F.Cu at (159.1, 104.0)
- added D12: sw.sw[1,2].d, Diode_SMD:D_SOD-323, B.Cu at (184.1, 104.0)
- added D13: sw.sw[1,2].npx.device, edg:LED_SK6812MINI-E, F.Cu at (178.1, 104.0)
- added D14: sw.sw[2,0].d, Diode_SMD:D_SOD-323, B.Cu at (146.0, 123.1)
- added D15: sw.sw[2,0].npx.device, edg:LED_SK6812MINI-E, F.Cu at (140.0, 123.1)
- added D16: sw.sw[2,1].d, Diode_SMD:D_SOD-323, B.Cu at (165.1, 123.1)
- added D17: sw.sw[2,1].npx.device, edg:LED_SK6812MINI-E, F.Cu at (159.1, 123.1)
- added D18: sw.sw[2,2].d, Diode_SMD:D_SOD-323, B.Cu at (184.1, 123.1)
- added D19: sw.sw[2,2].npx.device, edg:LED_SK6812MINI-E, F.Cu at (178.1, 123.1)
- added D20: sw.sw[3,0].d, Diode_SMD:D_SOD-323, B.Cu at (146.0, 142.2)
- added D21: sw.sw[3,0].npx.device, edg:LED_SK6812MINI-E, F.Cu at (140.0, 142.2)
- added D22: sw.sw[3,1].d, Diode_SMD:D_SOD-323, B.Cu at (165.1, 142.2)
- added D23: sw.sw[3,1].npx.device, edg:LED_SK6812MINI-E, F.Cu at (159.1, 142.2)
- added D24: sw.sw[3,2].d, Diode_SMD:D_SOD-323, B.Cu at (184.1, 142.2)
- added D25: sw.sw[3,2].npx.device, edg:LED_SK6812MINI-E, F.Cu at (178.1, 142.2)
- added D7: sw.sw[0,2].npx.device, edg:LED_SK6812MINI-E, F.Cu at (178.1, 85.0)
- added D8: sw.sw[1,0].d, Diode_SMD:D_SOD-323, B.Cu at (146.0, 104.0)
- added D9: sw.sw[1,0].npx.device, edg:LED_SK6812MINI-E, F.Cu at (140.0, 104.0)
- added J3: oled.device, Connector_FFC-FPC:Hirose_FH12-30S-0.5SH_1x30-1MP_P0.50mm_Horizontal, F.Cu at (159.1, 68.0)
- added R4: oled.iref_res, Resistor_SMD:R_0603_1608Metric, F.Cu at (103.4, 30.4)
- added SW10: sw.sw[3,0].sw, Switch_Keyboard_Hotswap_Kailh:SW_Hotswap_Kailh_MX, F.Cu at (140.0, 137.2)
- added SW11: sw.sw[3,1].sw, Switch_Keyboard_Hotswap_Kailh:SW_Hotswap_Kailh_MX, F.Cu at (159.1, 137.2)
- added SW12: sw.sw[3,2].sw, Switch_Keyboard_Hotswap_Kailh:SW_Hotswap_Kailh_MX, F.Cu at (178.1, 137.2)
- added SW13: enc, edg:RotaryEncoder_Bourns_PEC11S, F.Cu at (178.1, 61.0)
- added SW7: sw.sw[2,0].sw, Switch_Keyboard_Hotswap_Kailh:SW_Hotswap_Kailh_MX, F.Cu at (140.0, 118.1)
- added SW8: sw.sw[2,1].sw, Switch_Keyboard_Hotswap_Kailh:SW_Hotswap_Kailh_MX, F.Cu at (159.1, 118.1)
- added SW9: sw.sw[2,2].sw, Switch_Keyboard_Hotswap_Kailh:SW_Hotswap_Kailh_MX, F.Cu at (178.1, 118.1)
- added TP1: _npx_shift_output_link, TestPoint:TestPoint_Keystone_5015_Micro-Minature, F.Cu at (66.0, 58.0)
- added U3: usb_esd, Package_TO_SOT_SMD:SOT-23, F.Cu at (66.1, 53.4)
- added U4: oled.lcd, edg:Lcd_Er_Oled0.96_1.1_Outline, F.Cu at (38.4, 41.2)
- added U5: npx_shift.ic, Package_TO_SOT_SMD:SOT-23-5, F.Cu at (93.8, 55.8)
- C1: value (none) -> reg.in_cap
- C2: value (none) -> reg.out_cap
- C3: renamed from C9; value (none) -> mcu.crystal.cap_a
- C4: renamed from C10; value (none) -> mcu.crystal.cap_b
- C5: value (none) -> mcu.vdd_cap[0]
- C6: value (none) -> mcu.vdd_cap[1]
- C7: value (none) -> mcu.vdda_cap
- C8: value (none) -> mcu.reset_cap
- D1: value 40V 550mV@1A 1A SMA(DO-214AC) Schottky Barrier Diodes (SBD) ROHS -> ledr.package; footprint Diode_SMD:D_SMA -> LED_SMD:LED_0603_1608Metric
- D2: value 40V 550mV@1A 1A SMA(DO-214AC) Schottky Barrier Diodes (SBD) ROHS -> sw.sw[0,0].d; footprint Diode_SMD:D_SMA -> Diode_SMD:D_SOD-323; moved to B.Cu
- D3: value 40V 550mV@1A 1A SMA(DO-214AC) Schottky Barrier Diodes (SBD) ROHS -> sw.sw[0,0].npx.device; footprint Diode_SMD:D_SMA -> edg:LED_SK6812MINI-E
- D4: value 40V 550mV@1A 1A SMA(DO-214AC) Schottky Barrier Diodes (SBD) ROHS -> sw.sw[0,1].d; footprint Diode_SMD:D_SMA -> Diode_SMD:D_SOD-323; moved to B.Cu
- D5: value 40V 550mV@1A 1A SMA(DO-214AC) Schottky Barrier Diodes (SBD) ROHS -> sw.sw[0,1].npx.device; footprint Diode_SMD:D_SMA -> edg:LED_SK6812MINI-E
- D6: value 40V 550mV@1A 1A SMA(DO-214AC) Schottky Barrier Diodes (SBD) ROHS -> sw.sw[0,2].d; footprint Diode_SMD:D_SMA -> Diode_SMD:D_SOD-323; moved to B.Cu
- J1: value COM-15111 -> usb.conn
- J2: value PinHeader1.27 Shrouded 2x5 -> mcu.sdi; footprint Connector_PinHeader_1.27mm:PinHeader_2x05_P1.27mm_Vertical_SMD -> Connector_PinHeader_2.54mm:PinHeader_1x04_P2.54mm_Vertical
- R1: value (none) -> usb.cc_pull.cc1
- R2: value (none) -> usb.cc_pull.cc2
- R3: value (none) -> ledr.res
- SW1: value PG151101S11 -> sw.sw[0,0].sw
- SW2: value PG151101S11 -> sw.sw[0,1].sw
- SW3: value PG151101S11 -> sw.sw[0,2].sw
- SW4: value PG151101S11 -> sw.sw[1,0].sw
- SW5: value PG151101S11 -> sw.sw[1,1].sw
- SW6: value PG151101S11 -> sw.sw[1,2].sw
- U1: value LDL1117S33R -> reg.ic
- U2: value STM32F103xxT6 -> mcu.ic; footprint Package_QFP:LQFP-48_7x7mm_P0.5mm -> Package_QFP:LQFP-32_7x7mm_P0.8mm
- X1: value (none) -> mcu.crystal.package
- moved D4 45.1 mm to (165.1, 85.0)
- moved C6 43.7 mm to (197.0, 33.0), turned to 0 degrees
- moved C4 40.8 mm to (183.0, 29.0), turned to 0 degrees
- moved C3 38.6 mm to (183.0, 27.0), turned to 180 degrees
- moved C7 36.9 mm to (183.0, 31.0)
- moved X1 36.4 mm to (179.0, 28.0)
- moved C1 36.1 mm to (168.0, 25.0)
- moved C2 36.1 mm to (172.0, 25.0)
- moved U1 36.1 mm to (170.0, 31.0)
- moved U2 36.1 mm to (190.0, 30.0)
- moved R3 35.4 mm to (111.4, 77.9)
- moved C8 35.4 mm to (179.0, 31.0)
- moved J2 31.2 mm to (148.0, 28.9)
- moved C5 26.9 mm to (183.0, 25.0), turned to 180 degrees
- moved D3 26.9 mm to (140.0, 85.0), turned to 180 degrees
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Connections:
- net usb.conn.A5 renamed usb.conn.cc.cc1
- net usb.conn.B5 renamed usb.conn.cc.cc2
- C3 pad 1: mcu.xtal_node.driver.xtal_in -> mcu.xtal_node.xi
- C4 pad 1: mcu.xtal_node.driver.xtal_out -> mcu.xtal_node.xo
- C8 pad 1: reg.pwr_out -> mcu.ic.nrst
- D1 pad 1: sw.d[0,0].cathode -> ledr.package.k
- D1 pad 2: sw.rows.0 -> reg.pwr_out
- D2 pad 1: sw.d[0,1].cathode -> mcu.gpio.1_0
- D2 pad 2: sw.rows.1 -> sw.sw[0,0].sw.com
- D3 pad 1: sw.d[0,2].cathode -> usb.pwr
- D3 pad 2: sw.rows.2 -> sw.sw[0,0].npx_dout
- D4 pad 1: sw.d[1,0].cathode -> mcu.gpio.1_1
- D4 pad 2: sw.rows.0 -> sw.sw[0,1].sw.com
- D5 pad 1: sw.d[1,1].cathode -> usb.pwr
- D5 pad 2: sw.rows.1 -> sw.sw[0,1].npx_dout
- D6 pad 1: sw.d[1,2].cathode -> mcu.gpio.1_2
- D6 pad 2: sw.rows.2 -> sw.sw[0,2].sw.com
- J1 pad A6: usb.usb.dp -> usb_chain_0.d_P
- J1 pad A7: usb.usb.dm -> usb_chain_0.d_N
- J1 pad B6: usb.usb.dp -> usb_chain_0.d_P
- J1 pad B7: usb.usb.dm -> usb_chain_0.d_N
- J2 pad 2: mcu.swd_node.swdio -> usb.gnd
- J2 pad 3: usb.gnd -> mcu.ic.swdio
- J2 pad 4: mcu.swd_node.swclk -> mcu.ic.swclk
- R3 pad 1: reg.pwr_out -> ledr.package.k
- R3 pad 2: usb.usb.dp -> ledr.signal
- SW1 pad 1: sw.d[0,0].cathode -> mcu.gpio.0_0
- SW1 pad 2: sw.cols.0 -> sw.sw[0,0].sw.com
- SW2 pad 1: sw.d[0,1].cathode -> mcu.gpio.0_0
- SW2 pad 2: sw.cols.0 -> sw.sw[0,1].sw.com
- SW3 pad 1: sw.d[0,2].cathode -> mcu.gpio.0_0
- SW3 pad 2: sw.cols.0 -> sw.sw[0,2].sw.com
- SW4 pad 1: sw.d[1,0].cathode -> mcu.gpio.0_1
- SW4 pad 2: sw.cols.1 -> sw.sw[1,0].sw.com
- SW5 pad 1: sw.d[1,1].cathode -> mcu.gpio.0_1
- SW5 pad 2: sw.cols.1 -> sw.sw[1,1].sw.com
- SW6 pad 1: sw.d[1,2].cathode -> mcu.gpio.0_1
- SW6 pad 2: sw.cols.1 -> sw.sw[1,2].sw.com
- U2 pad 10: sw.cols.0 -> oled.cs
- U2 pad 11: sw.cols.1 -> oled.spi.sck
- U2 pad 12: sw.rows.0 -> oled.spi.miso
- U2 pad 13: sw.rows.1 -> oled.spi.mosi
- U2 pad 14: sw.rows.2 -> oled.dc
- U2 pad 15: (no net) -> oled.reset
- U2 pad 16: (no net) -> usb.gnd
- U2 pad 17: (no net) -> reg.pwr_out
- U2 pad 18: (no net) -> npx_shift.input
- U2 pad 19: (no net) -> mcu.gpio.0_0
- U2 pad 2: (no net) -> mcu.xtal_node.xi
- U2 pad 20: (no net) -> mcu.gpio.0_1
- U2 pad 21: (no net) -> usb_chain_0.d_N
- U2 pad 22: (no net) -> usb_chain_0.d_P
- U2 pad 23: usb.gnd -> mcu.ic.swdio
- U2 pad 24: reg.pwr_out -> mcu.ic.swclk
- U2 pad 25: (no net) -> mcu.gpio.0_2
- U2 pad 26: (no net) -> mcu.gpio.0_3
- U2 pad 27: (no net) -> mcu.gpio.1_0
- U2 pad 28: (no net) -> mcu.gpio.1_1
- U2 pad 29: (no net) -> mcu.gpio.1_2
- U2 pad 3: (no net) -> mcu.xtal_node.xo
- U2 pad 31: (no net) -> usb.gnd
- U2 pad 32: usb.usb.dm -> usb.gnd
- U2 pad 4: (no net) -> mcu.ic.nrst
- U2 pad 5: mcu.xtal_node.driver.xtal_in -> reg.pwr_out
- U2 pad 6: mcu.xtal_node.driver.xtal_out -> ledr.signal
- U2 pad 7: mcu.reset_node -> enc.a
- U2 pad 8: usb.gnd -> enc.b
- U2 pad 9: reg.pwr_out -> enc.sw
- X1 pad 1: mcu.xtal_node.driver.xtal_in -> mcu.xtal_node.xi
- X1 pad 3: mcu.xtal_node.driver.xtal_out -> mcu.xtal_node.xo
Routing:
- net mcu.gpio.1_0: track 0.00 -> 78.3 mm, vias 0 -> 4
- net mcu.gpio.0_3: track 0.00 -> 68.1 mm
- net mcu.gpio.0_2: track 0.00 -> 68.1 mm
- net mcu.gpio.0_1: track 0.00 -> 68.1 mm
- net mcu.gpio.1_1: track 0.00 -> 64.3 mm, vias 0 -> 4
- net mcu.gpio.1_2: track 0.00 -> 64.1 mm, vias 0 -> 4
- net usb.pwr: track 0.00 -> 57.8 mm, vias 0 -> 11
- net mcu.gpio.0_0: track 0.00 -> 49.9 mm
- net usb.gnd: track 0.00 -> 23.9 mm, vias 0 -> 13
- net sw.sw[2,2].sw.com: track 0.00 -> 11.0 mm
- net sw.sw[2,0].sw.com: track 0.00 -> 11.0 mm
- net sw.sw[1,2].sw.com: track 0.00 -> 11.0 mm
- net sw.sw[1,0].sw.com: track 0.00 -> 11.0 mm
- net sw.sw[0,2].sw.com: track 0.00 -> 11.0 mm
- net sw.sw[0,0].sw.com: track 0.00 -> 11.0 mm
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Other:
- board outline added: 3.4 x 4.2 mm

Commit message: macropad layout wip
Parts:
- removed TP1: _npx_shift_output_link, TestPoint:TestPoint_Keystone_5015_Micro-Minature
- added REF**: MountingHole_2.7mm_M2.5, MountingHole:MountingHole_2.7mm_M2.5, F.Cu at (130.0, 147.2)
- added REF**: MountingHole_2.7mm_M2.5, MountingHole:MountingHole_2.7mm_M2.5, F.Cu at (188.1, 50.0)
- added REF**: MountingHole_2.7mm_M2.5, MountingHole:MountingHole_2.7mm_M2.5, F.Cu at (130.0, 50.0)
- added REF**: MountingHole_2.7mm_M2.5, MountingHole:MountingHole_2.7mm_M2.5, F.Cu at (188.1, 147.2)
- moved U3 74.0 mm to (140.0, 58.0), turned to -90 degrees
- moved R1 15.9 mm to (143.0, 58.0)
- moved R2 15.0 mm to (137.0, 58.0)
- moved J1 3.00 mm to (140.0, 50.7)
Routing:
- net usb_chain_0.d_P: track 0.00 -> 2.90 mm
- net usb_chain_0.d_N: track 0.00 -> 2.52 mm
- added copper zone on F.Cu, net (none)
Other:
- board size 3.4 x 4.2 mm -> 64.1 x 103.2 mm

Commit message: Update Keyboard.kicad_pcb
Parts:
- C21, C22, C23, C24, C25, C26, R4: moved to B.Cu
- moved J3 81.1 mm to (80.0, 50.0)
- moved U4 43.5 mm to (80.0, 54.0), turned to 180 degrees
- moved C21 33.2 mm to (85.0, 48.0), turned to -90 degrees
- moved C24 31.8 mm to (81.0, 48.0), turned to 90 degrees
- moved R4 31.7 mm to (77.0, 48.0), turned to -90 degrees
- moved C22 30.0 mm to (87.0, 48.0), turned to 90 degrees
- moved C25 28.6 mm to (83.0, 48.0), turned to 90 degrees
- moved C26 25.3 mm to (73.0, 48.0), turned to 90 degrees
- moved C23 24.0 mm to (75.0, 48.0), turned to 90 degrees

Commit message: Update Keyboard.kicad_pcb
Parts:
- moved C27 16.9 mm to (110.0, 57.0), turned to 180 degrees
- moved U5 16.7 mm to (110.0, 60.0)
- moved C22 14.6 mm to (73.0, 52.0), turned to -90 degrees
- moved C26 14.6 mm to (87.0, 52.0), turned to -90 degrees
- moved C21 10.8 mm to (75.0, 52.0), turned to 90 degrees
- moved C23 10.8 mm to (85.0, 52.0), turned to -90 degrees
- moved U4 8.00 mm to (80.0, 46.0), turned to 0 degrees
- moved C25 7.21 mm to (77.0, 52.0), turned to -90 degrees
- moved R4 7.21 mm to (83.0, 52.0), turned to 90 degrees
- moved C24 4.47 mm to (79.0, 52.0), turned to -90 degrees
- turned J3 to 0 degrees

Commit message: Update Keyboard.kicad_pcb
Parts:
- moved R3 51.0 mm to (60.4, 77.9)
- moved C21 51.0 mm to (24.0, 52.0)
- moved C22 51.0 mm to (22.0, 52.0)
- moved C23 51.0 mm to (34.0, 52.0)
- moved C24 51.0 mm to (28.0, 52.0)
- moved C25 51.0 mm to (26.0, 52.0)
- moved C26 51.0 mm to (36.0, 52.0)
- moved C27 51.0 mm to (59.0, 57.0)
- moved D1 51.0 mm to (60.4, 75.3)
- moved J3 51.0 mm to (29.0, 50.0)
- moved R4 51.0 mm to (32.0, 52.0)
- moved U4 51.0 mm to (29.0, 46.0)
- moved U5 51.0 mm to (59.0, 60.0)
- moved C10 44.7 mm to (119.0, 108.0)
- moved C13 44.7 mm to (119.0, 127.0)
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
Commit message: generate in row order
Parts:
- C1, C27, C3, C4, C5, C6, C7, C8, D1, R1, R2, R3, U2, U3, U5, X1: moved to B.Cu
- C10: value sw.sw[0,1].npx.cap -> sw.sw[1,0].npx.cap
- C11: value sw.sw[0,2].npx.cap -> sw.sw[2,0].npx.cap
- C12: value sw.sw[1,0].npx.cap -> sw.sw[0,1].npx.cap
- C14: value sw.sw[1,2].npx.cap -> sw.sw[2,1].npx.cap
- C15: value sw.sw[2,0].npx.cap -> sw.sw[0,2].npx.cap
- C16: value sw.sw[2,1].npx.cap -> sw.sw[1,2].npx.cap
- C18: value sw.sw[3,0].npx.cap -> sw.sw[0,3].npx.cap
- C19: value sw.sw[3,1].npx.cap -> sw.sw[1,3].npx.cap
- C2: footprint Capacitor_SMD:C_0805_2012Metric -> Capacitor_SMD:C_0603_1608Metric; moved to B.Cu
- C20: value sw.sw[3,2].npx.cap -> sw.sw[2,3].npx.cap
- D12: value sw.sw[1,2].d -> sw.sw[2,1].d
- D13: value sw.sw[1,2].npx.device -> sw.sw[2,1].npx.device
- D14: value sw.sw[2,0].d -> sw.sw[0,2].d
- D15: value sw.sw[2,0].npx.device -> sw.sw[0,2].npx.device
- D16: value sw.sw[2,1].d -> sw.sw[1,2].d
- D17: value sw.sw[2,1].npx.device -> sw.sw[1,2].npx.device
- D20: value sw.sw[3,0].d -> sw.sw[0,3].d
- D21: value sw.sw[3,0].npx.device -> sw.sw[0,3].npx.device
- D22: value sw.sw[3,1].d -> sw.sw[1,3].d
- D23: value sw.sw[3,1].npx.device -> sw.sw[1,3].npx.device
- D24: value sw.sw[3,2].d -> sw.sw[2,3].d
- D25: value sw.sw[3,2].npx.device -> sw.sw[2,3].npx.device
- D4: value sw.sw[0,1].d -> sw.sw[1,0].d
- D5: value sw.sw[0,1].npx.device -> sw.sw[1,0].npx.device
- D6: value sw.sw[0,2].d -> sw.sw[2,0].d
- D7: value sw.sw[0,2].npx.device -> sw.sw[2,0].npx.device
- D8: value sw.sw[1,0].d -> sw.sw[0,1].d
- D9: value sw.sw[1,0].npx.device -> sw.sw[0,1].npx.device
- SW10: value sw.sw[3,0].sw -> sw.sw[0,3].sw
- SW11: value sw.sw[3,1].sw -> sw.sw[1,3].sw
- SW12: value sw.sw[3,2].sw -> sw.sw[2,3].sw
- SW2: value sw.sw[0,1].sw -> sw.sw[1,0].sw
- SW3: value sw.sw[0,2].sw -> sw.sw[2,0].sw
- SW4: value sw.sw[1,0].sw -> sw.sw[0,1].sw
- SW6: value sw.sw[1,2].sw -> sw.sw[2,1].sw
- SW7: value sw.sw[2,0].sw -> sw.sw[0,2].sw
- SW8: value sw.sw[2,1].sw -> sw.sw[1,2].sw
- U1: footprint Package_TO_SOT_SMD:SOT-223-3_TabPin2 -> Package_TO_SOT_SMD:SOT-89-3; moved to B.Cu
- moved C21 98.6 mm to (115.0, 90.0), turned to -90 degrees
- moved C22 98.6 mm to (113.0, 90.0)
- moved C23 98.6 mm to (125.0, 90.0)
- moved C24 98.6 mm to (119.0, 90.0)
- moved C25 98.6 mm to (117.0, 90.0)
- moved C26 98.6 mm to (127.0, 90.0)
- moved R4 98.6 mm to (123.0, 90.0)
- moved J3 97.5 mm to (120.0, 85.0)
- moved U4 97.1 mm to (120.0, 80.0)
- moved C6 52.6 mm to (116.0, 86.0)
- moved U5 50.8 mm to (100.0, 90.0), turned to -90 degrees
- moved C1 50.4 mm to (96.0, 84.0), turned to 90 degrees
- moved C27 50.3 mm to (97.0, 90.0), turned to 90 degrees
- moved C2 48.0 mm to (104.0, 84.0), turned to 90 degrees
- moved U1 44.6 mm to (100.0, 84.0)
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Connections:
- net sw.sw[3,0].sw.com renamed sw.sw[0,3].sw.com
- net sw.sw[3,1].sw.com renamed sw.sw[1,3].sw.com
- net sw.sw[3,2].sw.com renamed sw.sw[2,3].sw.com
- D12 pad 1: mcu.gpio.1_2 -> mcu.gpio.1_1
- D12 pad 2: sw.sw[1,2].sw.com -> sw.sw[2,1].sw.com
- D13 pad 2: sw.sw[1,2].npx_dout -> sw.sw[1,1].npx_din
- D13 pad 4: sw.sw[0,2].npx_dout -> sw.sw[2,0].npx_dout
- D14 pad 1: mcu.gpio.1_0 -> mcu.gpio.1_2
- D14 pad 2: sw.sw[2,0].sw.com -> sw.sw[0,2].sw.com
- D15 pad 2: sw.sw[2,0].npx_dout -> sw.sw[0,2].npx_dout
- D15 pad 4: sw.sw[1,0].npx_dout -> sw.sw[0,1].npx_dout
- D16 pad 1: mcu.gpio.1_1 -> mcu.gpio.1_2
- D16 pad 2: sw.sw[2,1].sw.com -> sw.sw[1,2].sw.com
- D17 pad 2: sw.sw[1,1].npx_din -> sw.sw[1,2].npx_dout
- D17 pad 4: sw.sw[2,1].npx_din -> sw.sw[0,2].npx_dout
- D20 pad 1: mcu.gpio.1_0 -> mcu.gpio.1_3
- D21 pad 2: sw.sw[3,0].npx_dout -> sw.npx_dout
- D21 pad 4: sw.sw[2,0].npx_dout -> sw.sw[0,3].npx_din
- D22 pad 1: mcu.gpio.1_1 -> mcu.gpio.1_3
- D23 pad 2: sw.sw[2,1].npx_din -> sw.sw[0,3].npx_din
- D23 pad 4: sw.sw[3,0].npx_dout -> sw.sw[1,3].npx_din
- D24 pad 1: mcu.gpio.1_2 -> mcu.gpio.1_3
- D25 pad 2: sw.npx_dout -> sw.sw[1,3].npx_din
- D4 pad 1: mcu.gpio.1_1 -> mcu.gpio.1_0
- D4 pad 2: sw.sw[0,1].sw.com -> sw.sw[1,0].sw.com
- D5 pad 2: sw.sw[0,1].npx_dout -> sw.sw[1,0].npx_dout
- D5 pad 4: sw.sw[0,1].npx_din -> sw.sw[0,0].npx_dout
- D6 pad 1: mcu.gpio.1_2 -> mcu.gpio.1_0
- D6 pad 2: sw.sw[0,2].sw.com -> sw.sw[2,0].sw.com
- D7 pad 2: sw.sw[0,2].npx_dout -> sw.sw[2,0].npx_dout
- D7 pad 4: sw.sw[0,1].npx_dout -> sw.sw[1,0].npx_dout
- D8 pad 1: mcu.gpio.1_0 -> mcu.gpio.1_1
- D8 pad 2: sw.sw[1,0].sw.com -> sw.sw[0,1].sw.com
- D9 pad 2: sw.sw[1,0].npx_dout -> sw.sw[0,1].npx_dout
- D9 pad 4: sw.sw[0,0].npx_dout -> sw.sw[0,1].npx_din
- SW10 pad 1: mcu.gpio.0_3 -> mcu.gpio.0_0
- SW11 pad 1: mcu.gpio.0_3 -> mcu.gpio.0_1
- SW12 pad 1: mcu.gpio.0_3 -> mcu.gpio.0_2
- SW2 pad 1: mcu.gpio.0_0 -> mcu.gpio.0_1
- SW2 pad 2: sw.sw[0,1].sw.com -> sw.sw[1,0].sw.com
- SW3 pad 1: mcu.gpio.0_0 -> mcu.gpio.0_2
- SW3 pad 2: sw.sw[0,2].sw.com -> sw.sw[2,0].sw.com
- SW4 pad 1: mcu.gpio.0_1 -> mcu.gpio.0_0
- SW4 pad 2: sw.sw[1,0].sw.com -> sw.sw[0,1].sw.com
- SW6 pad 1: mcu.gpio.0_1 -> mcu.gpio.0_2
- SW6 pad 2: sw.sw[1,2].sw.com -> sw.sw[2,1].sw.com
- SW7 pad 1: mcu.gpio.0_2 -> mcu.gpio.0_0
- SW7 pad 2: sw.sw[2,0].sw.com -> sw.sw[0,2].sw.com
- SW8 pad 1: mcu.gpio.0_2 -> mcu.gpio.0_1
- SW8 pad 2: sw.sw[2,1].sw.com -> sw.sw[1,2].sw.com
- U1 pad 2: reg.pwr_out -> usb.pwr
- U1 pad 3: usb.pwr -> reg.pwr_out
- U2 pad 26: mcu.gpio.0_3 -> mcu.gpio.1_0
- U2 pad 27: mcu.gpio.1_0 -> mcu.gpio.1_1
- U2 pad 28: mcu.gpio.1_1 -> mcu.gpio.1_2
- U2 pad 29: mcu.gpio.1_2 -> mcu.gpio.1_3
Routing:
- net usb.gnd: track 23.9 -> 116.0 mm, vias 13 -> 38
- net mcu.gpio.0_3: track 68.1 -> 0.00 mm
- net reg.pwr_out: track 0.00 -> 50.3 mm, vias 0 -> 3
- net usb_chain_0.d_N: track 2.52 -> 29.9 mm, vias 0 -> 1
- net usb_chain_0.d_P: track 2.90 -> 27.2 mm, vias 0 -> 1
- net mcu.gpio.0_2: track 68.1 -> 47.1 mm
- net mcu.gpio.0_1: track 68.1 -> 50.1 mm
- net mcu.gpio.0_0: track 49.9 -> 65.1 mm
- net oled.device.c2n: track 0.00 -> 9.67 mm, vias 0 -> 1
- net oled.device.c1n: track 0.00 -> 9.25 mm, vias 0 -> 1
- net (no net): track 0.00 -> 8.99 mm
- net mcu.xtal_node.xi: track 0.00 -> 8.96 mm
- net oled.device.iref: track 0.00 -> 8.27 mm, vias 0 -> 1
- net sw.sw[2,0].npx_dout: track 0.00 -> 8.00 mm
- net oled.device.c2p: track 0.00 -> 7.46 mm, vias 0 -> 1
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
Commit message: Update Keyboard.kicad_pcb
Parts:
- turned C12 to 0 degrees
- turned C13 to 0 degrees
- turned C14 to 0 degrees
- turned C18 to 0 degrees
- turned C19 to 0 degrees
- turned C20 to 0 degrees
- turned D11 to 0 degrees
- turned D13 to 0 degrees
- turned D21 to 0 degrees
- turned D23 to 0 degrees
- turned D25 to 0 degrees
- turned D9 to 0 degrees
Routing:
- net sw.sw[0,1].npx_dout: track 0.00 -> 30.0 mm
- net sw.sw[2,2].npx_dout: track 0.00 -> 28.9 mm
- net usb.gnd: track 116.0 -> 92.0 mm, vias 38 -> 32
- net usb.pwr: track 50.9 -> 74.9 mm, vias 1 -> 19
- net sw.sw[2,0].npx_dout: track 8.00 -> 29.0 mm
- net mcu.gpio.0_1: track 50.1 -> 68.1 mm
- net sw.sw[0,1].npx_din: track 0.00 -> 14.4 mm
- net sw.sw[0,0].npx_dout: track 0.00 -> 14.4 mm
- net sw.sw[0,3].npx_din: track 0.00 -> 14.4 mm
- net sw.sw[0,2].npx_dout: track 0.00 -> 14.4 mm
- net sw.sw[1,3].npx_din: track 0.00 -> 14.4 mm
- net sw.sw[1,1].npx_din: track 0.00 -> 14.4 mm
- net sw.sw[1,2].npx_dout: track 0.00 -> 14.4 mm
- net sw.sw[1,0].npx_dout: track 0.00 -> 14.4 mm
- net mcu.gpio.0_0: track 65.1 -> 51.6 mm
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