File: examples/IotFan/IotFan_control.kicad_pcb (KiCad board)
At the start: 2 copper layers, 24 x 70 mm, 47 parts

Commit message: wip
Parts:
- removed the FC15 at (124.0, 108.5)
- removed the FC16 at (124.0, 111.0)
- removed the FD4 at (128.0, 113.0)
- removed the FU7 at (115.1, 100.0)
- FJ6, FJ8: moved to B.Cu
- turned FJ6 to 180 degrees
- turned FJ8 to 180 degrees
- renumbered FC8 to FC10, FC9 to FC11, FC10 to FC12, FC11 to FC13, FC12 to FC14, FC13 to FC15, FC14 to FC16, FD5 to FD4, FD6 to FD5, FD7 to FD6, FD8 to FD7, FD9 to FD8, FD10 to FD9, FR7 to FR10, FR8 to FR11, FR9 to FR12, FR10 to FR13, FR11 to FR14, FR12 to FR15, FR13 to FR16, FR5 to FR8, FR6 to FR9, FU8 to FU7
Connections:
- FJ4 pad 2: Fcontrol.reg_qwiic.pwr_out -> Fcontrol.v3v3
Routing:
- net Fcontrol.gnd: track 12.3 -> 14.6 mm, vias 3 -> 5
- net Fcontrol.v5: track 0.00 -> 1.09 mm, vias 0 -> 1

Commit message: layout wip
Parts:
- moved FD6 16.0 mm to (106.9, 96.0)
- moved FD9 16.0 mm to (93.1, 104.0)
- moved FC20 12.0 mm to (105.2, 97.0)
- moved FC23 12.0 mm to (94.8, 103.0)
- moved FR10 9.49 mm to (98.0, 112.0), turned to 0 degrees
- moved FR11 8.54 mm to (102.0, 112.0)
- moved FD4 8.00 mm to (93.1, 96.0), turned to 60 degrees
- moved FD5 8.00 mm to (100.0, 92.0), turned to 0 degrees
- moved FD7 8.00 mm to (106.9, 104.0), turned to -120 degrees
- moved FD8 8.00 mm to (100.0, 108.0), turned to 180 degrees
- moved FC18 6.00 mm to (94.8, 97.0), turned to -120 degrees
- moved FC19 6.00 mm to (100.0, 94.0), turned to 180 degrees
- moved FC21 6.00 mm to (105.2, 103.0), turned to 60 degrees
- moved FC22 6.00 mm to (100.0, 106.0), turned to 0 degrees
- moved FC16 4.12 mm to (111.0, 120.0), turned to -90 degrees
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Connections:
- FJ6 pad 1: Fcontrol.v5 -> Fcontrol.v3v3
- FJ8 pad 1: Fcontrol.v3v3 -> Fcontrol.v5
- FJ8 pad 2: Fcontrol.drv -> Fcontrol.tach
- FJ8 pad 3: Fcontrol.tach -> Fcontrol.drv
- FR9 pad 2: Fcontrol.ledr.signal -> Fcontrol.mcu.program_boot_node
- FU4 pad 10: (no net) -> Fcontrol.pd_int
- FU4 pad 11: (no net) -> Fcontrol.i2c.scl
- FU4 pad 12: Fcontrol.pwm -> Fcontrol.i2c.sda
- FU4 pad 31: (no net) -> Fcontrol.enc_sw
- FU4 pad 32: (no net) -> Fcontrol.enc_b
- FU4 pad 33: (no net) -> Fcontrol.enc_a
- FU4 pad 35: (no net) -> Fcontrol.extra1
- FU4 pad 38: Fcontrol.i2c.sda -> Fcontrol.drv
- FU4 pad 39: Fcontrol.i2c.scl -> Fcontrol.tach
- FU4 pad 4: Fcontrol.pd_int -> (no net)
- FU4 pad 5: Fcontrol.spk -> (no net)
- FU4 pad 6: Fcontrol.drv -> Fcontrol.npx_shift.input
- FU4 pad 7: Fcontrol.tach -> Fcontrol.npx_en
- FU4 pad 8: (no net) -> Fcontrol.pwm
- FU4 pad 9: (no net) -> Fcontrol.spk
Routing:
- net Fcontrol.v5: track 1.09 -> 57.4 mm, vias 1 -> 7
- net Fcontrol.gnd: track 14.6 -> 49.7 mm, vias 5 -> 15
- net Fcontrol.npx_shift.input: track 0.00 -> 27.5 mm, vias 0 -> 2
- net Fcontrol.v3v3: track 1.70 -> 28.1 mm, vias 2 -> 9
- net Fcontrol.mcu.program_uart_node.b_tx: track 0.00 -> 25.2 mm, vias 0 -> 2
- net Fcontrol.mcu.program_uart_node.a_tx: track 0.00 -> 23.3 mm, vias 0 -> 2
- net Fcontrol.mcu.program_en_node: track 0.00 -> 23.1 mm
- net Fcontrol.i2c.scl: track 0.00 -> 15.5 mm, vias 0 -> 2
- net Fcontrol.i2c.sda: track 0.00 -> 14.6 mm, vias 0 -> 2
- net Fcontrol.mcu.program_boot_node: track 0.00 -> 12.7 mm
- net Fcontrol.npx.led[4].dout: track 0.00 -> 9.10 mm
- net Fcontrol.npx.led[1].dout: track 0.00 -> 9.10 mm
- net Fcontrol.npx.led[3].dout: track 0.00 -> 8.77 mm
- net Fcontrol.npx.led[0].dout: track 0.00 -> 8.74 mm
- net Fcontrol.drv: track 0.00 -> 8.71 mm, vias 0 -> 1
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- added copper zone on B.Cu, net Fcontrol.gnd
- added copper zone on F.Cu, net Fcontrol.gnd
- added copper zone on B.Cu, net Fcontrol.v3v3
- added copper zone on B.Cu, net Fcontrol.v5
- removed copper zone on B.Cu, net (none)
- removed copper zone on F.Cu, net (none)

Commit message: Update IotFan_control.kicad_pcb
Parts:
- moved UU4 36.1 mm to (98.0, 74.0)
- moved FC14 3.16 mm to (94.0, 116.0), turned to 90 degrees
- moved FR14 3.16 mm to (93.0, 113.0), turned to 180 degrees
Routing:
- net Fcontrol.i2c.sda: track 14.6 -> 61.4 mm, vias 2 -> 6
- net Fcontrol.i2c.scl: track 15.5 -> 61.2 mm, vias 2 -> 5
- net Fcontrol.v3v3: track 28.1 -> 58.3 mm, vias 9 -> 14
- net Fcontrol.dist.ic.int: track 0.00 -> 7.41 mm
- net Fcontrol.gnd: track 49.7 -> 54.0 mm, vias 15 -> 20
- net Fcontrol.dist.ic.rsvd6: track 0.00 -> 4.23 mm
- net Fcontrol.dist.ic.i2c_rst: track 0.00 -> 2.84 mm
- net Fcontrol.dist.ic.lpn: track 0.00 -> 2.13 mm
- net Fcontrol.v5: track 57.4 -> 56.6 mm

Commit message: Update IotFan_control.kicad_pcb
Routing:
- net Fcontrol.v3v3: track 58.3 -> 91.4 mm, vias 14 -> 15
- net Fcontrol.mcu.program_en_node: track 23.1 -> 41.2 mm, vias 0 -> 2
- net Fcontrol.gnd: track 54.0 -> 56.0 mm, vias 20 -> 22
- net Fcontrol.mcu.program_uart_node.a_tx: track 23.3 -> 24.1 mm
- net Fcontrol.i2c.sda: track 61.4 -> 62.1 mm
- net Fcontrol.i2c.scl: track 61.2 -> 61.9 mm

Commit message: routing
Parts:
- moved FC17 20.9 mm to (110.0, 103.0), turned to 0 degrees
- moved FU7 20.0 mm to (110.0, 100.0), turned to 180 degrees
- moved FD5 16.0 mm to (100.0, 108.0), turned to 180 degrees
- moved FD8 16.0 mm to (100.0, 92.0), turned to 0 degrees
- moved FD4 16.0 mm to (106.9, 104.0), turned to -120 degrees
- moved FD6 16.0 mm to (93.1, 104.0), turned to 120 degrees
- moved FD7 16.0 mm to (93.1, 96.0), turned to 60 degrees
- moved FD9 16.0 mm to (106.9, 96.0), turned to -60 degrees
- moved FR11 15.6 mm to (90.0, 102.0)
- moved FR10 14.4 mm to (90.0, 100.0)
- moved FC19 12.0 mm to (100.0, 106.0), turned to 0 degrees
- moved FC22 12.0 mm to (100.0, 94.0), turned to 180 degrees
- moved FC18 12.0 mm to (105.2, 103.0), turned to 60 degrees
- moved FC20 12.0 mm to (94.8, 103.0), turned to -60 degrees
- moved FC21 12.0 mm to (94.8, 97.0), turned to -120 degrees
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Connections:
- FU4 pad 4: (no net) -> Fcontrol.npx_shift.input
- FU4 pad 6: Fcontrol.npx_shift.input -> (no net)
Routing:
- net Fcontrol.i2c.sda: track 62.1 -> 31.0 mm, vias 6 -> 4
- net Fcontrol.i2c.scl: track 61.9 -> 30.9 mm, vias 5 -> 4
- net Fcontrol.gnd: track 56.0 -> 85.9 mm, vias 22 -> 34
- net Fcontrol.v5: track 56.6 -> 69.3 mm, vias 7 -> 12
- net Fcontrol.npx_shift.input: track 27.7 -> 40.1 mm, vias 2 -> 4
- net Fcontrol.v3v3: track 91.4 -> 92.8 mm, vias 15 -> 13
- net Fcontrol.enc_sw: track 8.48 -> 7.75 mm
- net Fcontrol.enc_a: track 7.15 -> 7.67 mm
- net Fcontrol.dist.ic.i2c_rst: track 2.84 -> 2.34 mm

Commit message: Update IotFan_control.kicad_pcb
Routing:
- net Fcontrol.v3v3: track 92.8 -> 93.5 mm
- net Fcontrol.gnd: vias 34 -> 42
Changed lines of the file:
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@@
-	)
-	(segment
-		(start 101 76)
-		(end 103 78)
-		(width 0.25)
-		(layer "F.Cu")
-		(net 21)
-	)
-	(segment
-		(start 103 86)
-		(end 105 88)
-		(width 0.25)
-		(layer "F.Cu")
-		(net 21)
 	)
 	(segment
@@
 	)
 	(segment
-		(start 103 78)
-		(end 103 86)
+		(start 101 76)
+		(end 105 80)
 		(width 0.25)
 		(layer "F.Cu")
@@
 		(net 21)
 	)
+	(segment
+		(start 105 80)
+		(end 105 88)
+		(width 0.25)
+		(layer "F.Cu")
+		(net 21)
+	)
 	(via
 		(at 94 76)
@@
 		(drill 0.3)
 		(layers "F.Cu" "B.Cu")
+		(net 21)
+	)
+	(segment
+		(start 109 94)
+		(end 109 100)
+		(width 0.25)
+		(layer "B.Cu")
 		(net 21)
 	)
@@
 	)
 	(segment
+		(start 94.89184 76.89184)
+		(end 94 76)
+		(width 0.25)
+		(layer "B.Cu")
+		(net 21)
+	)
+	(segment
+		(start 105 88)
+		(end 105 89.5)
+		(width 0.25)
+		(layer "B.Cu")
+		(net 21)
+	)
+	(segment
 		(start 108 92.5)
 		(end 108 93)
@@
 	)
 	(segment
-		(start 94.89184 76.89184)
-		(end 94 76)
+		(start 108 93)
+		(end 109 94)
 		(width 0.25)
 		(layer "B.Cu")
@@
 	)
 	(segment
-		(start 109 94)
-		(end 109 100)
+		(start 100.10816 76.89184)
+		(end 94.89184 76.89184)
 		(width 0.25)
 		(layer "B.Cu")
@@
 		(start 105 89.5)
 		(end 108 92.5)
-		(width 0.25)
-		(layer "B.Cu")
-		(net 21)
-	)
-	(segment
-		(start 100.10816 76.89184)
-		(end 94.89184 76.89184)
-		(width 0.25)
-		(layer "B.Cu")
-		(net 21)
-	)
-	(segment
-		(start 108 93)
-		(end 109 94)
-		(width 0.25)
-		(layer "B.Cu")
-		(net 21)
-	)
-	(segment
-		(start 105 88)
-		(end 105 89.5)
 		(width 0.25)
 		(layer "B.Cu")
@@
 	)
 	(segment
+		(start 111.5 96.5)
+		(end 110.865 96.5)
+		(width 0.25)
+		(layer "F.Cu")
+		(net 29)
+	)
+	(segment
 		(start 106.62 119.5)
 		(end 106.62 118.38)
@@
 		(start 89 94.5)
 		(end 89.525 93.975)
+		(width 0.25)
+		(layer "F.Cu")
+		(net 29)
+	)
+	(segment
+		(start 110.865 96.5)
+		(end 110.635 96.27)
 		(width 0.25)
 		(layer "F.Cu")
@@
 	)
 	(segment
-		(start 110.635 96.27)
-		(end 110.77 96.27)
-		(width 0.25)
-		(layer "F.Cu")
-		(net 29)
-	)
-	(segment
 		(start 90.825 115.325)
 		(end 91 115.5)
@@
 	)
 	(segment
-		(start 110.77 96.27)
-		(end 111 96.5)
-		(width 0.25)
-		(layer "F.Cu")
-		(net 29)
-	)
-	(segment
 		(start 93.95 110.95)
 		(end 94 111)
@@
 	)
 	(via
-		(at 111 96.5)
+		(at 111.5 96.5)
 		(size 0.7)
 		(drill 0.3)
@@
 	)
 	(segment
-		(start 111 96.5)
+		(start 111.5 110)
 		(end 111 110.5)
 		(width 0.5)
@@
 	)
 	(segment
+		(start 111.5 96.5)
+		(end 111.5 110)
+		(width 0.5)
+		(layer "B.Cu")
+		(net 29)
+	)
+	(segment
 		(start 94 123)
 		(end 93 122)
@@
 	)
 	(via
+		(at 102 86)
+		(size 0.7)
+		(drill 0.3)
+		(layers "F.Cu" "B.Cu")
+		(free yes)
+		(net 30)
+	)
+	(via
 		(at 91 120)
 		(size 0.7)
@@
 	)
 	(via
+		(at 93 82)
+		(size 0.7)
+		(drill 0.3)
+		(layers "F.Cu" "B.Cu")
+		(free yes)
+		(net 30)
+	)
+	(via
 		(at 103.830127 96.633975)
 		(size 0.7)
@@
 	)
 	(via
+		(at 103 73)
+		(size 0.7)
+		(drill 0.3)
+		(layers "F.Cu" "B.Cu")
+		(free yes)
+		(net 30)
+	)
+	(via
+		(at 105 75)
+		(size 0.7)
+		(drill 0.3)
+		(layers "F.Cu" "B.Cu")
+		(free yes)
+		(net 30)
+	)
+	(via
 		(at 91 118)
 		(size 0.7)
@@
 	)
 	(via
+		(at 108 98)
+		(size 0.7)
+		(drill 0.3)
+		(layers "F.Cu" "B.Cu")
+		(free yes)
+		(net 30)
+	)
+	(via
 		(at 101 105)
 		(size 0.7)
@@
 	)
 	(via
+		(at 93 80)
+		(size 0.7)
+		(drill 0.3)
+		(layers "F.Cu" "B.Cu")
+		(free yes)
+		(net 30)
+	)
+	(via
 		(at 108.111216 102.950962)
 		(size 0.7)
@@
 	)
 	(via
+		(at 104 86)
+		(size 0.7)
+		(drill 0.3)
+		(layers "F.Cu" "B.Cu")
+		(free yes)
+		(net 30)
+	)
+	(via
 		(at 103.830127 96.633975)
 		(size 0.7)
@@
 	(via
 		(at 92 90)
+		(size 0.7)
+		(drill 0.3)
+		(layers "F.Cu" "B.Cu")
+		(free yes)
+		(net 30)
+	)
+	(via
+		(at 106.999999 92.500645)
 		(size 0.7)
 		(drill 0.3)
@@
 		(min_thickness 0.2)
 		(filled_areas_thickness no)
-		(fill
+		(fill yes
 			(thermal_gap 0.2)
 			(thermal_bridge_width 0.25)
@@
 		(min_thickness 0.25)
 		(filled_areas_thickness no)
-		(fill
+		(fill yes
 			(thermal_gap 0.5)
 			(thermal_bridge_width 0.5)
@@
 		(min_thickness 0.2)
 		(filled_areas_thickness no)
-		(fill
+		(fill yes
 			(thermal_gap 0.2)
 			(thermal_bridge_width 0.25)
@@
 		(min_thickness 0.25)
 		(filled_areas_thickness no)
-		(fill
+		(fill yes
 			(thermal_gap 0.5)
 			(thermal_bridge_width 0.5)

Commit message: wip
Parts:
- added FJ5: control.qwiic2, Connector_JST:JST_SH_SM04B-SRSS-TB_1x04-1MP_P1.00mm_Horizontal, F.Cu at (109.0, 110.0)
- added FR17: control.i2c2_pull.scl_res, Resistor_SMD:R_0603_1608Metric, F.Cu at (103.0, 112.0)
- added FR18: control.i2c2_pull.sda_res, Resistor_SMD:R_0603_1608Metric, F.Cu at (103.0, 110.0)
- moved FJ4 18.0 mm to (91.0, 110.0), turned to -90 degrees
- moved FC13 4.47 mm to (97.0, 112.0), turned to 0 degrees
- moved FR15 4.47 mm to (97.0, 110.0)
- moved FR10 3.00 mm to (90.0, 97.0)
- moved FR11 3.00 mm to (90.0, 99.0)
- renumbered FJ6 to FJ7, FJ8 to FJ9
Connections:
- FU4 pad 5: (no net) -> Fcontrol.i2c2_pull.i2c.scl
- FU4 pad 6: (no net) -> Fcontrol.i2c2_pull.i2c.sda
Routing:
- net Fcontrol.i2c2_pull.i2c.scl: track 0.00 -> 36.8 mm, vias 0 -> 1
- net Fcontrol.i2c2_pull.i2c.sda: track 0.00 -> 32.4 mm, vias 0 -> 1
- net Fcontrol.v3v3: track 93.5 -> 88.2 mm, vias 13 -> 11
- net Fcontrol.gnd: track 85.9 -> 80.9 mm, vias 42 -> 39
- net Fcontrol.dist.ic.int: track 7.41 -> 6.77 mm
- net Fcontrol.i2c.sda: track 31.0 -> 30.6 mm, vias 4 -> 3
- net Fcontrol.i2c.scl: track 30.9 -> 31.1 mm, vias 4 -> 3

Commit message: wip
Connections:
- FU4 pad 5: Fcontrol.i2c2_pull.i2c.scl -> Fcontrol.npx_en
- FU4 pad 7: Fcontrol.npx_en -> Fcontrol.i2c2_pull.i2c.scl
Routing:
- net Fcontrol.i2c.scl: track 31.1 -> 47.6 mm, vias 3 -> 5
- net Fcontrol.i2c.sda: track 30.6 -> 42.0 mm, vias 3 -> 5
- net Fcontrol.i2c2_pull.i2c.sda: track 32.4 -> 38.9 mm
- net Fcontrol.gnd: track 80.9 -> 75.9 mm, vias 39 -> 40
- net Fcontrol.i2c2_pull.i2c.scl: track 36.8 -> 40.7 mm
- net Fcontrol.v3v3: track 88.2 -> 90.2 mm, vias 11 -> 12
