File: examples/BleJoystick/BleJoystick.kicad_pcb (KiCad board)
At the start: 2 copper layers, 26 x 70 mm, 55 parts

Commit message: Update BleJoystick.kicad_pcb
Routing:
- net Jv3v3: track 84.9 -> 84.2 mm
Changed lines of the file:
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@@
 	)
 	(segment
-		(start 94.882538 147)
-		(end 106 147)
+		(start 94 145)
+		(end 96 147)
 		(width 0.5)
 		(layer "B.Cu")
@@
 	)
 	(segment
-		(start 94 143)
-		(end 94 146.117462)
+		(start 96 147)
+		(end 106 147)
 		(width 0.5)
 		(layer "B.Cu")
@@
 	)
 	(segment
-		(start 94 146.117462)
-		(end 94.882538 147)
-		(width 0.5)
-		(layer "B.Cu")
-		(net 1)
-	)
-	(segment
 		(start 112.5 128)
 		(end 112.5 116.5)
@@
 		(start 93 142)
 		(end 94 143)
+		(width 0.5)
+		(layer "B.Cu")
+		(net 1)
+	)
+	(segment
+		(start 94 143)
+		(end 94 145)
 		(width 0.5)
 		(layer "B.Cu")
@@
 		(min_thickness 0.25)
 		(filled_areas_thickness no)
-		(fill yes
+		(fill
 			(thermal_gap 0.25)
 			(thermal_bridge_width 0.25)
@@
 		(min_thickness 0.2)
 		(filled_areas_thickness no)
-		(fill yes
+		(fill
 			(thermal_gap 0.25)
 			(thermal_bridge_width 0.25)

Commit message: Update BleJoystick.kicad_pcb
Parts:
- moved JTP1 27.8 mm to (81.0, 122.0)
- moved JTP3 5.00 mm to (106.0, 132.0)
- moved JR6 4.00 mm to (94.0, 121.0)
- moved JQ3 2.00 mm to (91.0, 121.0)
- turned JC4 to 90 degrees
Routing:
- net Jvusb: track 2.36 -> 49.7 mm, vias 0 -> 1
- net Jusb_chain_0.d_P: track 0.00 -> 9.83 mm
- net Jusb_chain_0.d_N: track 0.00 -> 8.65 mm
- net Jmcu.usb_res.interior.dm: track 0.00 -> 8.27 mm, vias 0 -> 1
- net Jmcu.usb_res.interior.dp: track 0.00 -> 5.90 mm, vias 0 -> 1
- net Jusb.conn.cc.cc1: track 0.00 -> 4.04 mm
- net Jusb.conn.cc.cc2: track 0.00 -> 3.83 mm
- net Jchg.ic.prog: track 3.48 -> 6.46 mm
- net Jgnd: track 30.2 -> 28.1 mm
- net Jchg.prog_res.gnd: track 2.40 -> 4.28 mm
- net Jv3v3: track 84.2 -> 83.3 mm
- added copper zone on F.Cu, net (none)

Commit message: Update BleJoystick.kicad_pcb
Parts:
- moved JTP1 11.7 mm to (91.0, 128.0)
Changed lines of the file:
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@@
 	(footprint "edg:TestPoint_TE_RCT_0805"
 		(layer "F.Cu")
-		(at 81 122 90)
+		(at 91 128 90)
 		(descr "Adapted from Resistor SMD 0805 (2012 Metric), square (rectangular) end terminal, IPC_7351 nominal, (Body size source: IPC-SM-782 page 72, https://www.pcb-3d.com/wordpress/wp-content/uploads/ipc-sm-782a_amendment_1_and_2.pdf), generated with kicad-footprint-generator")
 		(tags "resistor")

Commit message: Update BleJoystick.kicad_pcb
Parts:
- moved JC5 4.00 mm to (95.0, 114.0), turned to 0 degrees
- moved JC4 3.35 mm to (91.0, 114.0), turned to 180 degrees
Routing:
- net Jvusb: track 49.7 -> 51.8 mm
- net Jvbat: track 34.4 -> 32.6 mm

Commit message: wip
Parts:
- JD3: footprint Diode_SMD:D_SOD-323 -> Diode_SMD:D_SOD-123
- moved JTP3 7.81 mm to (112.0, 137.0)
- moved JD3 6.40 mm to (106.0, 132.0)
- moved JD4 3.14 mm to (101.6, 84.1), turned to -5.625 degrees
- moved JR9 3.14 mm to (98.4, 84.1), turned to -174.375 degrees
- moved JC3 2.00 mm to (110.0, 137.0)
- turned JC8 to -90 degrees
- turned JU6 to -90 degrees
Routing:
- net Jv3v3: track 83.3 -> 144.9 mm, vias 5 -> 9
- net Jbumper_sw.out: track 0.00 -> 32.4 mm, vias 0 -> 1
- net Jtrig.out: track 0.00 -> 29.9 mm, vias 0 -> 1
- net Jledr.signal: track 0.00 -> 28.4 mm, vias 0 -> 1
- net Jgnd: track 28.1 -> 25.4 mm, vias 11 -> 14
- net Jledr.package.k: track 0.00 -> 1.53 mm

Commit message: wip
Parts:
- moved JR11 14.9 mm to (97.0, 136.0), turned to 90 degrees
- moved JR10 13.9 mm to (95.0, 136.0), turned to 90 degrees
- moved JTP4 12.8 mm to (93.0, 132.0), turned to 90 degrees
- moved JTP5 12.2 mm to (93.0, 136.0), turned to 90 degrees
- moved JH3 6.71 mm to (89.0, 138.0)
- moved JR9 1.57 mm to (96.9, 84.3), turned to -168.75 degrees
- moved JD4 1.57 mm to (100.0, 84.0), turned to 0 degrees
- turned JC5 to 180 degrees
Connections:
- JD4 pad 2: Jv3v3 -> Jledr.signal
- JR9 pad 2: Jledr.signal -> Jgnd
- JU4 pad 10: Jbumper_sw.out -> Jgate.btn_out
- JU4 pad 11: Jtrig.out -> Jbtns.io0
- JU4 pad 12: Jvbat_sense.i2c.scl -> (no net)
- JU4 pad 13: Jvbat_sense.i2c.sda -> Jgate.control
- JU4 pad 2: Jbtns.io0 -> Jchg.prog_ctl
- JU4 pad 26: (no net) -> Jvbat_sense.i2c.sda
- JU4 pad 27: (no net) -> Jvbat_sense.i2c.scl
- JU4 pad 3: Jgate.control -> (no net)
- JU4 pad 4: Jgate.btn_out -> Jledr.signal
- JU4 pad 5: Jledr.signal -> Jbumper_sw.out
- JU4 pad 6: Jchg.prog_ctl -> Jtrig.out
- JU4 pad 8: Jstick.pwr -> Jstick.ax1
- JU4 pad 9: Jstick.ax1 -> Jstick.pwr
Routing:
- net Jbumper_sw.out: track 32.4 -> 0.00 mm, vias 1 -> 0
- net Jmcu.swd_node.swdio: track 0.00 -> 32.4 mm, vias 0 -> 2
- net Jmcu.swd_node.swclk: track 0.00 -> 31.3 mm, vias 0 -> 2
- net Jvbat_sense.i2c.scl: track 39.3 -> 70.0 mm, vias 3 -> 5
- net Jledr.signal: track 28.4 -> 0.00 mm, vias 1 -> 0
- net Jvbat_sense.i2c.sda: track 39.6 -> 67.6 mm, vias 3 -> 4
- net Jmcu.reset_node: track 0.00 -> 21.3 mm, vias 0 -> 2
- net Jvbat_gated: track 18.0 -> 33.5 mm
- net Jgate.btn_out: track 0.00 -> 8.30 mm, vias 0 -> 1
- net Jgate.btn_in: track 1.90 -> 9.08 mm
- net Jchg.prog_ctl: track 0.00 -> 6.03 mm, vias 0 -> 1
- net Jstick.pwr: track 0.00 -> 5.91 mm, vias 0 -> 1
- net Jstick.ax2: track 0.00 -> 5.83 mm, vias 0 -> 1
- net Jstick.ax1: track 0.00 -> 5.67 mm, vias 0 -> 1
- net Jv3v3: track 144.9 -> 139.8 mm, vias 9 -> 10
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
Commit message: wip
Parts:
- turned JC6 to 0 degrees
Connections:
- JU4 pad 10: Jgate.btn_out -> Jledr.signal
- JU4 pad 11: Jbtns.io0 -> Jbumper_sw.out
- JU4 pad 13: Jgate.control -> Jgate.btn_out
- JU4 pad 15: (no net) -> Jgate.control
- JU4 pad 4: Jledr.signal -> (no net)
- JU4 pad 5: Jbumper_sw.out -> Jbtns.io0
Routing:
- net Jbumper_sw.out: track 0.00 -> 50.4 mm, vias 0 -> 1
- net Jledr.signal: track 0.00 -> 49.8 mm, vias 0 -> 1
- net Jtrig.out: track 27.1 -> 50.8 mm
- net Jv3v3: track 139.8 -> 150.8 mm, vias 10 -> 14
- net Jgate.control: track 2.36 -> 13.3 mm
- net Jvbat_gated: track 33.5 -> 30.8 mm
- net Jgate.btn_out: track 8.30 -> 6.26 mm
- net Jgnd: track 22.3 -> 20.9 mm, vias 15 -> 18

Commit message: drc cleanish
Parts:
- turned JC7 to 90 degrees
- renumbered JC11 to JC10, JC12 to JC11, JC13 to JC12, JC8 to JC13, JC9 to JC8, JC10 to JC9, JU7 to JU6, JU8 to JU7, JU6 to JU9
Connections:
- JC13 pad 1: Jv3v3 -> Jtrig.pwr
- JU4 pad 12: (no net) -> Jtrig.pwr
- JU4 pad 20: (no net) -> Jbtns.io0
- JU4 pad 5: Jbtns.io0 -> (no net)
- JU9 pad 1: Jv3v3 -> Jtrig.pwr
Routing:
- net Jtrig.pwr: track 0.00 -> 63.6 mm, vias 0 -> 2
- net Jv3v3: track 150.8 -> 139.9 mm, vias 14 -> 11
- net Jmcu.reset_node: track 21.3 -> 31.5 mm
- net Jbtns.io0: track 1.95 -> 9.34 mm
- net Jbumper_sw.out: track 50.4 -> 56.6 mm
- net Jgnd: track 20.9 -> 24.0 mm, vias 18 -> 20
- net Jchg.prog_ctl: track 6.03 -> 5.03 mm
- net Jledr.signal: track 49.8 -> 50.7 mm
- net Jtrig.out: track 50.8 -> 51.4 mm
- added copper zone on F.Cu, net Jvusb
- removed copper zone on F.Cu, net (none)
- removed copper zone on B.Cu, net Jvusb
